Commit message: Hokuyo sensor ray origin corrected

File: tuw_gazebo_models/xacro/laser/hokuyo.xacro (robot description, xacro)
@@ -11,5 +11,5 @@
     <link name="${name}">
       <collision>
-        <origin xyz="0 0 0" rpy="0 0 0"/>
+        <origin xyz="0 0 -0.025" rpy="0 0 0"/>
         <geometry>
           <box size="0.1 0.1 0.1"/>
@@ -17,5 +17,5 @@
       </collision>
       <visual>
-        <origin xyz="0 0 0" rpy="0 0 0"/>
+        <origin xyz="0 0 -0.025" rpy="0 0 0"/>
         <geometry>
           <mesh filename="${meshes}/hokuyo.dae"/>
@@ -24,5 +24,5 @@
       <inertial>
         <mass value="1e-5" />
-        <origin xyz="0 0 0" rpy="0 0 0"/>
+        <origin xyz="0 0 -0.025" rpy="0 0 0"/>
         <inertia ixx="1e-6" ixy="0" ixz="0" iyy="1e-6" iyz="0" izz="1e-6" />
       </inertial>

File: tuw_gazebo_models/xacro/laser/hokuyo_gpu.xacro (robot description, xacro)
@@ -11,5 +11,5 @@
     <link name="${name}">
       <collision>
-        <origin xyz="0 0 0" rpy="0 0 0"/>
+        <origin xyz="0 0 -0.025" rpy="0 0 0"/>
         <geometry>
           <box size="0.1 0.1 0.1"/>
@@ -17,5 +17,5 @@
       </collision>
       <visual>
-        <origin xyz="0 0 0" rpy="0 0 0"/>
+        <origin xyz="0 0 -0.025" rpy="0 0 0"/>
         <geometry>
           <mesh filename="${meshes}/hokuyo.dae"/>
@@ -24,5 +24,5 @@
       <inertial>
         <mass value="1e-5" />
-        <origin xyz="0 0 0" rpy="0 0 0"/>
+        <origin xyz="0 0 -0.025" rpy="0 0 0"/>
         <inertia ixx="1e-6" ixy="0" ixz="0" iyy="1e-6" iyz="0" izz="1e-6" />
       </inertial>

File: tuw_gazebo_models/xacro/pioneer3dx/pioneer3dx.xacro (robot description, xacro)
@@ -6,10 +6,10 @@
   <xacro:include filename="$(find tuw_gazebo_models)/xacro/pioneer3dx/pioneer3dx_body.xacro"/>
   <xacro:pioneer3dx_body name="chassis" parent="base_link" meshes="package://tuw_gazebo_models/meshes/pioneer3dx"/>
-  <!-- Laser-->
+  <!-- Laser -->
   <xacro:include filename="$(find tuw_gazebo_models)/xacro/laser/hokuyo.xacro"/>
-  <xacro:laser name="front_laser" parent="chassis" xyz="0.16 0 0.1" rpy="0 0 0" meshes="package://tuw_gazebo_models/meshes/laser"/>
+  <xacro:laser name="front_laser" parent="chassis" xyz="0.16 0 0.125" rpy="0 0 0" meshes="package://tuw_gazebo_models/meshes/laser"/>
   <!-- GPU Laser
   <xacro:include filename="$(find tuw_gazebo_models)/xacro/laser/hokuyo_gpu.xacro"/>
-  <xacro:laser_gpu name="front_laser" parent="chassis" xyz="0.16 0 0.1" rpy="0 0 0" meshes="package://tuw_gazebo_models/meshes/laser" />
+  <xacro:laser_gpu name="front_laser" parent="chassis" xyz="0.16 0 0.125" rpy="0 0 0" meshes="package://tuw_gazebo_models/meshes/laser" />
   -->
   <!-- Camera
