Commit message: models cleanup

File: tuw_gazebo_models/xacro/laser/RPLidar.xacro (robot description, xacro)
@@ -2,5 +2,7 @@
 <robot xmlns:xacro="http://www.ros.org/wiki/xacro">
 <!-- Front Laser -->
-<xacro:macro name="laser" params="name parent xyz rpy meshes" >
+<xacro:macro name="laser" params="name parent xyz rpy driver:=gpu meshes" >
+  <xacro:if     value="${driver == 'gpu'}"> <xacro:property name="driver_name" value="_gpu"/></xacro:if>
+  <xacro:unless value="${driver == 'gpu'}"> <xacro:property name="driver_name" value=""    /></xacro:unless>
   <joint name="${parent}_${name}_joint" type="fixed">
       <axis xyz="0 0 1" />
@@ -11,5 +13,5 @@
     <link name="${name}">
       <collision>
-        <origin xyz="0 0 -0.025" rpy="0 0 0"/>
+        <origin xyz="0 0 -0.025" rpy="0 0 ${-pi/2}"/>
         <geometry>
           <box size="0.1 0.1 0.1"/>
@@ -17,7 +19,7 @@
       </collision>
       <visual name="RPLidar_visual">
-        <origin xyz="-0.07 -0.11 -0.045" rpy="${pi/2} 0 ${pi}"/>
+        <origin xyz="0 0 0" rpy="0 0 0"/>
         <geometry>
-          <mesh filename="${meshes}/RPLIDAR-A1M1R1_withmotor.STL" scale="0.001 0.001 0.001"/>
+          <mesh filename="${meshes}/RPLidar.dae"/>
         </geometry>
       </visual>
@@ -29,7 +31,9 @@
     </link>
     <gazebo reference="${name}">
-		<material value="Gazebo/FlatBlack"/>
         <sensor name="laser" type="ray">
 		  <pose>0 0 0 0 0 0</pose>
+		  <update_rate>5.5</update_rate>
+          <visualize>true</visualize>
+          <always_on>1</always_on>
           <ray>
             <scan>
@@ -37,24 +41,23 @@
                 <!-- The RPLidar has 360 steps with 1 Degree resolution -->
                 <resolution>1</resolution>
-                <max_angle>3.124139361</max_angle> <!-- 180 Degree -->
-                <min_angle>-3.141592</min_angle> <!-- -180 Degree -->
-                <samples>360</samples>
+                <samples>360</samples> <min_angle>-3.141592</min_angle> <max_angle>3.124139361</max_angle> <!-- -180 to 180 Degree -->
               </horizontal>
             </scan>
             <range>
-              <min>0.08</min>
+              <min>0.2</min>
               <max>6</max>
               <resolution>0.02</resolution>
             </range>
+			<noise>
+				<type>gaussian</type>
+				<mean>0.0</mean>
+				<stddev>0.03</stddev>
+			</noise>
           </ray>
-          <plugin name="laser" filename="libgazebo_ros_laser.so" >
-            <robotNamespace></robotNamespace>
-            <topicName>${name}/scan</topicName>
-            <frameName>${name}</frameName>
+          <plugin name="gazebo_ros_laser_RPLidar_driver" filename="libgazebo${driver_name}_ros_laser.so" >
+			<robotNamespace></robotNamespace>
+			<topicName>${name}/scan</topicName>
+			<frameName>${name}</frameName>
           </plugin>
-          <plugin name="gazebo_ros_laser_controller" filename="libRayPlugin.so" />
-          <always_on>1</always_on>
-          <update_rate>5.5</update_rate>
-          <visualize>true</visualize>
         </sensor>
     </gazebo>

File: tuw_gazebo_models/xacro/laser/Sick-LMS100.xacro (robot description, xacro)
@@ -2,82 +2,73 @@
 <robot xmlns:xacro="http://www.ros.org/wiki/xacro">
 <!-- Front Laser -->
-<xacro:macro name="laser" params="name parent xyz rpy meshes" >
+<xacro:macro name="laser" params="name parent xyz rpy driver:=gpu meshes" >
+  <xacro:if     value="${driver == 'gpu'}"> <xacro:property name="driver_name" value="_gpu"/></xacro:if>
+  <xacro:unless value="${driver == 'gpu'}"> <xacro:property name="driver_name" value=""    /></xacro:unless>
   <joint name="${parent}_${name}_chassis_joint" type="fixed">
-      <axis xyz="0 0 1" />
-      <origin xyz="${xyz}" rpy="${rpy}"/>
-      <parent link="${parent}"/>
-      <child link="${name}_chassis"/>
+	  <axis xyz="0 0 1" />
+	  <origin xyz="${xyz}" rpy="${rpy}"/>
+	  <parent link="${parent}"/>
+	  <child link="${name}_chassis"/>
   </joint>
   <material name="SickBlue">
-    <color rgba="${255/255} ${108/255} ${10/255} 1.0"/>
+	<color rgba="${255/255} ${108/255} ${10/255} 1.0"/>
   </material>
   <link name="${name}_chassis">
-    <collision>
-      <origin xyz="0 0 0.0751" rpy="0 0 0"/>
-      <geometry>
-        <box size="0.094 0.094 0.152"/>
-      </geometry>
-    </collision>
-    <visual>
-      <geometry>
-        <mesh filename="${meshes}/Sick-LMS100.dae"/>
-      </geometry>
-      <material name="SickBlue"/>
-    </visual>
-    <xacro:box_inertial x="0.094" y="0.094"  z="0.152" mass="1.1" />
+	<collision>
+	  <origin xyz="0 0 0.0751" rpy="0 0 0"/>
+	  <geometry>
+		<box size="0.094 0.094 0.152"/>
+	  </geometry>
+	</collision>
+	<visual>
+	  <geometry>
+		<mesh filename="${meshes}/Sick-LMS100.dae"/>
+	  </geometry>
+	  <material name="SickBlue"/>
+	</visual>
+	<xacro:box_inertial x="0.094" y="0.094"  z="0.152" mass="1.1" />
   </link>
   <joint name="${name}_chassis_${name}_joint" type="fixed">
-      <axis xyz="0 0 1" />
-      <origin xyz="0 0 0.115" rpy="0 0 0"/>
-      <parent link="${name}_chassis"/>
-      <child link="${name}"/>
+	  <axis xyz="0 0 1" />
+	  <origin xyz="0 0 0.115" rpy="0 0 0"/>
+	  <parent link="${name}_chassis"/>
+	  <child link="${name}"/>
   </joint>
   <link name="${name}"/>
-    <gazebo reference="${name}">
-        <sensor type="ray" name="${name}_laser_sensor">
-          <pose>0 0 0 0 0 0</pose>
-          <always_on>1</always_on>
-          <update_rate>25</update_rate>
-          <visualize>true</visualize>
-          <ray>
-            <scan>
-              <horizontal>
-                <resolution>1</resolution>
-                <!-- 135 to -135 Degree -->
-                <max_angle>2.356</max_angle>
-                <min_angle>-2.356</min_angle>
-                <samples>1080</samples>
-                <!-- 120 to -120 Degree -->
-                <!--max_angle>2.0944</max_angle>
-                <min_angle>-2.0944</min_angle>
-                <samples>683</samples-->
-                <!-- 100 to -100 Degree -->
-                <!--max_angle>1.745329252</max_angle>
-                <min_angle>-1.745329252</min_angle>
-                <samples>570</samples-->
-                <!-- 110 to -110 Degree -->
-                <!--max_angle>1.919862177</max_angle>
-                <min_angle>-1.919862177</min_angle>
-                <samples>626</samples-->
-              </horizontal>
-            </scan>
-            <range>
-              <min>0.2</min>
-              <max>20.0</max>
-              <resolution>0.01</resolution>
-            </range>
-            <noise>
-              <type>gaussian</type>
-              <mean>0.0</mean>
-              <stddev>0.01</stddev>
-            </noise>
-          </ray>
-          <plugin name="gazebo_ros_head_sick_controller" filename="libgazebo_ros_laser.so" >
-            <robotNamespace></robotNamespace>
-            <topicName>${name}/scan</topicName>
-            <frameName>${name}</frameName>
-          </plugin>
-        </sensor>
-    </gazebo>
+	<gazebo reference="${name}">
+		<sensor type="ray" name="${name}_laser_sensor">
+			<pose>0 0 0 0 0 0</pose>
+			<update_rate>25</update_rate>
+			<always_on>1</always_on>
+			<visualize>true</visualize>
+			<ray>
+				<scan>
+				  <horizontal>
+					<!-- Sick-LMS100 has  683 steps with 0.35139 Degree resolution-->
+					<resolution>1</resolution>
+					<max_angle>2.356000000</max_angle> <min_angle>-2.356000000</min_angle> <samples>1080</samples>     <!-- 135 to -135 Degree -->
+					<!--max_angle>2.094400000</max_angle> <min_angle>-2.094400000</min_angle> <samples>683</samples--> <!-- 120 to -120 Degree -->
+					<!--max_angle>1.745329252</max_angle> <min_angle>-1.745329252</min_angle> <samples>570</samples--> <!-- 100 to -100 Degree -->
+					<!--max_angle>1.919862177</max_angle> <min_angle>-1.919862177</min_angle> <samples>626</samples--> <!-- 110 to -110 Degree -->
+					</horizontal>
+				</scan>
+				<range>
+					<min>0.2</min>
+					<max>20.0</max>
+					<resolution>0.01</resolution>
+				</range>
+				<noise>
+					<type>gaussian</type>
+					<mean>0.0</mean>
+					<stddev>0.01</stddev>
+				</noise>
+			</ray>
+			<plugin name="gazebo_ros_laser_sick_driver" filename="libgazebo${driver_name}_ros_laser.so" >
+				<robotNamespace></robotNamespace>
+				<topicName>${name}/scan</topicName>
+				<frameName>${name}</frameName>
+			</plugin>
+		</sensor>
+	</gazebo>
 </xacro:macro>
 </robot>

File: tuw_gazebo_models/xacro/laser/hokuyo.xacro (robot description, xacro)
@@ -2,5 +2,7 @@
 <robot xmlns:xacro="http://www.ros.org/wiki/xacro">
 <!-- Front Laser -->
-<xacro:macro name="laser" params="name parent xyz rpy meshes" >
+<xacro:macro name="laser" params="name parent xyz rpy driver:=gpu meshes" >
+  <xacro:if     value="${driver == 'gpu'}"> <xacro:property name="driver_name" value="_gpu"/></xacro:if>
+  <xacro:unless value="${driver == 'gpu'}"> <xacro:property name="driver_name" value=""    /></xacro:unless>
   <joint name="${parent}_${name}_joint" type="fixed">
       <axis xyz="0 0 1" />
@@ -28,36 +30,36 @@
       </inertial>
     </link>
-    <gazebo reference="${name}">
-        <sensor name="laser" type="ray">
-        <pose>0 0 0 0 0 0</pose>
-          <ray>
-            <scan>
-              <horizontal>
-                <!-- The URG-04LX-UG01  has  683 steps with 0.35139 Degree resolution -->
-                <resolution>1</resolution>
-                <max_angle>2.0944</max_angle> <!-- 120 Degree -->
-                <min_angle>-2.0944</min_angle> <!-- -120 Degree -->
-                <samples>683</samples>
-              </horizontal>
-            </scan>
-            <range>
-              <min>0.08</min>
-              <max>5</max>
-              <resolution>0.01</resolution>
-            </range>
-          </ray>
-          <plugin name="laser" filename="libgazebo_ros_laser.so" >
-            <robotNamespace></robotNamespace>
-            <topicName>${name}/scan</topicName>
-            <frameName>${name}</frameName>
-          </plugin>
-          <!--
-          <plugin name="laser" filename="libRayPlugin.so" />
-          -->
-          <always_on>1</always_on>
-          <update_rate>30</update_rate>
-          <visualize>true</visualize>
-        </sensor>
-    </gazebo>
+	<gazebo reference="${name}">
+		<sensor name="laser" type="ray">
+			<pose>0 0 0 0 0 0</pose>
+			<update_rate>10</update_rate>
+			<visualize>true</visualize>
+			<always_on>1</always_on>
+			<ray>
+				<scan>
+					<horizontal>
+						<!-- The URG-04LX-UG01  has  683 steps with 0.35139 Degree resolution -->
+						<resolution>1</resolution>
+						<samples>683</samples> <min_angle>-2.0944</min_angle> <max_angle>2.0944</max_angle> <!-- -120 to 120 Degree -->
+					</horizontal>
+				</scan>
+				<range>
+					<min>0.08</min>
+					<max>5</max>
+					<resolution>0.01</resolution>
+				</range>
+				<noise>
+					<type>gaussian</type>
+					<mean>0.0</mean>
+					<stddev>0.03</stddev>
+				</noise>
+			</ray>
+			<plugin name="gazebo_ros_laser_hokuyo_driver" filename="libgazebo${driver_name}_ros_laser.so" >
+				<robotNamespace></robotNamespace>
+				<topicName>${name}/scan</topicName>
+				<frameName>${name}</frameName>
+			</plugin>
+		</sensor>
+	</gazebo>
 </xacro:macro>
 </robot>

File: tuw_gazebo_models/xacro/pioneer3dx/pioneer3dx.xacro (robot description, xacro)
@@ -8,9 +8,5 @@
   <!-- Laser -->
   <xacro:include filename="$(find tuw_gazebo_models)/xacro/laser/hokuyo.xacro"/>
-  <xacro:laser name="front_laser" parent="chassis" xyz="0.16 0 0.125" rpy="0 0 0" meshes="package://tuw_gazebo_models/meshes/laser"/>
-  <!-- GPU Laser
-  <xacro:include filename="$(find tuw_gazebo_models)/xacro/laser/hokuyo_gpu.xacro"/>
-  <xacro:laser_gpu name="front_laser" parent="chassis" xyz="0.16 0 0.125" rpy="0 0 0" meshes="package://tuw_gazebo_models/meshes/laser" />
-  -->
+  <xacro:laser name="front_laser" parent="chassis" xyz="0.16 0 0.125" rpy="0 0 0" driver="gpu" meshes="package://tuw_gazebo_models/meshes/laser"/>
   <!-- Camera
   <xacro:include filename="$(find tuw_gazebo_models)/xacro/camera/camera.xacro"/>

File: tuw_gazebo_models/xacro/pioneer3dx/pioneer3dx_body.xacro (robot description, xacro)
@@ -1,5 +1,5 @@
 <?xml version="1.0"?>
 <robot xmlns:xacro="http://www.ros.org/wiki/xacro">
-  <xacro:include filename="inertia_tensors.xacro"/>
+  <xacro:include filename="../inertia_tensors.xacro"/>
   <xacro:include filename="pioneer3dx_chassis.xacro"/>
   <xacro:include filename="battery_block.xacro"/>
