Commit message: added many environments & sensors

File: tuw_gazebo_models/xacro/pioneer3dx/pioneer3dx_swivel.xacro (robot description, xacro)
@@ -86,5 +86,5 @@
       <inertia ixx="0.012411765597" ixy="-0.000711733678" ixz="0.00050272983" iyy="0.015218160428" iyz="-0.000004273467" izz="0.011763977943"/>
     </inertial>
-    <visual name="base_visual">
+    <visual name="hubcap_visual">
       <origin xyz="0 0 0" rpy="0 0 0"/>
       <geometry name="pioneer_geom">

File: tuw_gazebo_models/xacro/pioneer3dx/pioneer3dx_wheel.xacro (robot description, xacro)
@@ -49,5 +49,5 @@
       <inertia ixx="0.012411765597" ixy="0" ixz="0" iyy="0.015218160428" iyz="0" izz="0.011763977943"/>
     </inertial>
-    <visual name="base_visual">
+    <visual name="wheel_visual">
       <origin xyz="0 0 0" rpy="0 0 0"/>
       <geometry name="pioneer_geom">
