Commit message: RPLidar collision mesh fix

File: tuw_gazebo_models/models/sensors/laser/RPLidar.xacro (robot description, xacro)
@@ -15,5 +15,5 @@
 	    <origin xyz="0 0 -0.025" rpy="0 0 ${-pi/2}"/>
 	    <geometry>
-		<box size="0.1 0.1 0.1"/>
+		<box size="0.05 0.05 0.05"/>
 	    </geometry>
 	</collision>
