Commit message: configurable laser ranges

File: tuw_gazebo_models/models/sensors/laser/hokuyo_30LX.xacro (robot description, xacro)
@@ -2,5 +2,5 @@
 <robot xmlns:xacro="http://ros.org/wiki/xacro">
   <!-- Front Laser -->
-  <xacro:macro name="laser" params="name frame_names topic_names parent xyz rpy driver:=cpu model_dir:=^">
+  <xacro:macro name="laser" params="name frame_names topic_names parent xyz rpy max_angle:=2.3562 driver:=cpu model_dir:=^">
     <xacro:if value="${driver == 'gpu'}">
       <xacro:property name="sensor_type" value="gpu_ray"/>
@@ -45,10 +45,10 @@
           <scan>
             <horizontal>
-              <!-- The UTM-30LX  has  1080 steps with 0.25 Degree resolution -->
+              <!-- the UTM-30LX has 1080 steps with 0.25 Degree resolution -->
               <resolution>1</resolution>
               <samples>1080</samples>
-              <min_angle>-2.3562</min_angle>
-              <max_angle>2.3562</max_angle>
               <!-- -135 to 135 Degree -->
+              <min_angle>${-max_angle}</min_angle>
+              <max_angle>${max_angle}</max_angle>
             </horizontal>
           </scan>
