Commit message: Changes: -added i2ws platform -various minor fixes

File: tuw_gazebo_models/models/platforms/blue/blue_body/body.xacro (robot description, xacro)
@@ -3,5 +3,5 @@
 <xacro:include filename="chassis.xacro"/>
 <xacro:include filename="piston_steering_wheel.xacro"/>
-<xacro:macro name="BlueBody" params="name parent meshes mesh_collis mesh_visual" >
+<xacro:macro name="BlueBody" params="name parent mesh_collis mesh_visual" >
     <!-- base_link -->
     <link name="${parent}_link"/>

File: tuw_gazebo_models/models/platforms/i2ws/i2ws.xacro (robot description, xacro)
@@ -1,20 +1,20 @@
 <?xml version="1.0"?>
-<robot xmlns:xacro="http://ros.org/wiki/xacro" name="Blue" >
-    <xacro:arg name="model_dir" default="$(find tuw_gazebo_models)/models/platforms/blue"/>
+<robot xmlns:xacro="http://ros.org/wiki/xacro" name="I2ws" >
+    <xacro:arg name="model_dir" default="$(find tuw_gazebo_models)/models/platforms/i2ws"/>
     <!-- Import colors (for Rviz)-->
     <xacro:include filename="$(find tuw_gazebo_models)/models/materials.xacro" />
     <!-- Import robot -->
-    <xacro:property name="model_dir" value="$(arg model_dir)/blue_body"/>
+    <xacro:property name="model_dir" value="$(arg model_dir)/i2ws_body"/>
     <xacro:include filename="${model_dir}/body.xacro"/>
-    <xacro:BlueBody name="body" parent="base" mesh_collis="simplified" mesh_visual="detailed"/><!-- simplified detailed empty-->
+    <xacro:I2wsBody name="body" parent="base" mesh_collis="simplified" mesh_visual="detailed"/><!-- simplified detailed empty-->
     <!-- Import platform plugins -->
     <xacro:property name="model_dir" value="$(arg model_dir)"/>
-    <xacro:include filename="${model_dir}/blue_plugins.xacro" />
-    <xacro:BlueGazeboRosBridgePlugin        />
-    <xacro:BlueGazeboRosFlatControllerPlugin/>
+    <xacro:include filename="${model_dir}/i2ws_plugins.xacro" />
+    <!--xacro:BlueGazeboRosBridgePlugin        /-->
+    <!--xacro:BlueGazeboRosFlatControllerPlugin/-->
     <!-- Laser -->
     <xacro:property name="model_dir" value="$(find tuw_gazebo_models)/models/sensors/laser"/>
     <xacro:include filename="${model_dir}/Sick-LMS100.xacro"/>
-    <xacro:laser name="front_laser" parent="base_link" xyz="0 0.16 0.4" rpy="0 0 ${pi/2}" driver="cpu"/>
+    <xacro:laser name="front_laser" parent="base_link" xyz="0 0.16 0.4" rpy="0 0 ${pi/2}" driver="gpu"/>
     <!-- IMU -->
     <xacro:property name="model_dir" value="$(find tuw_gazebo_models)/models/sensors/imu"/>

File: tuw_gazebo_models/models/platforms/i2ws/i2ws_body/steering_mount.xacro (robot description, xacro)
@@ -2,20 +2,23 @@
 <robot xmlns:xacro="http://ros.org/wiki/xacro">
 <xacro:include filename="$(find tuw_gazebo_models)/models/inertia_tensors.xacro"/>
-<xacro:macro name="BlueWheelMount" params="name parent fb lr mesh_collis:=^|simplified mesh_visual:=^|detailed model_dir:=^">
+<xacro:macro name="I2wsSteeringMount" params="name parent fb lr TransDirX TransDirY RotYaw mesh_collis:=^|simplified mesh_visual:=^|detailed model_dir:=^">
+    <xacro:property name="x_ParrentLink2Piston_Link"  value="0.1750" />
+    <xacro:property name="y_ParrentLink2Piston_Link"  value="0.1744" />
+    <xacro:property name="z_ParrentLink2Piston_Link"  value="0.3400" />
     <xacro:property name="ParrentLink2ThisLink"> <!--parrent link to this joint tf-->
-	<origin xyz="0 0 -0.309"  rpy="0 0 0"/>
+	<origin xyz="${x_ParrentLink2Piston_Link*TransDirX} ${y_ParrentLink2Piston_Link*TransDirY} ${z_ParrentLink2Piston_Link}"  rpy="0 0 ${RotYaw}"/>
     </xacro:property>
     <xacro:property name="ThisLink2Inert"> <!--this link 2 inertial center tf, mass data-->
-	<cylinder_inertial_with_origin radius="0.05" length="0.025" mass="0.197"> <origin xyz="0 0 -0.060" rpy="0 ${-pi/2} 0"/> </cylinder_inertial_with_origin>
+	<cylinder_inertial_with_origin radius="0.04" length="0.1666" mass="0.251"> <origin xyz="0 0 -0.23" rpy="0 0 0"/> </cylinder_inertial_with_origin>
     </xacro:property>
     <xacro:property name="ThisLink2STL"> <!--this link 2 mesh center tf, file-->
-	<origin xyz="0 0 -0.060" rpy="${-pi/2} 0 0"/>
-	<geometry> <mesh filename="file://${model_dir}/meshes/wheel_mount_red.stl"/> </geometry>
-	<material name="orange"/>
+	<origin xyz="0 0 -0.371" rpy="${-pi/2} 0 0"/>
+	<geometry> <mesh filename="file://${model_dir}/meshes/steering_mount_red.stl"/> </geometry>
+	<material name="red"/>
     </xacro:property>
     <xacro:property name="ThisLink2XML"> <!--this link 2 simple mesh center tf, file-->
-	<origin xyz="0 0 -0.060" rpy="${-pi/2} 0 0"/>
-	<geometry> <box size="0.0001 0.0001 0.0001" /> </geometry>
-	<material name="orange"/>
+	<origin xyz="0 0 -0.23" rpy="0 0 0"/>
+	<geometry> <cylinder length="0.1666" radius="0.04"/> </geometry>
+	<material name="red"/>
     </xacro:property>
     <!-- choosing the appropriate collision and visual mesh -->
@@ -27,9 +30,10 @@
     <xacro:if value="${mesh_collis == 'simplified'}"> <xacro:property name="ThisCollis">  <xacro:insert_block name="ThisLink2XML"/> </xacro:property> </xacro:if><!--minimalist mesh-->
     <!-- joint and link definition -->
-    <joint name="${parent}${fb}${lr}2${name}${fb}${lr}_joint" type="revolute"><!--revolute  continuous-->
-	<parent link="${parent}${fb}${lr}_link"/>
+    <joint name="${parent}2${name}${fb}${lr}_joint" type="fixed"><!--prismatic-->
+	<parent link="${parent}_link"/>
 	<child  link="${name}${fb}${lr}_link"/>
-	<axis xyz=" 0 0 1"/>
-	<limit effort="12" velocity="12" lower= "${-M_PI}" upper="${M_PI}" /> <!--velocity="5" -->
+	<axis   xyz="0 0 1"/>
+	<!--limit effort= "10" velocity="0.55" lower= "-0.17" upper="0.0"/-->
+	<!--dynamics damping="0.0" friction="0.0"/-->
 	<xacro:insert_block name="ParrentLink2ThisLink" />
     </joint>
@@ -40,5 +44,5 @@
     </link>
     <gazebo reference="${name}${fb}${lr}_link">
-	<material>Gazebo/Orange</material>
+	<material>Gazebo/Red</material>
 	<selfCollide>false</selfCollide>
     </gazebo>

File: tuw_gazebo_models/models/platforms/i2ws/i2ws_body/wheel_mount.xacro (robot description, xacro)
@@ -2,5 +2,5 @@
 <robot xmlns:xacro="http://ros.org/wiki/xacro">
 <xacro:include filename="$(find tuw_gazebo_models)/models/inertia_tensors.xacro"/>
-<xacro:macro name="BlueWheelMount" params="name parent fb lr mesh_collis:=^|simplified mesh_visual:=^|detailed model_dir:=^">
+<xacro:macro name="I2wsWheelMount" params="name parent fb lr mesh_collis:=^|simplified mesh_visual:=^|detailed model_dir:=^">
     <xacro:property name="ParrentLink2ThisLink"> <!--parrent link to this joint tf-->
 	<origin xyz="0 0 -0.309"  rpy="0 0 0"/>

File: tuw_gazebo_models/models/platforms/i2ws/i2ws_plugins.xacro (robot description, xacro)
@@ -1,5 +1,5 @@
 <?xml version="1.0"?>
 <robot xmlns:xacro="http://ros.org/wiki/xacro">
-<xacro:include filename="blue_plugins_param.xacro"/>
+<xacro:include filename="i2ws_plugins_param.xacro"/>
 <xacro:macro name="BlueGazeboRosBridgePlugin">
     <gazebo>

File: tuw_gazebo_models/models/sensors/laser/Sick-LMS100.xacro (robot description, xacro)
@@ -54,5 +54,5 @@
 		</scan>
 		<range>
-		    <min>0.06</min>
+		    <min>0.11</min>
 		    <max>20.0</max>
 		    <resolution>0.01</resolution>
