Commit message: minor changes

File: tuw_gazebo_models/models/materials.xacro (robot description, xacro)
@@ -12,4 +12,7 @@
   <material name="green">
     <color rgba="0.0 0.8 0.0 1.0"/>
+  </material>
+  <material name="light_grey">
+    <color rgba="0.5 0.5 0.5 1.0"/>
   </material>
   <material name="grey">

File: tuw_gazebo_models/models/platforms/i2ws/i2ws.xacro (robot description, xacro)
@@ -11,14 +11,15 @@
     <xacro:property name="model_dir" value="$(arg model_dir)"/>
     <xacro:include filename="${model_dir}/i2ws_plugins.xacro" />
-    <!--xacro:BlueGazeboRosBridgePlugin        /-->
+    <xacro:BlueGazeboRosBridgePlugin        />
     <!--xacro:BlueGazeboRosFlatControllerPlugin/-->
     <!-- Laser -->
     <xacro:property name="model_dir" value="$(find tuw_gazebo_models)/models/sensors/laser"/>
     <xacro:include filename="${model_dir}/Sick-LMS100.xacro"/>
-    <xacro:laser name="front_laser" parent="base_link" xyz="0 0.16 0.4" rpy="0 0 ${pi/2}" driver="gpu"/>
-    <!-- IMU -->
+    <xacro:laser name="front_laser" parent="base_link" xyz="0.16 0  0.4" rpy="0 0 0" driver="gpu"/>
+    <!-- IMU
     <xacro:property name="model_dir" value="$(find tuw_gazebo_models)/models/sensors/imu"/>
     <xacro:include filename="$(find tuw_gazebo_models)/models/sensors/imu/imu.xacro"/>
-    <xacro:imu_sensor name="imu9dof" parent="base_link" xyz="0.0 0.05 0.262" rpy="0 0 ${pi/2}"/>
+    <xacro:imu_sensor name="imu9dof" parent="base_link" xyz="0.05 0.0 0.262" rpy="0 0 0"/>
+    -->
     <!-- Camera
     <xacro:include filename="$(find blue_gazebo)/xacro/camera/camera.xacro"/>

File: tuw_gazebo_models/models/platforms/i2ws/i2ws_body/body.xacro (robot description, xacro)
@@ -10,6 +10,6 @@
     <xacro:I2wsChassis name="${name}" parent="${parent}"/>
     <!-- Piston-Steering-Wheel modules -->
-    <Steer_WheelMnt_Wheel fb="F" lr="R" parent="${name}" TransDirX=  "1" TransDirY=  "1" RotYaw="0"/>
-    <Steer_WheelMnt_Wheel fb="F" lr="L" parent="${name}" TransDirX= "-1" TransDirY=  "1" RotYaw="0"/>
+    <Steer_WheelMnt_Wheel fb="F" lr="R" parent="${name}" TransDirX=  "1" TransDirY= "-1" RotYaw="0"/>
+    <Steer_WheelMnt_Wheel fb="B" lr="L" parent="${name}" TransDirX= "-1" TransDirY=  "1" RotYaw="0"/>
     <xacro:property name="swivel_contact_data">
       <mu1 value="0.7"/>
@@ -19,6 +19,6 @@
       <minDepth value="0.002"/>
     </xacro:property>
-    <Swivel fb="B" lr="R" parent="${name}" TransDirX=  "1" TransDirY= "-1" RotYaw="0"> <container> <xacro:insert_block name="swivel_contact_data"/> </container> </Swivel>
-    <Swivel fb="B" lr="L" parent="${name}" TransDirX= "-1" TransDirY= "-1" RotYaw="0"> <container> <xacro:insert_block name="swivel_contact_data"/> </container> </Swivel>
+    <Swivel fb="F" lr="L" parent="${name}" TransDirX=  "1" TransDirY=  "1" RotYaw="0"> <container> <xacro:insert_block name="swivel_contact_data"/> </container> </Swivel>
+    <Swivel fb="B" lr="R" parent="${name}" TransDirX= "-1" TransDirY= "-1" RotYaw="0"> <container> <xacro:insert_block name="swivel_contact_data"/> </container> </Swivel>
 </xacro:macro>
 </robot>

File: tuw_gazebo_models/models/platforms/i2ws/i2ws_body/chassis.xacro (robot description, xacro)
@@ -4,5 +4,5 @@
 <xacro:macro name="I2wsChassis" params="name parent mesh_collis:=^|simplified mesh_visual:=^|detailed model_dir:=^" >
     <xacro:property name="ParrentLink2ThisLink"> <!--parrent link to this joint tf-->
-	<origin xyz="0 0 0.07" rpy="0 0 0"/>
+	<origin xyz="0 0 0.07" rpy="0 0 ${-pi/2}"/>
     </xacro:property>
     <xacro:property name="ThisLink2Inert"> <!--this link 2 inertial center tf, mass data-->
@@ -12,5 +12,5 @@
 	<origin xyz="0 0 0.20" rpy="0 0 0"/>
 	<geometry> <box size="0.5 0.5 0.4" /> </geometry>
-	<material name="grey"/>
+	<material name="light_grey"/>
     </xacro:property>
     <!-- choosing the appropriate collision and visual mesh -->

File: tuw_gazebo_models/models/platforms/i2ws/i2ws_body/swivel.xacro (robot description, xacro)
@@ -5,5 +5,5 @@
   <xacro:property name="x_ParrentLink2Piston_Link"  value= "0.1750" />
   <xacro:property name="y_ParrentLink2Piston_Link"  value= "0.1744" />
-  <xacro:property name="z_ParrentLink2Piston_Link"  value="-0.0270" />
+  <xacro:property name="z_ParrentLink2Piston_Link"  value="-0.0230" />
   <xacro:property name="ParrentLink2ThisLink"> <!--parrent link to this joint tf-->
       <origin xyz="${x_ParrentLink2Piston_Link*TransDirX} ${y_ParrentLink2Piston_Link*TransDirY} ${z_ParrentLink2Piston_Link}"  rpy="0 0 ${RotYaw}"/>

File: tuw_gazebo_models/models/platforms/i2ws/i2ws_plugins.xacro (robot description, xacro)
@@ -4,5 +4,5 @@
 <xacro:macro name="BlueGazeboRosBridgePlugin">
     <gazebo>
-        <plugin name="tuw_gazebo_ros_i4ws_bridge_plugin" filename="libtuw_gazebo_ros_i4ws_bridge_plugin.so">
+        <plugin name="tuw_gazebo_ros_i2ws_bridge_plugin" filename="libtuw_gazebo_ros_i2ws_bridge_plugin.so">
             <xacro:insert_block name="BlueGazeboPluginsData" />
         </plugin>
@@ -11,5 +11,5 @@
 <xacro:macro name="BlueGazeboRosFlatControllerPlugin">
     <gazebo>
-	<plugin name="tuw_gazebo_ros_iws_controller_plugin" filename="libtuw_gazebo_ros_iws_controller_plugin.so">
+	<plugin name="tuw_gazebo_ros_i2ws_controller_plugin" filename="libtuw_gazebo_ros_i2ws_controller_plugin.so">
 	    <xacro:insert_block name="BlueGazeboPluginsData" />
 	</plugin>
@@ -20,7 +20,9 @@
 	<plugin name="joint_state_publisher" filename="libgazebo_ros_joint_state_publisher.so">
 	    <robotNamespace></robotNamespace>
-	    <jointName>  pistonFR2steermntFR_joint,   pistonFL2steermntFL_joint,   pistonBR2steermntBR_joint,   pistonBL2steermntBL_joint,
-		       steermntFR2wheelmntFR_joint, steermntFL2wheelmntFL_joint, steermntBR2wheelmntBR_joint, steermntBL2wheelmntBL_joint,
-			  wheelmntFR2wheelFR_joint,    wheelmntFL2wheelFL_joint,    wheelmntBR2wheelBR_joint,    wheelmntBL2wheelBL_joint  </jointName>
+	    <jointName>  pistonFR2steermntFR_joint,   pistonBL2steermntBL_joint,
+		       steermntFR2wheelmntFR_joint, steermntBL2wheelmntBL_joint,
+			  wheelmntFR2wheelFR_joint,    wheelmntBL2wheelBL_joint,
+			  chassis_swivelFL_joint, swivelFL_wheel_joint,
+			  chassis_swivelBR_joint, swivelBR_wheel_joint</jointName>
 	    <updateRate>10.0</updateRate>
 	    <alwaysOn>true</alwaysOn>

File: tuw_gazebo_models/models/platforms/i2ws/i2ws_plugins_param.xacro (robot description, xacro)
@@ -11,6 +11,4 @@
 	<robotBaseFrame>base_link</robotBaseFrame>
 	<tr_piston_joint>pistonFR2steermntFR_joint</tr_piston_joint>
-	<tl_piston_joint>pistonFL2steermntFL_joint</tl_piston_joint>
-	<br_piston_joint>pistonBR2steermntBR_joint</br_piston_joint>
 	<bl_piston_joint>pistonBL2steermntBL_joint</bl_piston_joint>
 	<piston_hi_stop>       0.0</piston_hi_stop>
@@ -21,6 +19,4 @@
 	<piston_friction>      0.0</piston_friction>
 	<tr_steering_joint>steermntFR2wheelmntFR_joint</tr_steering_joint>
-	<tl_steering_joint>steermntFL2wheelmntFL_joint</tl_steering_joint>
-	<br_steering_joint>steermntBR2wheelmntBR_joint</br_steering_joint>
 	<bl_steering_joint>steermntBL2wheelmntBL_joint</bl_steering_joint>
 	<steering_hi_stop>     2.70526034</steering_hi_stop>    <!-- rad -->
@@ -31,9 +27,7 @@
 	<steering_friction>           0.0</steering_friction>   <!--Nm   -->
 	<tr_wheel_joint>wheelmntFR2wheelFR_joint</tr_wheel_joint>
-	<tl_wheel_joint>wheelmntFL2wheelFL_joint</tl_wheel_joint>
-	<br_wheel_joint>wheelmntBR2wheelBR_joint</br_wheel_joint>
 	<bl_wheel_joint>wheelmntBL2wheelBL_joint</bl_wheel_joint>
 	<wheel_max_torque>           10.0</wheel_max_torque> <!-- Nm  -->
-	<wheel_max_vel>             100.0</wheel_max_vel>    <!--rad/s-->
+	<wheel_max_vel>              10.0</wheel_max_vel>    <!--rad/s-->
 	<wheel_damping>               0.1</wheel_damping>    <!--Nms/rad-->
 	<wheel_friction>              0.0</wheel_friction>   <!--Nm   -->
@@ -44,5 +38,5 @@
 	<odometryTopic>odom</odometryTopic>
 	<odometryFrame>odom</odometryFrame>
-	<useForceControl>true</useForceControl>
+	<useForceControl>false</useForceControl>
 </xacro:property>
 </robot>

File: tuw_gazebo_models/models/platforms/pioneer3dx/pioneer3dx.xacro (robot description, xacro)
@@ -17,12 +17,11 @@
   <xacro:include filename="${model_dir}/hokuyo.xacro"/>
   <xacro:laser name="front_laser" parent="chassis" xyz="0.16 0 0.125" rpy="0 0 0" driver="cpu"/>
-  <!-- Laser -->
+  <!-- IMU -->
   <xacro:property name="model_dir" value="$(find tuw_gazebo_models)/models/sensors/imu"/>
   <xacro:include filename="$(find tuw_gazebo_models)/models/sensors/imu/imu.xacro"/>
   <xacro:imu_sensor name="imu9dof" parent="chassis" xyz="0.05 0.0 0.262" rpy="0 0 0"/>
-  <!-- Camera
+  <!-- Camera -->
   <xacro:property name="model_dir" value="$(find tuw_gazebo_models)/models/sensors/camera"/>
   <xacro:include filename="${model_dir}/camera.xacro"/>
-  <xacro:cam name="front_camera" parent="chassis" xyz="0 0 0.5" rpy="0 0 0" />
-  -->
+  <xacro:cam name="front_camera" parent="chassis" xyz="0 0 0.5" rpy="${-pi/2}  0 ${-pi/2}" />
 </robot>

File: tuw_gazebo_models/models/sensors/camera/camera.xacro (robot description, xacro)
@@ -17,5 +17,5 @@
     </inertial>
     <visual>
-      <origin xyz="0 0 0" rpy="0 1.57 0"/>
+      <origin xyz="0 0 0" rpy="0 0 0"/>
       <geometry>
         <cylinder radius="0.03" length="0.1"/>
@@ -24,5 +24,5 @@
     </visual>
     <collision>
-      <origin xyz="0 0 0" rpy="0 1.57 0"/>
+      <origin xyz="0 0 0" rpy="0 0 0"/>
       <geometry>
         <cylinder radius="0.03" length="0.1"/>
@@ -37,4 +37,5 @@
       <update_rate>30.0</update_rate>
       <camera name="head">
+        <pose>0 0 0 0 -${pi/2}  ${pi/2}</pose>
         <horizontal_fov>1.3962634</horizontal_fov>
         <image>
