Commit message: chassis and inertia ready

File: tuw_gazebo_models/models/inertia_tensors.xacro (robot description, xacro)
@@ -44,8 +44,8 @@
     </inertial>
   </xacro:macro>
-  <xacro:macro name="cylinder_inertial_with_origin" params="radius length mass *origin">
+  <xacro:macro name="cylinder_inertial_with_origin" params="radius length mass xyz rpy">
     <inertial>
       <mass value="${mass}" />
-      <xacro:insert_block name="origin" />
+      <origin xyz="${xyz}" rpy="${rpy}" />
       <inertia ixx="${0.0833333 * mass * (3 * radius * radius + length * length)}" ixy="0.0" ixz="0.0"
         iyy="${0.0833333 * mass * (3 * radius * radius + length * length)}" iyz="0.0"
@@ -53,8 +53,8 @@
     </inertial>
   </xacro:macro>
-  <xacro:macro name="box_inertial_with_origin" params="x y z mass *origin">
+  <xacro:macro name="box_inertial_with_origin" params="x y z mass xyz">
     <inertial>
       <mass value="${mass}" />
-      <xacro:insert_block name="origin" />
+      <origin xyz="${xyz}" />
       <inertia ixx="${0.0833333 * mass * (y*y + z*z)}" ixy="0.0" ixz="0.0"
         iyy="${0.0833333 * mass * (x*x + z*z)}" iyz="0.0"

File: tuw_gazebo_models/models/pioneer3dx/body/chassis.xacro (robot description, xacro)
@@ -2,4 +2,6 @@
 <robot xmlns:xacro="http://ros.org/wiki/xacro">
   <xacro:property name="M_PI" value="3.1415926535897931" />
+  <xacro:property name="chassis_width" value="0.27" />
+  <xacro:property name="chassis_collision_ellipse_height" value="0.17" />
   <xacro:macro name="pioneer_chassis" params="name parent xyz rpy models_dir:=^">
   <!-- Chassis -->
@@ -10,6 +12,7 @@
   </joint>
   <link name="${name}">
+    <xacro:box_inertial_with_origin x="${chassis_width}" y="${chassis_width}"  z="${chassis_collision_ellipse_height}" mass="5.67" xyz="${-chassis_width/4} 0 ${chassis_collision_ellipse_height/2}"/>
     <visual>
-      <origin xyz="-0.045 0 0.085" rpy="0 0 0"/>
+      <origin xyz="-0.045 0 ${chassis_collision_ellipse_height/2}" rpy="0 0 0"/>
       <geometry>
         <mesh filename="file://${models_dir}/pioneer3dx/body/meshes/chassis.dae"/>
@@ -20,16 +23,15 @@
     </visual>
     <collision>
-      <origin xyz="0.01 0 0.09" rpy="0 0 0"/>
+      <origin xyz="0 0 ${chassis_collision_ellipse_height/2}" rpy="0 0 0"/>
       <geometry>
-          <cylinder radius="0.17" length="0.17"/>
+          <cylinder radius="${chassis_width/2}" length="${chassis_collision_ellipse_height}"/>
       </geometry>
-      <!--origin xyz="-0.045 0 0.148" rpy="0 0 0"/>
+    </collision>
+    <collision>
+      <origin xyz="-${chassis_width/2} 0 ${chassis_collision_ellipse_height/2}" rpy="0 0 0"/>
       <geometry>
-        <mesh filename="file://${model_dir}/meshes/body/chassis.dae"/>
-      </geometry-->
+          <cylinder radius="${chassis_width/2}" length="${chassis_collision_ellipse_height}"/>
+      </geometry>
     </collision>
-    <box_inertial_with_origin x="0.35" y="0.25"  z="0.17" mass="9.0">
-        <origin xyz="-0.04 0 0.15" rpy="0 0 0"/>
-    </box_inertial_with_origin>
   </link>
   <gazebo reference="${name}">
@@ -52,13 +54,4 @@
       </material>
     </visual>
-    <collision>
-    <origin xyz="${-0.045-0.05} 0 ${-0.235+0.15}" rpy="0 0 0"/>
-    <geometry><cylinder radius="0.17" length="0.17"/> </geometry>
-    <!--origin xyz="0.0 0 0.0" rpy="0 0 0"/>
-      <geometry>
-        <mesh filename="file://${models_dir}/pioneer3dx/body/meshes/top.dae"/>
-      </geometry-->
-    </collision>
-    <box_inertial_with_origin x="0.45" y="0.35"  z="0.001" mass="1.0"> <origin xyz="0.00 0 0.00" rpy="0 0 0"/> </box_inertial_with_origin>
   </link>
   <gazebo reference="top">
