Commit message: better i2ws simulation

File: tuw_gazebo_models/models/platforms/i2ws/i2ws_body/swivel.xacro (robot description, xacro)
@@ -5,5 +5,5 @@
   <xacro:property name="x_ParrentLink2Piston_Link"  value= "0.1750" />
   <xacro:property name="y_ParrentLink2Piston_Link"  value= "0.1744" />
-  <xacro:property name="z_ParrentLink2Piston_Link"  value="-0.0230" />
+  <xacro:property name="z_ParrentLink2Piston_Link"  value="-0.0235" />
   <xacro:property name="ParrentLink2ThisLink"> <!--parrent link to this joint tf-->
       <origin xyz="${x_ParrentLink2Piston_Link*TransDirX} ${y_ParrentLink2Piston_Link*TransDirY} ${z_ParrentLink2Piston_Link}"  rpy="0 0 ${RotYaw}"/>

File: tuw_gazebo_models/models/platforms/i2ws/i2ws_body/wheel.xacro (robot description, xacro)
@@ -39,6 +39,6 @@
 	<material>Gazebo/White</material>
 	<selfCollide>false</selfCollide>
-	<mu1 value="5.9"/>
-	<mu2 value="5.9"/>
+	<mu1 value="0.7"/>
+	<mu2 value="0.7"/>
 	<!--fdir1>0 0 1</fdir1-->
 	<minDepth value="0.002"/>

File: tuw_gazebo_models/models/platforms/i2ws/i2ws_plugins_param.xacro (robot description, xacro)
@@ -13,10 +13,10 @@
 	<steering_max_torque>        10.0</steering_max_torque> <!-- Nm  -->
 	<steering_max_vel>            5.0</steering_max_vel>    <!--rad/s-->
-	<steering_damping>            0.1</steering_damping>    <!--Nms/rad-->
+	<steering_damping>            0.7</steering_damping>    <!--Nms/rad-->
 	<steering_friction>           0.0</steering_friction>   <!--Nm   -->
 	<revolute_joints_names>wheelmntFL2wheelFL_joint, wheelmntBR2wheelBR_joint</revolute_joints_names>
 	<revolute_max_torque>        10.0</revolute_max_torque> <!-- Nm  -->
 	<revolute_max_vel>           50.0</revolute_max_vel>    <!--rad/s-->
-	<revolute_damping>            0.1</revolute_damping>    <!--Nms/rad-->
+	<revolute_damping>            0.7</revolute_damping>    <!--Nms/rad-->
 	<revolute_friction>           0.0</revolute_friction>   <!--Nm   -->
 	<steering_measures_type>measured_position</steering_measures_type>
