Commit message: gazebo renders swivel properly

File: tuw_gazebo_models/models/platforms/pioneer3dx/pioneer3dx_body/body.xacro (robot description, xacro)
@@ -17,7 +17,7 @@
     <xacro:pioneer_battery_block name="battery0" parent="${name}" x="-0.14" y="0.00"  z="0.13" mass="2.5" />
     <!-- Wheels -->
+    <xacro:pioneer_swivel parent="${name}"  xyz="-0.185 0 0.055" rpy="0 0 0"/>
     <xacro:pioneer_wheel side="right" parent="${name}"  xyz="0  0.15 0.09" rpy="0 0 0" radius="0.09"/>
     <xacro:pioneer_wheel side="left"  parent="${name}"  xyz="0 -0.15 0.09" rpy="0 0 0" radius="0.09"/>
-    <xacro:pioneer_swivel parent="${name}"  xyz="-0.185 0 0.055" rpy="0 0 0"/>
   </xacro:macro>
 </robot>

File: tuw_gazebo_models/models/platforms/pioneer3dx/pioneer3dx_body/chassis.xacro (robot description, xacro)
@@ -10,7 +10,7 @@
   </joint>
   <link name="${name}">
-    <visual name="chassis_visual">
+    <visual>
       <origin xyz="-0.045 0 0.148" rpy="0 0 0"/>
-      <geometry name="pioneer_geom">
+      <geometry>
 		  <mesh filename="file://${model_dir}/meshes/chassis.dae"/>
       </geometry>
@@ -39,5 +39,5 @@
     <visual>
       <origin xyz="0 0 0" rpy="0 0 0"/>
-      <geometry name="top_geom">
+      <geometry>
         <mesh filename="file://${model_dir}/meshes/top.dae"/>
       </geometry>

File: tuw_gazebo_models/models/platforms/pioneer3dx/pioneer3dx_body/sonar.xacro (robot description, xacro)
@@ -15,7 +15,7 @@
       <inertia ixx="1" ixy="0" ixz="0" iyy="1" iyz="0" izz="1"/>
     </inertial>
-    <visual name="front_sonar_vis">
+    <visual>
       <origin xyz="0 0 0" rpy="0 0 0"/>
-      <geometry name="pioneer_geom">
+      <geometry>
         <mesh filename="file://${model_dir}/meshes/back_sonar.dae"/>
       </geometry>

File: tuw_gazebo_models/models/platforms/pioneer3dx/pioneer3dx_body/swivel.xacro (robot description, xacro)
@@ -19,7 +19,7 @@
       <inertia ixx="0.01" ixy="0" ixz="0" iyy="0.01" iyz="0" izz="0.01"/>
     </inertial>
-    <visual name="base_visual">
+    <visual>
       <origin xyz="0 0 0" rpy="0 0 0"/>
-      <geometry name="pioneer_geom">
+      <geometry>
         <mesh filename="file://${model_dir}/meshes/swivel.stl"/>
       </geometry>
@@ -54,7 +54,7 @@
       <inertia ixx="0.012411765597" ixy="-0.000711733678" ixz="0.00050272983" iyy="0.015218160428" iyz="-0.000004273467" izz="0.011763977943"/>
     </inertial>
-    <visual name="base_visual">
+    <visual>
       <origin xyz="0 0 0" rpy="0 0 0"/>
-      <geometry name="pioneer_geom">
+      <geometry>
         <mesh filename="file://${model_dir}/meshes/center_wheel.stl"/>
       </geometry>
@@ -86,7 +86,7 @@
       <inertia ixx="0.012411765597" ixy="-0.000711733678" ixz="0.00050272983" iyy="0.015218160428" iyz="-0.000004273467" izz="0.011763977943"/>
     </inertial>
-    <visual name="hubcap_visual">
+    <visual>
       <origin xyz="0 0 0" rpy="0 0 0"/>
-      <geometry name="pioneer_geom">
+      <geometry>
         <mesh filename="file://${model_dir}/meshes/center_hubcap.stl"/>
       </geometry>

File: tuw_gazebo_models/models/platforms/pioneer3dx/pioneer3dx_body/wheel.xacro (robot description, xacro)
@@ -17,7 +17,7 @@
       <inertia ixx="0.012411765597" ixy="0" ixz="0" iyy="0.015218160428" iyz="0" izz="0.011763977943"/>
     </inertial>
-    <visual name="base_visual">
+    <visual>
       <origin xyz="0 0 0" rpy="0 0 0"/>
-      <geometry name="pioneer_geom">
+      <geometry>
         <mesh filename="file://${model_dir}/meshes/hubcap.dae"/>
       </geometry>
@@ -49,7 +49,7 @@
       <inertia ixx="0.012411765597" ixy="0" ixz="0" iyy="0.015218160428" iyz="0" izz="0.011763977943"/>
     </inertial>
-    <visual name="wheel_visual">
+    <visual>
       <origin xyz="0 0 0" rpy="0 0 0"/>
-      <geometry name="pioneer_geom">
+      <geometry>
         <mesh filename="file://${model_dir}/meshes/wheel.dae"/>
       </geometry>

Commit message: diffdrive not drifting when stopped anymoregit status -s :)

File: tuw_gazebo_models/models/platforms/pioneer3dx/pioneer3dx_body/body.xacro (robot description, xacro)
@@ -25,6 +25,6 @@
 	<mu2 value="0.7"/>
 	<minDepth value="0.002"/>
-	<kp value="1000000.0"/>
-	<kd value="10.0"/>
+	<!--kp value="1000000.0"/-->
+	<!--kd value="10.0"/-->
     </xacro:property>
     <xacro:pioneer_swivel             parent="${parent}"  xyz="-0.185 0    0.0535" rpy="0 0 0">               <container> <xacro:insert_block name="contact_data"/> </container> </xacro:pioneer_swivel>

File: tuw_gazebo_models/models/platforms/pioneer3dx/pioneer3dx_body/sonar.xacro (robot description, xacro)
@@ -10,5 +10,5 @@
   </joint>
   <link name="${name}">
-    <xacro:box_inertial x="0.001" y="0.001"  z="0.001" mass="0.001" />
+    <xacro:box_inertial x="0.01" y="0.01"  z="0.01" mass="0.01" />
     <visual>
       <origin xyz="0 0 0" rpy="0 0 0"/>

File: tuw_gazebo_models/models/platforms/pioneer3dx/pioneer3dx_body/swivel.xacro (robot description, xacro)
@@ -8,5 +8,5 @@
     <axis xyz="0 0 1"/>
     <anchor xyz="0 0 0"/>
-    <limit effort="100" velocity="100" k_velocity="0"/>
+    <!--limit effort="100" velocity="100" k_velocity="0"/-->
     <joint_properties damping="0.1" friction="0.0"/>
     <parent link="${parent}"/>
@@ -44,5 +44,5 @@
     <axis xyz="0 1 0"/>
     <anchor xyz="0 0 0"/>
-    <limit effort="100" velocity="100" k_velocity="0"/>
+    <!--limit effort="100" velocity="100" k_velocity="0"/-->
     <joint_properties damping="0.0" friction="0.0"/>
     <parent link="swivel"/>
