Commit message: mesh viz bug in rviz

File: tuw_gazebo_models/models/platforms/pioneer3dx/pioneer3dx.xacro (robot description, xacro)
@@ -1,5 +1,5 @@
 <?xml version="1.0"?>
 <robot xmlns:xacro="http://www.ros.org/wiki/xacro" name="pioneer3dx" >
-   <xacro:arg name="model_dir" default="$(find tuw_gazebo_models)/models/platforms/pioneer3dx"/>
+  <xacro:arg name="model_dir" default="$(find tuw_gazebo_models)/models/platforms/pioneer3dx"/>
   <!-- Import Rviz colors -->
   <xacro:include filename="$(find tuw_gazebo_models)/models/materials.xacro" />

File: tuw_gazebo_models/models/platforms/pioneer3dx/pioneer3dx_body/chassis.xacro (robot description, xacro)
@@ -13,5 +13,5 @@
       <origin xyz="-0.045 0 0.148" rpy="0 0 0"/>
       <geometry name="pioneer_geom">
-		  <mesh filename="${model_dir}/meshes/chassis.dae"/>
+		  <mesh filename="file://${model_dir}/meshes/chassis.dae"/>
       </geometry>
       <material name="ChassisRed">
@@ -22,5 +22,5 @@
       <origin xyz="-0.045 0 0.148" rpy="0 0 0"/>
       <geometry>
-		  <mesh filename="${model_dir}/meshes/chassis.dae"/>
+		  <mesh filename="file://${model_dir}/meshes/chassis.dae"/>
       </geometry>
     </collision>
@@ -40,5 +40,5 @@
       <origin xyz="0 0 0" rpy="0 0 0"/>
       <geometry name="top_geom">
-        <mesh filename="${model_dir}/meshes/top.dae"/>
+        <mesh filename="file://${model_dir}/meshes/top.dae"/>
       </geometry>
       <material name="TopBlack">
@@ -49,5 +49,5 @@
     <origin xyz="0.0 0 0.0" rpy="0 0 0"/>
       <geometry>
-        <mesh filename="${model_dir}/meshes/top.dae"/>
+        <mesh filename="file://${model_dir}/meshes/top.dae"/>
       </geometry>
     </collision>

File: tuw_gazebo_models/models/platforms/pioneer3dx/pioneer3dx_body/sonar.xacro (robot description, xacro)
@@ -18,5 +18,5 @@
       <origin xyz="0 0 0" rpy="0 0 0"/>
       <geometry name="pioneer_geom">
-        <mesh filename="${model_dir}/meshes/back_sonar.dae"/>
+        <mesh filename="file://${model_dir}/meshes/back_sonar.dae"/>
       </geometry>
       <material name="SonarYellow">

File: tuw_gazebo_models/models/platforms/pioneer3dx/pioneer3dx_body/swivel.xacro (robot description, xacro)
@@ -22,5 +22,5 @@
       <origin xyz="0 0 0" rpy="0 0 0"/>
       <geometry name="pioneer_geom">
-        <mesh filename="${model_dir}/meshes/swivel.stl"/>
+        <mesh filename="file://${model_dir}/meshes/swivel.stl"/>
       </geometry>
       <material name="swivel">
@@ -57,5 +57,5 @@
       <origin xyz="0 0 0" rpy="0 0 0"/>
       <geometry name="pioneer_geom">
-        <mesh filename="${model_dir}/meshes/center_wheel.stl"/>
+        <mesh filename="file://${model_dir}/meshes/center_wheel.stl"/>
       </geometry>
       <material name="WheelBlack">
@@ -89,5 +89,5 @@
       <origin xyz="0 0 0" rpy="0 0 0"/>
       <geometry name="pioneer_geom">
-        <mesh filename="${model_dir}/meshes/center_hubcap.stl"/>
+        <mesh filename="file://${model_dir}/meshes/center_hubcap.stl"/>
       </geometry>
       <material name="swivel">

File: tuw_gazebo_models/models/platforms/pioneer3dx/pioneer3dx_body/wheel.xacro (robot description, xacro)
@@ -20,5 +20,5 @@
       <origin xyz="0 0 0" rpy="0 0 0"/>
       <geometry name="pioneer_geom">
-        <mesh filename="${model_dir}/meshes/hubcap.dae"/>
+        <mesh filename="file://${model_dir}/meshes/hubcap.dae"/>
       </geometry>
       <material name="HubcapYellow">
@@ -52,5 +52,5 @@
       <origin xyz="0 0 0" rpy="0 0 0"/>
       <geometry name="pioneer_geom">
-        <mesh filename="${model_dir}/meshes/wheel.dae"/>
+        <mesh filename="file://${model_dir}/meshes/wheel.dae"/>
       </geometry>
       <material name="WheelBlack">

File: tuw_gazebo_models/models/sensors/laser/RPLidar.xacro (robot description, xacro)
@@ -21,5 +21,5 @@
         <origin xyz="0 0 0" rpy="0 0 0"/>
         <geometry>
-          <mesh filename="${model_dir}/meshes/RPLidar.dae"/>
+          <mesh filename="file://${model_dir}/meshes/RPLidar.dae"/>
         </geometry>
       </visual>

File: tuw_gazebo_models/models/sensors/laser/Sick-LMS100.xacro (robot description, xacro)
@@ -23,5 +23,5 @@
 	<visual>
 	  <geometry>
-		<mesh filename="${model_dir}/meshes/Sick-LMS100.dae"/>
+		<mesh filename="file://${model_dir}/meshes/Sick-LMS100.dae"/>
 	  </geometry>
 	  <material name="SickBlue"/>

File: tuw_gazebo_models/models/sensors/laser/hokuyo.xacro (robot description, xacro)
@@ -21,5 +21,5 @@
         <origin xyz="0 0 -0.025" rpy="0 0 0"/>
         <geometry>
-          <mesh filename="${model_dir}/meshes/hokuyo.dae"/>
+          <mesh filename="file://${model_dir}/meshes/hokuyo.dae"/>
         </geometry>
       </visual>

Commit message: changes: -added redesigned plugins for laser and gpu_laser. Notable modifications:        - cleaned up class design        - now plugin does not subscribe to the gazebo laser topic but to the gazebo sensor directly        - proper destruction of everything        - NOTE: the Gazebo GpuRay is buggy and thus does not work anymore after deleting the model. This is NOT a plugin problem but an internal Gazebo GpuRay problem (TESTED!) -resaved meshes that were not visualisable in Rviz (if saved in collada format from Sketchup, they become invisible. I opened and saved them in Blender) -no more errors on p3dx load in Gazebo (reason was some links not having a collision/visual element -- now set to something super small) -gazebo has visualization errors if geometry/visual xml properties are named (=> now not named anymore)

File: tuw_gazebo_models/models/platforms/pioneer3dx/pioneer3dx.xacro (robot description, xacro)
@@ -17,4 +17,8 @@
   <xacro:include filename="${model_dir}/hokuyo.xacro"/>
   <xacro:laser name="front_laser" parent="chassis" xyz="0.16 0 0.125" rpy="0 0 0" driver="cpu"/>
+  <!-- Laser -->
+  <!--xacro:property name="model_dir" value="$(find tuw_gazebo_models)/models/sensors/imu"/-->
+  <!--xacro:include filename="$(find tuw_gazebo_models)/models/sensors/imu/imu.xacro"/>
+  <xacro:imu_sensor name="imu" parent="chassis" xyz="0.05 0.0 0.262" rpy="0 0 0"/-->
   <!-- Camera
   <xacro:property name="model_dir" value="$(find tuw_gazebo_models)/models/sensors/camera"/>

File: tuw_gazebo_models/models/platforms/pioneer3dx/pioneer3dx_body/sonar.xacro (robot description, xacro)
@@ -27,5 +27,5 @@
       <origin xyz="0 0 0" rpy="0 0 0"/>
       <geometry>
-        <box size="0 0 0"/>
+        <box size="0.001 0.001 0.001"/>
       </geometry>
     </collision>

File: tuw_gazebo_models/models/platforms/pioneer3dx/pioneer3dx_body/swivel.xacro (robot description, xacro)
@@ -31,5 +31,5 @@
       <origin xyz="0 0 0" rpy="0 0 0"/>
       <geometry>
-        <box size="0 0 0"/>
+        <box size="0.001 0.001 0.001"/>
       </geometry>
     </collision>
@@ -98,5 +98,5 @@
       <origin xyz="0 0 0" rpy="0 0 0"/>
       <geometry>
-        <box size="0 0 0"/>
+        <box size="0.001 0.001 0.001"/>
       </geometry>
     </collision>

File: tuw_gazebo_models/models/platforms/pioneer3dx/pioneer3dx_body/wheel.xacro (robot description, xacro)
@@ -29,5 +29,5 @@
       <origin xyz="0 0 0" rpy="0 0 0"/>
       <geometry>
-        <box size="0 0 0"/>
+        <box size="0.001 0.001 0.001"/>
       </geometry>
     </collision>
@@ -68,4 +68,6 @@
   <gazebo reference="${side}_wheel">
     <material value="Gazebo/Black"/>
+    <mu1 value="0.5"/>
+    <mu2 value="0.5"/>
   </gazebo>
   </xacro:macro>

File: tuw_gazebo_models/models/platforms/pioneer3dx/pioneer3dx_plugins.xacro (robot description, xacro)
@@ -16,5 +16,6 @@
             <rosDebugLevel>Debug</rosDebugLevel>
             <robotNamespace></robotNamespace>
-            <publishWheelTF>false</publishWheelTF>
+            <publishTf>true</publishTf>
+	    <publishWheelTF>true</publishWheelTF>
             <publishWheelJointState>true</publishWheelJointState>
             <alwaysOn>true</alwaysOn>

File: tuw_gazebo_models/models/sensors/laser/RPLidar.xacro (robot description, xacro)
@@ -2,7 +2,7 @@
 <robot xmlns:xacro="http://www.ros.org/wiki/xacro">
 <!-- Front Laser -->
-<xacro:macro name="laser" params="name parent xyz rpy driver:=gpu model_dir:=^" >
-  <xacro:if     value="${driver == 'gpu'}"> <xacro:property name="driver_name" value="_gpu"/></xacro:if>
-  <xacro:unless value="${driver == 'gpu'}"> <xacro:property name="driver_name" value=""    /></xacro:unless>
+<xacro:macro name="laser" params="name parent xyz rpy driver:=cpu model_dir:=^" >
+  <xacro:if     value="${driver == 'gpu'}"> <xacro:property name="sensor_type" value="gpu_ray"/> <xacro:property name="driver_type" value="libtuw_gazebo_ros_gpu_laser.so"/> </xacro:if>
+  <xacro:unless value="${driver == 'gpu'}"> <xacro:property name="sensor_type" value="ray"    /> <xacro:property name="driver_type" value="libtuw_gazebo_ros_laser.so"    /> </xacro:unless>
   <joint name="${parent}_${name}_joint" type="fixed">
       <axis xyz="0 0 1" />
@@ -18,12 +18,12 @@
         </geometry>
       </collision>
-      <visual name="RPLidar_visual">
+      <visual>
         <origin xyz="0 0 0" rpy="0 0 0"/>
         <geometry>
-          <mesh filename="file://${model_dir}/meshes/RPLidar.dae"/>
+          <mesh filename="file://${model_dir}/meshes/RPLidar_.dae"/>
         </geometry>
       </visual>
       <inertial>
-        <mass value="1e-5" />
+        <mass value="1e-2" />
         <origin xyz="0 0 -0.025" rpy="0 0 0"/>
         <inertia ixx="1e-6" ixy="0" ixz="0" iyy="1e-6" iyz="0" izz="1e-6" />
@@ -31,33 +31,34 @@
     </link>
     <gazebo reference="${name}">
-        <sensor name="laser" type="${driver_name}ray">
-		  <pose>0 0 0 0 0 0</pose>
-		  <update_rate>5.5</update_rate>
-          <visualize>true</visualize>
-          <always_on>1</always_on>
-          <ray>
-            <scan>
-              <horizontal>
-                <!-- The RPLidar has 360 steps with 1 Degree resolution -->
-                <resolution>1</resolution>
-                <samples>360</samples> <min_angle>-3.141592</min_angle> <max_angle>3.124139361</max_angle> <!-- -180 to 180 Degree -->
-              </horizontal>
-            </scan>
-            <range>
-              <min>0.2</min>
-              <max>6</max>
-              <resolution>0.02</resolution>
-            </range>
-			<noise>
-				<type>gaussian</type>
-				<mean>0.0</mean>
-				<stddev>0.03</stddev>
-			</noise>
-          </ray>
-          <plugin name="gazebo_ros_laser_RPLidar_driver" filename="libgazebo_ros_${driver_name}laser.so" >
-			<robotNamespace></robotNamespace>
-			<topicName>${name}/scan</topicName>
-			<frameName>${name}</frameName>
-          </plugin>
+        <sensor name="laser" type="${sensor_type}">
+	    <pose>0 0 0 0 0 0</pose>
+	    <update_rate>5.5</update_rate>
+	    <visualize>true</visualize>
+	    <always_on>1</always_on>
+	    <ray>
+		<scan>
+		    <horizontal>
+			<!-- The RPLidar has 360 steps with 1 Degree resolution -->
+			<resolution>1</resolution>
+			<samples>360</samples> <min_angle>-3.141592</min_angle> <max_angle>3.124139361</max_angle> <!-- -180 to 180 Degree -->
+		    </horizontal>
+		</scan>
+		<range>
+		    <min>0.2</min>
+		    <max>6</max>
+		    <resolution>0.02</resolution>
+		</range>
+		<noise>
+		    <type>gaussian</type>
+		    <mean>0.0</mean>
+		    <stddev>0.03</stddev>
+		</noise>
+	    </ray>
+	    <plugin name="gazebo_ros_laser_RPLidar_driver" filename="${driver_type}" >
+		<rosDebugLevel>Debug</rosDebugLevel>
+		<robotNamespace></robotNamespace>
+		<topicName>${name}/scan</topicName>
+		<frameName>${name}</frameName>
+	    </plugin>
         </sensor>
     </gazebo>

File: tuw_gazebo_models/models/sensors/laser/Sick-LMS100.xacro (robot description, xacro)
@@ -2,7 +2,7 @@
 <robot xmlns:xacro="http://www.ros.org/wiki/xacro">
 <!-- Front Laser -->
-<xacro:macro name="laser" params="name parent xyz rpy driver:=gpu model_dir:=^">
-  <xacro:if     value="${driver == 'gpu'}"> <xacro:property name="driver_name" value="_gpu"/></xacro:if>
-  <xacro:unless value="${driver == 'gpu'}"> <xacro:property name="driver_name" value=""    /></xacro:unless>
+<xacro:macro name="laser" params="name parent xyz rpy driver:=cpu model_dir:=^">
+  <xacro:if     value="${driver == 'gpu'}"> <xacro:property name="sensor_type" value="gpu_ray"/> <xacro:property name="driver_type" value="libtuw_gazebo_ros_gpu_laser.so"/> </xacro:if>
+  <xacro:unless value="${driver == 'gpu'}"> <xacro:property name="sensor_type" value="ray"    /> <xacro:property name="driver_type" value="libtuw_gazebo_ros_laser.so"    /> </xacro:unless>
   <joint name="${parent}_${name}_chassis_joint" type="fixed">
 	  <axis xyz="0 0 1" />
@@ -36,39 +36,40 @@
   </joint>
   <link name="${name}"/>
-	<gazebo reference="${name}">
-		<sensor name="laser" type="${driver_name}ray">
-			<pose>0 0 0 0 0 0</pose>
-			<update_rate>25</update_rate>
-			<always_on>1</always_on>
-			<visualize>true</visualize>
-			<ray>
-				<scan>
-				  <horizontal>
-					<!-- Sick-LMS100 has  683 steps with 0.35139 Degree resolution-->
-					<resolution>1</resolution>
-					<max_angle>2.356000000</max_angle> <min_angle>-2.356000000</min_angle> <samples>1080</samples>     <!-- 135 to -135 Degree -->
-					<!--max_angle>2.094400000</max_angle> <min_angle>-2.094400000</min_angle> <samples>683</samples--> <!-- 120 to -120 Degree -->
-					<!--max_angle>1.745329252</max_angle> <min_angle>-1.745329252</min_angle> <samples>570</samples--> <!-- 100 to -100 Degree -->
-					<!--max_angle>1.919862177</max_angle> <min_angle>-1.919862177</min_angle> <samples>626</samples--> <!-- 110 to -110 Degree -->
-					</horizontal>
-				</scan>
-				<range>
-					<min>0.2</min>
-					<max>20.0</max>
-					<resolution>0.01</resolution>
-				</range>
-				<noise>
-					<type>gaussian</type>
-					<mean>0.0</mean>
-					<stddev>0.01</stddev>
-				</noise>
-			</ray>
-			<plugin name="gazebo_ros_laser_sick_driver" filename="libgazebo_ros_${driver_name}laser.so" >
-				<robotNamespace></robotNamespace>
-				<topicName>${name}/scan</topicName>
-				<frameName>${name}</frameName>
-			</plugin>
-		</sensor>
-	</gazebo>
+    <gazebo reference="${name}">
+	<sensor name="laser" type="${sensor_type}">
+	    <pose>0 0 0 0 0 0</pose>
+	    <update_rate>25</update_rate>
+	    <always_on>1</always_on>
+	    <visualize>true</visualize>
+	    <ray>
+		<scan>
+		    <horizontal>
+			<!-- Sick-LMS100 has  683 steps with 0.35139 Degree resolution-->
+			<resolution>1</resolution>
+			<max_angle>2.356000000</max_angle> <min_angle>-2.356000000</min_angle> <samples>1080</samples>     <!-- 135 to -135 Degree -->
+			<!--max_angle>2.094400000</max_angle> <min_angle>-2.094400000</min_angle> <samples>683</samples--> <!-- 120 to -120 Degree -->
+			<!--max_angle>1.745329252</max_angle> <min_angle>-1.745329252</min_angle> <samples>570</samples--> <!-- 100 to -100 Degree -->
+			<!--max_angle>1.919862177</max_angle> <min_angle>-1.919862177</min_angle> <samples>626</samples--> <!-- 110 to -110 Degree -->
+		    </horizontal>
+		</scan>
+		<range>
+		    <min>0.2</min>
+		    <max>20.0</max>
+		    <resolution>0.01</resolution>
+		</range>
+		<noise>
+		    <type>gaussian</type>
+		    <mean>0.0</mean>
+		    <stddev>0.01</stddev>
+		</noise>
+	    </ray>
+	    <plugin name="gazebo_ros_laser_SICK_driver" filename="${driver_type}" >
+		<rosDebugLevel>Debug</rosDebugLevel>
+		<robotNamespace></robotNamespace>
+		<topicName>${name}/scan</topicName>
+		<frameName>${name}</frameName>
+	    </plugin>
+	</sensor>
+    </gazebo>
 </xacro:macro>
 </robot>

File: tuw_gazebo_models/models/sensors/laser/hokuyo.xacro (robot description, xacro)
@@ -2,7 +2,7 @@
 <robot xmlns:xacro="http://www.ros.org/wiki/xacro">
 <!-- Front Laser -->
-<xacro:macro name="laser" params="name parent xyz rpy driver:=gpu model_dir:=^" >
-  <xacro:if     value="${driver == 'gpu'}"> <xacro:property name="driver_name" value="gpu_"/></xacro:if>
-  <xacro:unless value="${driver == 'gpu'}"> <xacro:property name="driver_name" value=""    /></xacro:unless>
+<xacro:macro name="laser" params="name parent xyz rpy driver:=cpu model_dir:=^" >
+  <xacro:if     value="${driver == 'gpu'}"> <xacro:property name="sensor_type" value="gpu_ray"/> <xacro:property name="driver_type" value="libtuw_gazebo_ros_gpu_laser.so"/> </xacro:if>
+  <xacro:unless value="${driver == 'gpu'}"> <xacro:property name="sensor_type" value="ray"    /> <xacro:property name="driver_type" value="libtuw_gazebo_ros_laser.so"    /> </xacro:unless>
   <joint name="${parent}_${name}_joint" type="fixed">
       <axis xyz="0 0 1" />
@@ -25,41 +25,42 @@
       </visual>
       <inertial>
-        <mass value="1e-5" />
+        <mass value="1e-2" />
         <origin xyz="0 0 -0.025" rpy="0 0 0"/>
         <inertia ixx="1e-6" ixy="0" ixz="0" iyy="1e-6" iyz="0" izz="1e-6" />
       </inertial>
     </link>
-	<gazebo reference="${name}">
-		<sensor name="laser" type="${driver_name}ray">
-			<pose>0 0 0 0 0 0</pose>
-			<update_rate>10</update_rate>
-			<visualize>true</visualize>
-			<always_on>1</always_on>
-			<ray>
-				<scan>
-					<horizontal>
-						<!-- The URG-04LX-UG01  has  683 steps with 0.35139 Degree resolution -->
-						<resolution>1</resolution>
-						<samples>683</samples> <min_angle>-2.0944</min_angle> <max_angle>2.0944</max_angle> <!-- -120 to 120 Degree -->
-					</horizontal>
-				</scan>
-				<range>
-					<min>0.08</min>
-					<max>5</max>
-					<resolution>0.01</resolution>
-				</range>
-				<noise>
-					<type>gaussian</type>
-					<mean>0.0</mean>
-					<stddev>0.03</stddev>
-				</noise>
-			</ray>
-			<plugin name="gazebo_ros_laser_hokuyo_driver" filename="libgazebo_ros_${driver_name}laser.so" >
-				<robotNamespace></robotNamespace>
-				<topicName>${name}/scan</topicName>
-				<frameName>${name}</frameName>
-			</plugin>
-		</sensor>
-	</gazebo>
+    <gazebo reference="${name}">
+	<sensor name="laser" type="${sensor_type}">
+	    <pose>0 0 0 0 0 0</pose>
+	    <update_rate>10</update_rate>
+	    <visualize>true</visualize>
+	    <always_on>1</always_on>
+	    <ray>
+		<scan>
+		    <horizontal>
+			<!-- The URG-04LX-UG01  has  683 steps with 0.35139 Degree resolution -->
+			<resolution>1</resolution>
+			<samples>683</samples> <min_angle>-2.0944</min_angle> <max_angle>2.0944</max_angle> <!-- -120 to 120 Degree -->
+		    </horizontal>
+		</scan>
+		<range>
+		    <min>0.08</min>
+		    <max>5</max>
+		    <resolution>0.01</resolution>
+		</range>
+		<noise>
+		    <type>gaussian</type>
+		    <mean>0.0</mean>
+		    <stddev>0.03</stddev>
+		</noise>
+	    </ray>
+	    <plugin name="gazebo_ros_laser_hokuyo_driver" filename="${driver_type}" >
+		<rosDebugLevel>Debug</rosDebugLevel>
+		<robotNamespace></robotNamespace>
+		<topicName>${name}/scan</topicName>
+		<frameName>${name}</frameName>
+	    </plugin>
+	</sensor>
+    </gazebo>
 </xacro:macro>
 </robot>
