Commit message: changes: -ray plugins now properly "not identify" too close obstacles -xmlns namespaces are now consistent -minor model tweaks

File: tuw_gazebo_models/models/platforms/pioneer3dx/pioneer3dx.xacro (robot description, xacro)
@@ -1,4 +1,4 @@
 <?xml version="1.0"?>
-<robot xmlns:xacro="http://www.ros.org/wiki/xacro" name="pioneer3dx" >
+<robot xmlns:xacro="http://ros.org/wiki/xacro" name="pioneer3dx" >
   <xacro:arg name="model_dir" default="$(find tuw_gazebo_models)/models/platforms/pioneer3dx"/>
   <!-- Import Rviz colors -->

File: tuw_gazebo_models/models/platforms/pioneer3dx/pioneer3dx_body/battery_block.xacro (robot description, xacro)
@@ -1,4 +1,4 @@
 <?xml version="1.0"?>
-<robot xmlns:xacro="http://www.ros.org/wiki/xacro">
+<robot xmlns:xacro="http://ros.org/wiki/xacro">
   <xacro:property name="M_PI" value="3.1415926535897931" />
   <xacro:macro name="pioneer_battery_block" params="name parent x y z mass">

File: tuw_gazebo_models/models/platforms/pioneer3dx/pioneer3dx_body/body.xacro (robot description, xacro)
@@ -1,4 +1,4 @@
 <?xml version="1.0"?>
-<robot xmlns:xacro="http://www.ros.org/wiki/xacro">
+<robot xmlns:xacro="http://ros.org/wiki/xacro">
   <xacro:include filename="$(find tuw_gazebo_models)/models/inertia_tensors.xacro"/>
   <xacro:include filename="chassis.xacro"/>

File: tuw_gazebo_models/models/platforms/pioneer3dx/pioneer3dx_body/chassis.xacro (robot description, xacro)
@@ -1,4 +1,4 @@
 <?xml version="1.0"?>
-<robot xmlns:xacro="http://www.ros.org/wiki/xacro">
+<robot xmlns:xacro="http://ros.org/wiki/xacro">
   <xacro:property name="M_PI" value="3.1415926535897931" />
   <xacro:macro name="pioneer_chassis" params="name parent xyz rpy model_dir:=^">

File: tuw_gazebo_models/models/platforms/pioneer3dx/pioneer3dx_body/sonar.xacro (robot description, xacro)
@@ -1,4 +1,4 @@
 <?xml version="1.0"?>
-<robot xmlns:xacro="http://www.ros.org/wiki/xacro">
+<robot xmlns:xacro="http://ros.org/wiki/xacro">
   <xacro:property name="M_PI" value="3.1415926535897931" />
   <xacro:macro name="pioneer_sonar" params="name parent xyz rpy model_dir:=^">

File: tuw_gazebo_models/models/platforms/pioneer3dx/pioneer3dx_body/swivel.xacro (robot description, xacro)
@@ -1,4 +1,4 @@
 <?xml version="1.0"?>
-<robot xmlns:xacro="http://www.ros.org/wiki/xacro">
+<robot xmlns:xacro="http://ros.org/wiki/xacro">
   <xacro:property name="M_PI" value="3.1415926535897931" />
   <xacro:macro name="pioneer_swivel" params="parent xyz rpy model_dir:=^ **contact_data">

File: tuw_gazebo_models/models/platforms/pioneer3dx/pioneer3dx_body/wheel.xacro (robot description, xacro)
@@ -1,5 +1,5 @@
 <?xml version="1.0"?>
 <robot
-  xmlns:xacro="http://www.ros.org/wiki/xacro">
+  xmlns:xacro="http://ros.org/wiki/xacro">
   <xacro:property name="M_PI" value="3.1415926535897931" />
   <xacro:macro name="pioneer_wheel" params="side parent xyz rpy radius model_dir:=^ **contact_data">

File: tuw_gazebo_models/models/platforms/pioneer3dx/pioneer3dx_plugins.xacro (robot description, xacro)
@@ -1,4 +1,4 @@
 <?xml version="1.0"?>
-<robot xmlns:xacro="http://www.ros.org/wiki/xacro">
+<robot xmlns:xacro="http://ros.org/wiki/xacro">
   <xacro:macro name="pioneer3dx_joints_state_publisher">
     <gazebo>

File: tuw_gazebo_models/models/sensors/laser/RPLidar.xacro (robot description, xacro)
@@ -45,5 +45,5 @@
 		</scan>
 		<range>
-		    <min>0.2</min>
+		    <min>0.04</min>
 		    <max>6</max>
 		    <resolution>0.02</resolution>
@@ -60,4 +60,5 @@
 		<topicName>${name}/scan</topicName>
 		<frameName>${name}</frameName>
+		<rangeMin>0.2</rangeMin>
 	    </plugin>
         </sensor>

File: tuw_gazebo_models/models/sensors/laser/Sick-LMS100.xacro (robot description, xacro)
@@ -54,5 +54,5 @@
 		</scan>
 		<range>
-		    <min>0.2</min>
+		    <min>0.06</min>
 		    <max>20.0</max>
 		    <resolution>0.01</resolution>
@@ -69,4 +69,5 @@
 		<topicName>${name}/scan</topicName>
 		<frameName>${name}</frameName>
+		<rangeMin>0.2</rangeMin>
 	    </plugin>
 	</sensor>

File: tuw_gazebo_models/models/sensors/laser/hokuyo.xacro (robot description, xacro)
@@ -15,5 +15,5 @@
 	    <origin xyz="0 0 -0.025" rpy="0 0 0"/>
 	    <geometry>
-		<box size="0.1 0.1 0.1"/>
+		<box size="0.05 0.05 0.05"/>
 	    </geometry>
 	</collision>
@@ -45,5 +45,5 @@
 		</scan>
 		<range>
-		    <min>0.08</min>
+		    <min>0.04</min>
 		    <max>5</max>
 		    <resolution>0.01</resolution>
@@ -60,4 +60,5 @@
 		<topicName>${name}/scan</topicName>
 		<frameName>${name}</frameName>
+		<rangeMin>0.2</rangeMin>
 	    </plugin>
 	</sensor>

Commit message: changes: - minor changes for gazebo_ros_bridge_model plugin p3dx: - modified collision box of model to cope better with hitting walls (now it doesn't explode) - modified fricition parameters for more realistic values - now the model stays really flat on the ground - the launch file pioneer3dx.gazebo.launch now has a parameter plugin_type that can be switched between generic plugins or tuw plugins - fixed gazebo_ros_diff_drive plugin to again work ok with set-velocity (previously broken)

File: tuw_gazebo_models/models/platforms/pioneer3dx/pioneer3dx.xacro (robot description, xacro)
@@ -1,5 +1,7 @@
 <?xml version="1.0"?>
 <robot xmlns:xacro="http://ros.org/wiki/xacro" name="pioneer3dx" >
-  <xacro:arg name="model_dir" default="$(find tuw_gazebo_models)/models/platforms/pioneer3dx"/>
+  <xacro:arg name="model_dir"   default="$(find tuw_gazebo_models)/models/platforms/pioneer3dx"/>
+  <xacro:arg name="namespace"   default="p3dx"/>
+  <xacro:arg name="plugin_type" default="tuw"/> <!-- tuw or generic. If something else is set, no plugin will be loaded-->
   <!-- Import Rviz colors -->
   <xacro:include filename="$(find tuw_gazebo_models)/models/materials.xacro" />
@@ -9,11 +11,17 @@
   <xacro:pioneer3dx_body name="chassis" parent="base_link"/>
   <!-- Import platform plugins -->
-  <xacro:property name="model_dir" value="$(arg model_dir)"/>
+  <xacro:property name="model_dir"   value="$(arg model_dir)"/>
+  <xacro:property name="namespace"   value="$(arg namespace)"/>
+  <xacro:property name="plugin_type" value="$(arg plugin_type)"/>
   <xacro:include filename="${model_dir}/pioneer3dx_plugins.xacro" />
-  <!--xacro:pioneer3dx_diff_drive             /--> <!-- Motor  plugin -->
-  <!--xacro:pioneer3dx_joints_state_publisher /--> <!-- Joints plugin -->
-  <xacro:P3dxRosBridgeModelPlugin/>
+  <xacro:if value="${plugin_type == 'tuw'}">
+    <xacro:P3dxRosBridgeModelPlugin/> <!-- Motor  plugin -->
+  </xacro:if>
+  <xacro:if value="${plugin_type == 'generic'}">
+    <xacro:pioneer3dx_diff_drive/> <!-- Motor  plugin -->
+  </xacro:if>
+  <!-- Joints plugin -->
   <xacro:p3dx_joints_state_publisher ns=""/>
-  <xacro:p3dx_joints_state_publisher ns="p3dx/ground_truth"/>
+  <xacro:p3dx_joints_state_publisher ns="${namespace}/ground_truth"/>
   <!-- Laser -->
   <xacro:property name="model_dir" value="$(find tuw_gazebo_models)/models/sensors/laser"/>

File: tuw_gazebo_models/models/platforms/pioneer3dx/pioneer3dx_body/body.xacro (robot description, xacro)
@@ -18,13 +18,13 @@
     <!-- Wheels -->
     <xacro:property name="contact_data">
-        <mu1 value="5.9"/>
-	<mu2 value="5.9"/>
+        <mu1 value="0.7"/>
+	<mu2 value="0.7"/>
 	<minDepth value="0.002"/>
 	<kp value="1000000.0"/>
 	<kd value="10.0"/>
     </xacro:property>
-    <xacro:pioneer_swivel             parent="${name}"  xyz="-0.185 0    0.055" rpy="0 0 0">               <container> <xacro:insert_block name="contact_data"/> </container> </xacro:pioneer_swivel>
-    <xacro:pioneer_wheel side="right" parent="${name}"  xyz=" 0    -0.15 0.09"  rpy="0 0 0" radius="0.09"> <container> <xacro:insert_block name="contact_data"/> </container> </xacro:pioneer_wheel>
-    <xacro:pioneer_wheel side="left"  parent="${name}"  xyz=" 0     0.15 0.09"  rpy="0 0 0" radius="0.09"> <container> <xacro:insert_block name="contact_data"/> </container> </xacro:pioneer_wheel>
+    <xacro:pioneer_swivel             parent="${name}"  xyz="-0.185 0    0.0535" rpy="0 0 0">               <container> <xacro:insert_block name="contact_data"/> </container> </xacro:pioneer_swivel>
+    <xacro:pioneer_wheel side="right" parent="${name}"  xyz=" 0    -0.15 0.09"   rpy="0 0 0" radius="0.09"> <container> <xacro:insert_block name="contact_data"/> </container> </xacro:pioneer_wheel>
+    <xacro:pioneer_wheel side="left"  parent="${name}"  xyz=" 0     0.15 0.09"   rpy="0 0 0" radius="0.09"> <container> <xacro:insert_block name="contact_data"/> </container> </xacro:pioneer_wheel>
   </xacro:macro>
 </robot>

File: tuw_gazebo_models/models/platforms/pioneer3dx/pioneer3dx_body/chassis.xacro (robot description, xacro)
@@ -20,8 +20,10 @@
     </visual>
     <collision>
-      <origin xyz="-0.045 0 0.148" rpy="0 0 0"/>
+      <origin xyz="0.01 0 0.15" rpy="0 0 0"/>
+      <geometry><cylinder radius="0.17" length="0.17"/> </geometry>
+      <!--origin xyz="-0.045 0 0.148" rpy="0 0 0"/>
       <geometry>
 	<mesh filename="file://${model_dir}/meshes/chassis.dae"/>
-      </geometry>
+      </geometry-->
     </collision>
     <box_inertial_with_origin x="0.35" y="0.25"  z="0.17" mass="9.0"> <origin xyz="-0.04 0 0.15" rpy="0 0 0"/> </box_inertial_with_origin>
@@ -47,8 +49,10 @@
     </visual>
     <collision>
-    <origin xyz="0.0 0 0.0" rpy="0 0 0"/>
+    <origin xyz="-0.05 0 ${-0.235+0.15}" rpy="0 0 0"/>
+    <geometry><cylinder radius="0.17" length="0.17"/> </geometry>
+    <!--origin xyz="0.0 0 0.0" rpy="0 0 0"/>
       <geometry>
         <mesh filename="file://${model_dir}/meshes/top.dae"/>
-      </geometry>
+      </geometry-->
     </collision>
     <box_inertial_with_origin x="0.45" y="0.35"  z="0.001" mass="1.0"> <origin xyz="0.00 0 0.00" rpy="0 0 0"/> </box_inertial_with_origin>

File: tuw_gazebo_models/models/platforms/pioneer3dx/pioneer3dx_body/swivel.xacro (robot description, xacro)
@@ -9,5 +9,5 @@
     <anchor xyz="0 0 0"/>
     <limit effort="100" velocity="100" k_velocity="0"/>
-    <joint_properties damping="0.0" friction="0.0"/>
+    <joint_properties damping="0.1" friction="0.0"/>
     <parent link="${parent}"/>
     <child link="swivel"/>

Commit message: pioneer xacro update

File: tuw_gazebo_models/models/platforms/pioneer3dx/pioneer3dx.xacro (robot description, xacro)
@@ -27,5 +27,5 @@
   <xacro:property name="model_dir" value="$(find tuw_gazebo_models)/models/sensors/laser"/>
   <xacro:include filename="${model_dir}/hokuyo.xacro"/>
-  <xacro:laser name="laser_front" frame_names="laser_front" topic_names="laser_front/scan" parent="top" xyz="0.17 0 0.04" rpy="0 0 0" driver="cpu"/>
+  <xacro:laser name="laser_front" frame_names="laser_front" topic_names="laser_front/scan" parent="top" xyz="0.06 -0.14 0.08" rpy="0 0 -0.78" driver="cpu"/>
   <!-- xyz="0.16 0 0.125" -->
   <!-- IMU

File: tuw_gazebo_models/models/platforms/pioneer3dx/pioneer3dx_body/body.xacro (robot description, xacro)
@@ -3,17 +3,21 @@
   <xacro:include filename="$(find tuw_gazebo_models)/models/inertia_tensors.xacro"/>
   <xacro:include filename="chassis.xacro"/>
+  <xacro:include filename="mount.xacro"/>
   <xacro:include filename="battery_block.xacro"/>
   <xacro:include filename="wheel.xacro"/>
   <xacro:include filename="swivel.xacro"/>
   <xacro:include filename="sonar.xacro"/>
+  <xacro:property name="wheel_radius" value="0.097" />
   <xacro:macro name="pioneer3dx_body" params="name parent">
     <!-- base_link -->
     <link name="${parent}"/>
     <!-- Chassis -->
-    <xacro:pioneer_chassis name="${name}" parent="base_link" xyz="0 0 0" rpy="0 0 0"/>
+    <xacro:pioneer_chassis name="${name}" parent="${parent}" xyz="0 0 0.068" rpy="0 0 0"/>
+    <!-- Mount -->
+    <xacro:pioneer_mount name="mount" parent="top" xyz="0 0 0.0" rpy="0 0 0"/>
     <!-- Front Sonar -->
-    <xacro:pioneer_sonar name="sonar" parent="${name}" xyz="0.109 0 0.209" rpy="0 0 0"/>
+    <xacro:pioneer_sonar name="sonar" parent="${name}" xyz="0.109 0 0.15" rpy="0 0 0"/>
     <!-- Akku0 -->
-    <xacro:pioneer_battery_block name="battery0" parent="${name}" x="-0.14" y="0.00"  z="0.13" mass="2.5" />
+    <xacro:pioneer_battery_block name="battery0" parent="${name}" x="-0.14" y="0.00"  z="${0.13-0.068}" mass="2.5" />
     <!-- Wheels -->
     <xacro:property name="contact_data">
@@ -24,7 +28,7 @@
 	<kd value="10.0"/>
     </xacro:property>
-    <xacro:pioneer_swivel             parent="${name}"  xyz="-0.185 0    0.0535" rpy="0 0 0">               <container> <xacro:insert_block name="contact_data"/> </container> </xacro:pioneer_swivel>
-    <xacro:pioneer_wheel side="right" parent="${name}"  xyz=" 0    -0.15 0.09"   rpy="0 0 0" radius="0.09"> <container> <xacro:insert_block name="contact_data"/> </container> </xacro:pioneer_wheel>
-    <xacro:pioneer_wheel side="left"  parent="${name}"  xyz=" 0     0.15 0.09"   rpy="0 0 0" radius="0.09"> <container> <xacro:insert_block name="contact_data"/> </container> </xacro:pioneer_wheel>
+    <xacro:pioneer_swivel             parent="${parent}"  xyz="-0.185 0    0.0535" rpy="0 0 0">               <container> <xacro:insert_block name="contact_data"/> </container> </xacro:pioneer_swivel>
+    <xacro:pioneer_wheel side="right" parent="${parent}"  xyz=" 0    -0.15 ${wheel_radius}"   rpy="0 0 0" radius="${wheel_radius}"> <container> <xacro:insert_block name="contact_data"/> </container> </xacro:pioneer_wheel>
+    <xacro:pioneer_wheel side="left"  parent="${parent}"  xyz=" 0     0.15 ${wheel_radius}"   rpy="0 0 0" radius="${wheel_radius}"> <container> <xacro:insert_block name="contact_data"/> </container> </xacro:pioneer_wheel>
   </xacro:macro>
 </robot>

File: tuw_gazebo_models/models/platforms/pioneer3dx/pioneer3dx_body/chassis.xacro (robot description, xacro)
@@ -11,5 +11,5 @@
   <link name="${name}">
     <visual>
-      <origin xyz="-0.045 0 0.148" rpy="0 0 0"/>
+      <origin xyz="-0.045 0 0.085" rpy="0 0 0"/>
       <geometry>
 	<mesh filename="file://${model_dir}/meshes/chassis.dae"/>
@@ -20,5 +20,5 @@
     </visual>
     <collision>
-      <origin xyz="0.01 0 0.15" rpy="0 0 0"/>
+      <origin xyz="0.01 0 0.09" rpy="0 0 0"/>
       <geometry><cylinder radius="0.17" length="0.17"/> </geometry>
       <!--origin xyz="-0.045 0 0.148" rpy="0 0 0"/>
@@ -34,11 +34,11 @@
   <!-- Top -->
   <joint name="${name}_top_joint" type="fixed">
-    <origin xyz="-0.045 0 0.235" rpy="0 0 0"/>
-    <parent link="${name}"/>
+    <origin xyz="0 0 0.245" rpy="0 0 0"/>
+    <parent link="${parent}"/>
     <child link="top"/>
   </joint>
   <link name="top">
     <visual>
-      <origin xyz="0 0 0" rpy="0 0 0"/>
+      <origin xyz="-0.045 0 0" rpy="0 0 0"/>
       <geometry>
         <mesh filename="file://${model_dir}/meshes/top.dae"/>
@@ -49,5 +49,5 @@
     </visual>
     <collision>
-    <origin xyz="-0.05 0 ${-0.235+0.15}" rpy="0 0 0"/>
+    <origin xyz="${-0.045-0.05} 0 ${-0.235+0.15}" rpy="0 0 0"/>
     <geometry><cylinder radius="0.17" length="0.17"/> </geometry>
     <!--origin xyz="0.0 0 0.0" rpy="0 0 0"/>

Commit message: second laser added

File: tuw_gazebo_models/models/platforms/pioneer3dx/pioneer3dx.xacro (robot description, xacro)
@@ -27,5 +27,9 @@
   <xacro:property name="model_dir" value="$(find tuw_gazebo_models)/models/sensors/laser"/>
   <xacro:include filename="${model_dir}/hokuyo.xacro"/>
-  <xacro:laser name="laser_front" frame_names="laser_front" topic_names="laser_front/scan" parent="top" xyz="0.06 -0.14 0.08" rpy="0 0 -0.78" driver="cpu"/>
+  <xacro:laser name="laser_front_right" frame_names="laser_front_right" topic_names="laser_front_right/scan" parent="top" xyz="0.06 -0.14 0.08" rpy="0 0 ${-pi/4}" driver="cpu"/>
+  <!-- Laser -->
+  <xacro:property name="model_dir" value="$(find tuw_gazebo_models)/models/sensors/laser"/>
+  <xacro:include filename="${model_dir}/Sick-LMS100.xacro"/>
+  <xacro:laser name="laser_front_center" frame_names="laser_front_center" topic_names="laser_front_center/scan" parent="top" xyz="0.08 0.0 0.26" rpy="${pi} 0 0" driver="cpu"/>
   <!-- xyz="0.16 0 0.125" -->
   <!-- IMU

File: tuw_gazebo_models/models/platforms/pioneer3dx/pioneer3dx_body/mount.xacro (robot description, xacro)
@@ -52,4 +52,10 @@
       </material>
     </visual>
+    <collision>
+      <origin xyz="-0.04 +${0.27/2.} 0.01"/>
+      <geometry>
+        <box size="0.31 0.04 0.02"/>
+      </geometry>
+    </collision>
     <!-- left base bar -->
     <visual>
@@ -62,4 +68,10 @@
       </material>
     </visual>
+    <collision>
+      <origin xyz="-0.04 -${0.27/2.} 0.01"/>
+      <geometry>
+        <box size="0.31 0.04 0.02"/>
+      </geometry>
+    </collision>
     <!-- right column -->
     <visual>
@@ -72,4 +84,10 @@
       </material>
     </visual>
+    <collision>
+      <origin xyz="-0.0 +${0.25/2.} ${0.02+0.92/2}"/>
+      <geometry>
+        <box size="0.02 0.02 0.92"/>
+      </geometry>
+    </collision>
     <!-- left column -->
     <visual>
@@ -82,4 +100,10 @@
       </material>
     </visual>
+    <collision>
+      <origin xyz="-0.0 -${0.25/2.} ${0.02+0.92/2}"/>
+      <geometry>
+        <box size="0.02 0.02 0.92"/>
+      </geometry>
+    </collision>
     <!-- laser bar -->
     <visual>
@@ -92,4 +116,10 @@
       </material>
     </visual>
+    <collision>
+      <origin xyz="0.02 0 0.19"/>
+      <geometry>
+        <box size="0.02 0.27 0.02 "/>
+      </geometry>
+    </collision>
     <!-- camera tof bar low -->
     <visual>
@@ -102,4 +132,10 @@
       </material>
     </visual>
+    <collision>
+      <origin xyz="-0.02 0 0.36"/>
+      <geometry>
+        <box size="0.02 0.27 0.02 "/>
+      </geometry>
+    </collision>
     <!-- camera tof bar bottom -->
     <visual>
@@ -112,4 +148,10 @@
       </material>
     </visual>
+    <collision>
+      <origin xyz="-0.02 0 0.47"/>
+      <geometry>
+        <box size="0.02 0.27 0.02 "/>
+      </geometry>
+    </collision>
     <!-- Top bar -->
     <visual>
@@ -122,4 +164,10 @@
       </material>
     </visual>
+    <collision>
+      <origin xyz="0 0 ${0.02+0.92+0.02/2}"/>
+      <geometry>
+        <box size="0.02 0.30 0.02 "/>
+      </geometry>
+    </collision>
   </link>
   <gazebo reference="${name}_bottom_left">

File: tuw_gazebo_models/models/sensors/laser/RPLidar.xacro (robot description, xacro)
@@ -31,5 +31,5 @@
     </link>
     <gazebo reference="${name}">
-        <sensor name="laser" type="${sensor_type}">
+        <sensor name="${name}" type="${sensor_type}">
 	    <pose>0 0 0 0 0 0</pose>
 	    <update_rate>5.5</update_rate>

File: tuw_gazebo_models/models/sensors/laser/Sick-LMS100.xacro (robot description, xacro)
@@ -37,5 +37,5 @@
     <link name="${name}"/>
     <gazebo reference="${name}">
-	<sensor name="laser" type="${sensor_type}">
+	<sensor name="${name}" type="${sensor_type}">
 	    <pose>0 0 0 0 0 0</pose>
 	    <update_rate>25</update_rate>

File: tuw_gazebo_models/models/sensors/laser/hokuyo.xacro (robot description, xacro)
@@ -31,5 +31,5 @@
     </link>
     <gazebo reference="${name}">
-	<sensor name="laser" type="${sensor_type}">
+	<sensor name="${name}" type="${sensor_type}">
 	    <pose>0 0 0 0 0 0</pose>
 	    <update_rate>10</update_rate>

Commit message: depth camera added

File: tuw_gazebo_models/models/platforms/pioneer3dx/pioneer3dx.xacro (robot description, xacro)
@@ -27,9 +27,9 @@
   <xacro:property name="model_dir" value="$(find tuw_gazebo_models)/models/sensors/laser"/>
   <xacro:include filename="${model_dir}/hokuyo.xacro"/>
-  <xacro:laser name="laser_front_right" frame_names="laser_front_right" topic_names="laser_front_right/scan" parent="top" xyz="0.06 -0.14 0.08" rpy="0 0 ${-pi/4}" driver="cpu"/>
+  <xacro:laser name="laser_front_right" frame_names="laser_front_right" topic_names="laser_front_right/scan" parent="top" xyz="0.06 -0.14 0.08" rpy="0 0 ${-pi/4}" driver="gpu"/>
   <!-- Laser -->
   <xacro:property name="model_dir" value="$(find tuw_gazebo_models)/models/sensors/laser"/>
   <xacro:include filename="${model_dir}/Sick-LMS100.xacro"/>
-  <xacro:laser name="laser_front_center" frame_names="laser_front_center" topic_names="laser_front_center/scan" parent="top" xyz="0.08 0.0 0.26" rpy="${pi} 0 0" driver="cpu"/>
+  <xacro:laser name="laser_front_center" frame_names="laser_front_center" topic_names="laser_front_center/scan" parent="top" xyz="0.08 0.0 0.26" rpy="${pi} 0 0" driver="gpu"/>
   <!-- xyz="0.16 0 0.125" -->
   <!-- IMU
@@ -41,5 +41,10 @@
   <xacro:property name="model_dir" value="$(find tuw_gazebo_models)/models/sensors/camera"/>
   <xacro:include filename="${model_dir}/camera.xacro"/>
-  <xacro:cam name="front_camera" parent="chassis" xyz="0 0 0.5" rpy="${-pi/2}  0 ${-pi/2}" />
-  -->
+  <xacro:cam name="front_camera" parent="top" xyz="0 0 1" rpy="${-pi/2}  0 ${-pi/2}" />
+   -->
+  <!-- Depth Camera
+  <xacro:property name="model_dir" value="$(find tuw_gazebo_models)/models/sensors/camera"/>
+  <xacro:include filename="${model_dir}/depth_camera.xacro"/>
+  <xacro:cam name="front_depth_camera" parent="top" xyz="0 0 1" rpy="0  0 0" />
+ -->
 </robot>

Commit message: parameter plugin_type changed to moter_plugin

File: tuw_gazebo_models/models/platforms/pioneer3dx/pioneer3dx.xacro (robot description, xacro)
@@ -3,5 +3,5 @@
   <xacro:arg name="model_dir"   default="$(find tuw_gazebo_models)/models/platforms/pioneer3dx"/>
   <xacro:arg name="namespace"   default="p3dx"/>
-  <xacro:arg name="plugin_type" default="tuw"/> <!-- tuw or generic. If something else is set, no plugin will be loaded-->
+  <xacro:arg name="motor_plugin" default="diff_twist"/> <!-- diff_iws or diff_twist. If something else is set, no plugin will be loaded-->
   <!-- Import Rviz colors -->
   <xacro:include filename="$(find tuw_gazebo_models)/models/materials.xacro" />
@@ -13,10 +13,10 @@
   <xacro:property name="model_dir"   value="$(arg model_dir)"/>
   <xacro:property name="namespace"   value="$(arg namespace)"/>
-  <xacro:property name="plugin_type" value="$(arg plugin_type)"/>
+  <xacro:property name="motor_plugin" value="$(arg motor_plugin)"/>
   <xacro:include filename="${model_dir}/pioneer3dx_plugins.xacro" />
-  <xacro:if value="${plugin_type == 'tuw'}">
+  <xacro:if value="${motor_plugin == 'diff_iws'}">
     <xacro:P3dxRosBridgeModelPlugin/> <!-- Motor  plugin -->
   </xacro:if>
-  <xacro:if value="${plugin_type == 'generic'}">
+  <xacro:if value="${motor_plugin == 'diff_twist'}">
     <xacro:pioneer3dx_diff_drive/> <!-- Motor  plugin -->
   </xacro:if>
