Commit message: file names for robot model simplyfied

File: tuw_gazebo_models/models/platforms/pioneer3dx/main.xacro (robot description, xacro)
@@ -7,5 +7,5 @@
   <xacro:include filename="$(find tuw_gazebo_models)/models/materials.xacro" />
   <!-- Import platform -->
-  <xacro:property name="model_dir" value="$(arg model_dir)/pioneer3dx_body"/>
+  <xacro:property name="model_dir" value="$(arg model_dir)/body"/>
   <xacro:include filename="${model_dir}/body.xacro"/>
   <xacro:pioneer3dx_body name="chassis" parent="base_link"/>
@@ -14,10 +14,10 @@
   <xacro:property name="namespace"   value="$(arg namespace)"/>
   <xacro:property name="motor_plugin" value="$(arg motor_plugin)"/>
-  <xacro:include filename="${model_dir}/pioneer3dx_plugins.xacro" />
+  <xacro:include filename="${model_dir}/plugins.xacro" />
   <xacro:if value="${motor_plugin == 'diff_iws'}">
-    <xacro:P3dxRosBridgeModelPlugin/> <!-- Motor  plugin -->
+    <xacro:iws_drive/> <!-- Motor  plugin -->
   </xacro:if>
   <xacro:if value="${motor_plugin == 'diff_twist'}">
-    <xacro:pioneer3dx_diff_drive/> <!-- Motor  plugin -->
+    <xacro:differential_drive/> <!-- Motor  plugin -->
   </xacro:if>
   <!-- Joints plugin -->

File: tuw_gazebo_models/models/platforms/pioneer3dx/plugins_param.xacro (robot description, xacro)
@@ -1,5 +1,5 @@
 <?xml version="1.0"?>
 <robot xmlns:xacro="http://ros.org/wiki/xacro">
-<xacro:property name="P3dxGazeboPluginsData">
+  <xacro:property name="IWSPluginsData">
 	<rosDebugLevel>Debug</rosDebugLevel>
 	<robotNamespace></robotNamespace>
@@ -22,4 +22,4 @@
 	<base_cmd_topic>base_cmds</base_cmd_topic>
 	<joints_cmd_topic>joint_cmds</joints_cmd_topic>
-</xacro:property>
+  </xacro:property>
 </robot>

Commit message: update on joint_state_publisher in xacro

File: tuw_gazebo_models/models/platforms/pioneer3dx/main.xacro (robot description, xacro)
@@ -16,12 +16,16 @@
   <xacro:include filename="${model_dir}/plugins.xacro" />
   <xacro:if value="${motor_plugin == 'diff_iws'}">
-    <xacro:iws_drive/> <!-- Motor  plugin -->
+    <!-- Motor  plugin -->
+    <xacro:iws_drive/>
+    <!-- Joints plugin -->
+    <xacro:iws_joints_state_publisher ns=""/>
+    <xacro:iws_joints_state_publisher ns="${namespace}/ground_truth"/>
   </xacro:if>
   <xacro:if value="${motor_plugin == 'diff_twist'}">
-    <xacro:differential_drive/> <!-- Motor  plugin -->
+    <!-- Motor  plugin -->
+    <xacro:differential_drive/>
+    <!-- Joints plugin -->
+	<xacro:diff_joints_state_publisher ns="${namespace}"/>
   </xacro:if>
-  <!-- Joints plugin -->
-  <xacro:p3dx_joints_state_publisher ns=""/>
-  <xacro:p3dx_joints_state_publisher ns="${namespace}/ground_truth"/>
   <!-- Laser -->
   <xacro:property name="model_dir" value="$(find tuw_gazebo_models)/models/sensors/laser"/>

File: tuw_gazebo_models/models/platforms/pioneer3dx/plugins.xacro (robot description, xacro)
@@ -1,8 +1,8 @@
 <?xml version="1.0"?>
 <robot xmlns:xacro="http://ros.org/wiki/xacro">
-  <!--xacro:macro name="pioneer3dx_joints_state_publisher">
+  <xacro:macro name="diff_joints_state_publisher" params="ns">
     <gazebo>
         <plugin name="joint_state_publisher" filename="libgazebo_ros_joint_state_publisher.so">
-          <robotNamespace></robotNamespace>
+          <robotNamespace>${ns}</robotNamespace>
           <jointName>chassis_swivel_joint, swivel_wheel_joint, left_hub_joint, right_hub_joint</jointName>
           <updateRate>10.0</updateRate>
@@ -10,5 +10,5 @@
         </plugin>
     </gazebo>
-  </xacro:macro -->
+  </xacro:macro>
   <xacro:macro name="differential_drive">
     <gazebo>
@@ -38,4 +38,14 @@
     </gazebo>
   </xacro:macro>
+  <xacro:macro name="iws_joints_state_publisher" params="ns">
+	<gazebo>
+	  <plugin name="joint_state_publisher" filename="libgazebo_ros_joint_state_publisher.so">
+		<robotNamespace>${ns}</robotNamespace>
+		<jointName>chassis_swivel_joint, swivel_wheel_joint</jointName>
+		<updateRate>50.0</updateRate>
+		<alwaysOn>true</alwaysOn>
+	  </plugin>
+	</gazebo>
+  </xacro:macro>
   <xacro:include filename="plugins_param.xacro"/>
   <xacro:macro name="iws_drive">
@@ -46,13 +56,3 @@
 	</gazebo>
   </xacro:macro>
-  <xacro:macro name="p3dx_joints_state_publisher" params="ns">
-	<gazebo>
-	  <plugin name="joint_state_publisher" filename="libgazebo_ros_joint_state_publisher.so">
-		<robotNamespace>${ns}</robotNamespace>
-		<jointName>   chassis_swivel_joint, swivel_wheel_joint</jointName>
-		<updateRate>50.0</updateRate>
-		<alwaysOn>true</alwaysOn>
-	  </plugin>
-	</gazebo>
-  </xacro:macro>
 </robot>

Commit message: pioneer discribtion independet to ros pkg name

File: tuw_gazebo_models/models/platforms/pioneer3dx/main.xacro (robot description, xacro)
@@ -1,15 +1,16 @@
 <?xml version="1.0"?>
 <robot xmlns:xacro="http://ros.org/wiki/xacro" name="pioneer3dx" >
-  <xacro:arg name="model_dir"   default="$(find tuw_gazebo_models)/models/platforms/pioneer3dx"/>
-  <xacro:arg name="namespace"   default="p3dx"/>
+  <xacro:arg name="model_dir"      default=""/>
+  <xacro:arg name="platform_dir"   default=""/>
+  <xacro:arg name="namespace"      default="r1"/>
   <xacro:arg name="motor_plugin" default="diff_twist"/> <!-- diffdrive or iws. If something else is set, no plugin will be loaded-->
   <!-- Import Rviz colors -->
-  <xacro:include filename="$(find tuw_gazebo_models)/models/materials.xacro" />
+  <xacro:include filename="$(arg model_dir)/materials.xacro" />
   <!-- Import platform -->
-  <xacro:property name="model_dir" value="$(arg model_dir)/body"/>
+  <xacro:property name="model_dir" value="$(arg model_dir)/$(arg platform_dir)/body"/>
   <xacro:include filename="${model_dir}/body.xacro"/>
   <xacro:pioneer3dx_body name="chassis" parent="base_link"/>
   <!-- Import platform plugins -->
-  <xacro:property name="model_dir"   value="$(arg model_dir)"/>
+  <xacro:property name="model_dir"   value="$(arg model_dir)/$(arg platform_dir)"/>
   <xacro:property name="namespace"   value="$(arg namespace)"/>
   <xacro:property name="motor_plugin" value="$(arg motor_plugin)"/>
@@ -29,24 +30,24 @@
   </xacro:if>
   <!-- Laser -->
-  <xacro:property name="model_dir" value="$(find tuw_gazebo_models)/models/sensors/laser"/>
+  <xacro:property name="model_dir" value="$(arg model_dir)/sensors/laser"/>
   <xacro:include filename="${model_dir}/hokuyo.xacro"/>
   <xacro:laser name="laser_front_right" frame_names="laser_front_right" topic_names="laser_front_right/scan/raw" parent="top" xyz="0.15 0.0 0.06" rpy="0 0 0" driver="cpu" visualize="true"/>
   <!-- Laser -->
-  <xacro:property name="model_dir" value="$(find tuw_gazebo_models)/models/sensors/laser"/>
+  <xacro:property name="model_dir" value="$(arg model_dir)/sensors/laser"/>
   <xacro:include filename="${model_dir}/Sick-LMS100.xacro"/>
   <xacro:laser name="laser_front_center" frame_names="laser_front_center" topic_names="laser_front_center/scan/raw" parent="top" xyz="0.08 0.0 0.26" rpy="${pi} 0 0" driver="cpu" visualize="false"/>
   <!-- xyz="0.16 0 0.125" -->
   <!-- IMU
-  <xacro:property name="model_dir" value="$(find tuw_gazebo_models)/models/sensors/imu"/>
-  <xacro:include filename="$(find tuw_gazebo_models)/models/sensors/imu/imu.xacro"/>
+  <xacro:property name="model_dir" value="$(arg model_dir)/sensors/imu"/>
+  <xacro:include filename="$(arg model_dir)/sensors/imu/imu.xacro"/>
   <xacro:imu_sensor name="imu9dof" parent="chassis" xyz="0.05 0.0 0.262" rpy="0 0 0"/>
   -->
   <!-- Camera
-  <xacro:property name="model_dir" value="$(find tuw_gazebo_models)/models/sensors/camera"/>
+  <xacro:property name="model_dir" value="$(arg model_dir)/sensors/camera"/>
   <xacro:include filename="${model_dir}/camera.xacro"/>
   <xacro:cam name="front_camera" parent="top" xyz="0 0 1" rpy="${-pi/2}  0 ${-pi/2}" />
    -->
   <!-- Depth Camera
-  <xacro:property name="model_dir" value="$(find tuw_gazebo_models)/models/sensors/camera"/>
+  <xacro:property name="model_dir" value="$(arg model_dir)/sensors/camera"/>
   <xacro:include filename="${model_dir}/depth_camera.xacro"/>
   <xacro:cam name="front_depth_camera" parent="top" xyz="0 0 1" rpy="0  0 0" />

Commit message: launch file update to support velodyne ranger

File: tuw_gazebo_models/models/platforms/pioneer3dx/main.xacro (robot description, xacro)
@@ -3,4 +3,6 @@
   <xacro:arg name="model_dir"      default=""/>
   <xacro:arg name="platform_dir"   default=""/>
+  <xacro:arg name="laser0"         default="hokuyo"/>    <!-- hokuyo or velodyne -->
+  <xacro:arg name="gpu"            default="false"/>
   <xacro:arg name="namespace"      default="r0"/>
   <xacro:arg name="motor_plugin"   default="diff_twist"/> <!-- diffdrive or diff_iws. If something else is set, no plugin will be loaded-->
@@ -12,7 +14,9 @@
   <xacro:vehicle_body name="chassis" parent="base_link"/>
   <!-- Import platform plugins -->
-  <xacro:property name="model_dir"   value="$(arg model_dir)/$(arg platform_dir)"/>
-  <xacro:property name="namespace"   value="$(arg namespace)"/>
+  <xacro:property name="model_dir"    value="$(arg model_dir)/$(arg platform_dir)"/>
+  <xacro:property name="namespace"    value="$(arg namespace)"/>
   <xacro:property name="motor_plugin" value="$(arg motor_plugin)"/>
+  <xacro:property name="laser0"       value="$(arg laser0)"/>
+  <xacro:property name="gpu"          value="$(arg gpu)"/>
   <xacro:include filename="${model_dir}/plugins.xacro" />
   <xacro:if value="${motor_plugin == 'diff_iws'}">
@@ -29,8 +33,21 @@
     <xacro:diff_joints_state_publisher ns="${namespace}"/>
   </xacro:if>
-  <!-- Laser -->
-  <xacro:property name="model_dir" value="$(arg model_dir)/sensors/laser"/>
-  <xacro:include filename="${model_dir}/hokuyo.xacro"/>
-  <xacro:laser name="laser0" frame_names="laser0" topic_names="laser0/scan/raw" parent="top" xyz="0.15 0.0 0.06" rpy="0 0 0" driver="cpu" visualize="true"/>
+  <!-- Laser0 -->
+  <xacro:if value="${laser0 == 'hokuyo'}">
+    <xacro:property name="model_dir" value="$(arg model_dir)/sensors/laser"/>
+    <xacro:include filename="${model_dir}/hokuyo.xacro"/>
+    <xacro:if value="${gpu}">
+        <xacro:laser name="laser0" frame_names="laser0" topic_names="laser0/scan/raw" parent="top" xyz="0.15 0.0 0.06" rpy="0 0 0" driver="cpu" visualize="true"/>
+    </xacro:if>
+    <xacro:unless value="${gpu}">
+        <xacro:laser name="laser0" frame_names="laser0" topic_names="laser0/scan/raw" parent="top" xyz="0.15 0.0 0.06" rpy="0 0 0" driver="gpu" visualize="true"/>
+    </xacro:unless>
+  </xacro:if>
+  <xacro:if value="${laser0 == 'velodyne'}">
+    <xacro:include filename="$(find velodyne_description)/urdf/VLP-16.urdf.xacro"/>
+    <VLP-16 parent="top" name="velodyne" topic="velodyne_points" hz="10" samples="440" gpu="${gpu}">
+        <origin xyz="0.10 0.0 0.0" rpy="0 0 0" />
+    </VLP-16>
+  </xacro:if>
   <!-- Laser
   <xacro:property name="model_dir" value="$(arg model_dir)/sensors/laser"/>

Commit message: laser topic name as parameter added

File: tuw_gazebo_models/models/platforms/pioneer3dx/main.xacro (robot description, xacro)
@@ -7,4 +7,5 @@
   <xacro:arg name="namespace"      default="r0"/>
   <xacro:arg name="motor_plugin"   default="diff_twist"/> <!-- diffdrive or diff_iws. If something else is set, no plugin will be loaded-->
+  <xacro:arg name="laser0_topic"   default="laser0/scan/raw"/>
   <!-- Import Rviz colors -->
   <xacro:include filename="$(arg model_dir)/materials.xacro" />
@@ -18,4 +19,5 @@
   <xacro:property name="motor_plugin" value="$(arg motor_plugin)"/>
   <xacro:property name="laser0"       value="$(arg laser0)"/>
+  <xacro:property name="laser0_topic" value="$(arg laser0_topic)"/>
   <xacro:property name="gpu"          value="$(arg gpu)"/>
   <xacro:include filename="${model_dir}/plugins.xacro" />
@@ -38,8 +40,8 @@
     <xacro:include filename="${model_dir}/hokuyo.xacro"/>
     <xacro:if value="${gpu}">
-        <xacro:laser name="laser0" frame_names="laser0" topic_names="laser0/scan/raw" parent="top" xyz="0.15 0.0 0.06" rpy="0 0 0" driver="cpu" visualize="true"/>
+        <xacro:laser name="laser0" frame_names="laser0" topic_names="${laser0_topic}" parent="top" xyz="0.15 0.0 0.06" rpy="0 0 0" driver="cpu" visualize="true"/>
     </xacro:if>
     <xacro:unless value="${gpu}">
-        <xacro:laser name="laser0" frame_names="laser0" topic_names="laser0/scan/raw" parent="top" xyz="0.15 0.0 0.06" rpy="0 0 0" driver="gpu" visualize="true"/>
+        <xacro:laser name="laser0" frame_names="laser0" topic_names="${laser0_topic}" parent="top" xyz="0.15 0.0 0.06" rpy="0 0 0" driver="gpu" visualize="true"/>
     </xacro:unless>
   </xacro:if>

Commit message: diffdrive plugin fixed and as launch parameter added

File: tuw_gazebo_models/models/platforms/pioneer3dx/main.xacro (robot description, xacro)
@@ -1,11 +1,12 @@
 <?xml version="1.0"?>
 <robot xmlns:xacro="http://ros.org/wiki/xacro" name="pioneer3dx" >
-  <xacro:arg name="model_dir"      default=""/>
-  <xacro:arg name="platform_dir"   default=""/>
-  <xacro:arg name="laser0"         default="hokuyo"/>    <!-- hokuyo or velodyne -->
-  <xacro:arg name="gpu"            default="false"/>
-  <xacro:arg name="namespace"      default="r0"/>
-  <xacro:arg name="motor_plugin"   default="diff_twist"/> <!-- diffdrive or diff_iws. If something else is set, no plugin will be loaded-->
-  <xacro:arg name="laser0_topic"   default="laser0/scan/raw"/>
+  <xacro:arg name="model_dir"                  default=""/>
+  <xacro:arg name="platform_dir"               default=""/>
+  <xacro:arg name="laser0"                     default="hokuyo"/>    <!-- hokuyo or velodyne -->
+  <xacro:arg name="gpu"                        default="false"/>
+  <xacro:arg name="namespace"                  default="r0"/>
+  <xacro:arg name="motor_plugin"               default="diff_twist"/> <!-- diffdrive or diff_iws. If something else is set, no plugin will be loaded-->
+  <xacro:arg name="differential_odom_source"   default="differential_odom_source"/>  <!-- endocer or world. Only used with diff_twist -->
+  <xacro:arg name="laser0_topic"               default="laser0/scan/raw"/>
   <!-- Import Rviz colors -->
   <xacro:include filename="$(arg model_dir)/materials.xacro" />
@@ -15,10 +16,11 @@
   <xacro:vehicle_body name="chassis" parent="base_link"/>
   <!-- Import platform plugins -->
-  <xacro:property name="model_dir"    value="$(arg model_dir)/$(arg platform_dir)"/>
-  <xacro:property name="namespace"    value="$(arg namespace)"/>
-  <xacro:property name="motor_plugin" value="$(arg motor_plugin)"/>
-  <xacro:property name="laser0"       value="$(arg laser0)"/>
-  <xacro:property name="laser0_topic" value="$(arg laser0_topic)"/>
-  <xacro:property name="gpu"          value="$(arg gpu)"/>
+  <xacro:property name="model_dir"                value="$(arg model_dir)/$(arg platform_dir)"/>
+  <xacro:property name="namespace"                value="$(arg namespace)"/>
+  <xacro:property name="motor_plugin"             value="$(arg motor_plugin)"/>
+  <xacro:property name="differential_odom_source" value="$(arg differential_odom_source)"/>
+  <xacro:property name="laser0"                   value="$(arg laser0)"/>
+  <xacro:property name="laser0_topic"             value="$(arg laser0_topic)"/>
+  <xacro:property name="gpu"                      value="$(arg gpu)"/>
   <xacro:include filename="${model_dir}/plugins.xacro" />
   <xacro:if value="${motor_plugin == 'diff_iws'}">
@@ -31,5 +33,5 @@
   <xacro:if value="${motor_plugin == 'diff_twist'}">
     <!-- Motor  plugin -->
-    <xacro:differential_drive/>
+    <xacro:differential_drive ns="${namespace}" odom_source="${differential_odom_source}"/>
     <!-- Joints plugin -->
     <xacro:diff_joints_state_publisher ns="${namespace}"/>

File: tuw_gazebo_models/models/platforms/pioneer3dx/plugins.xacro (robot description, xacro)
@@ -11,5 +11,5 @@
     </gazebo>
   </xacro:macro>
-  <xacro:macro name="differential_drive">
+  <xacro:macro name="differential_drive" params="ns odom_source">
     <gazebo>
         <plugin name="differential_drive_controller" filename="libtuw_gazebo_ros_diff_drive.so">
@@ -22,16 +22,16 @@
 	      <odometryFrame>odom</odometryFrame>
 	      <commandTopic>cmd_vel</commandTopic>
-          <odometryTopic>odom</odometryTopic>
-          <!-- odom source world or encoder, world uses the simulated ground truth and encoder the wheel odometry -->
-          <odometrySource>encoder</odometrySource>
-          <leftJoint>left_hub_joint</leftJoint>
-          <rightJoint>right_hub_joint</rightJoint>
-          <wheelSeparation>0.3</wheelSeparation>
-          <wheelDiameter>0.18</wheelDiameter>
-          <wheelTorque>10</wheelTorque>
-          <wheelAcceleration>1.5</wheelAcceleration>
-          <publishTf>true</publishTf>
+        <odometryTopic>odom</odometryTopic>
+        <!-- odom source world or encoder, world uses the simulated ground truth and encoder the wheel odometry -->
+        <odometrySource>${odom_source}</odometrySource>
+        <leftJoint>left_hub_joint</leftJoint>
+        <rightJoint>right_hub_joint</rightJoint>
+        <wheelSeparation>0.3</wheelSeparation>
+        <wheelDiameter>0.18</wheelDiameter>
+        <wheelTorque>10</wheelTorque>
+        <wheelAcceleration>1.5</wheelAcceleration>
+        <publishTf>true</publishTf>
 	      <publishWheelTF>true</publishWheelTF>
-          <publishWheelJointState>true</publishWheelJointState>
+        <publishWheelJointState>true</publishWheelJointState>
         </plugin>
     </gazebo>
