Commit message: extend camera configuration

File: tuw_gazebo_models/models/sensors/camera/zed.xacro (robot description, xacro)
@@ -1,5 +1,5 @@
 <?xml version="1.0"?>
 <robot xmlns:xacro="http://ros.org/wiki/xacro">
-<xacro:macro name="zed" params="name parent xyz rpy">
+<xacro:macro name="zed" params="name parent frame_name robot_ns='' xyz rpy">
   <joint name="${parent}_${name}_joint" type="fixed">
       <axis xyz="0 0 1" />
@@ -33,5 +33,5 @@
   </gazebo>
   <gazebo reference="${name}">
-    <sensor type="camera" name="zed_left">
+    <sensor type="camera" name="${name}_left">
       <update_rate>30.0</update_rate>
       <camera name="head">
@@ -57,11 +57,11 @@
       </camera>
       <plugin name="camera_controller" filename="libgazebo_ros_camera.so">
-        <robotNamespace></robotNamespace>
+        <robotNamespace>${robot_ns}</robotNamespace>
         <alwaysOn>true</alwaysOn>
         <updateRate>30.0</updateRate>
         <cameraName>${name}</cameraName>
-        <imageTopicName>image_raw</imageTopicName>
-        <cameraInfoTopicName>camera_info</cameraInfoTopicName>
-        <frameName>${name}</frameName>
+        <imageTopicName>left/image_raw</imageTopicName>
+        <cameraInfoTopicName>left/camera_info</cameraInfoTopicName>
+        <frameName>${frame_name}/left_frame</frameName>
         <hackBaseline>0.06</hackBaseline>
         <distortionK1>0.0</distortionK1>

Commit message: update sensor descriptions

File: tuw_gazebo_models/models/sensors/camera/zed.xacro (robot description, xacro)
@@ -1,19 +1,19 @@
 <?xml version="1.0"?>
 <robot xmlns:xacro="http://ros.org/wiki/xacro">
-<xacro:macro name="zed" params="name parent frame_name robot_ns='' xyz rpy">
-  <joint name="${parent}_${name}_joint" type="fixed">
-      <axis xyz="0 0 1" />
+  <xacro:macro name="zed" params="name parent frame_name robot_ns='' xyz rpy">
+    <joint name="${parent}_${name}_joint" type="fixed">
+      <axis xyz="0 0 1"/>
       <origin xyz="${xyz}" rpy="${rpy}"/>
       <parent link="${parent}"/>
       <child link="${name}"/>
-  </joint>
-  <!-- robot link -->
-  <link name="${name}">
-    <inertial>
-      <mass value="1e-5" />
-      <origin xyz="0 0 0" rpy="0 0 0"/>
-      <inertia ixx="1e-6" ixy="0" ixz="0" iyy="1e-6" iyz="0" izz="1e-6" />
-    </inertial>
-    <!--visual>
+    </joint>
+    <!-- robot link -->
+    <link name="${name}">
+      <inertial>
+        <mass value="1e-5"/>
+        <origin xyz="0 0 0" rpy="0 0 0"/>
+        <inertia ixx="1e-6" ixy="0" ixz="0" iyy="1e-6" iyz="0" izz="1e-6"/>
+      </inertial>
+      <!--visual>
       <origin xyz="0 0 0" rpy="0 0 0"/>
       <geometry>
@@ -22,5 +22,5 @@
       <material name="grey"/>
     </visual-->
-    <!--collision>
+      <!--collision>
       <origin xyz="0 0 0" rpy="0 0 0"/>
       <geometry>
@@ -28,49 +28,49 @@
       </geometry>
     </collision-->
-  </link>
-  <gazebo reference="${name}">
-    <material value="Gazebo/Grey"/>
-  </gazebo>
-  <gazebo reference="${name}">
-    <sensor type="camera" name="${name}_left">
-      <update_rate>30.0</update_rate>
-      <camera name="head">
-        <pose>0 0 0 0 0 0</pose>
-        <horizontal_fov>1.7</horizontal_fov>
-        <image>
-          <width>1280</width>
-          <height>720</height>
-          <format>B8G8R8</format>
-        </image>
-        <clip>
-          <near>0.02</near>
-          <far>300</far>
-        </clip>
-        <noise>
-          <type>gaussian</type>
-          <!-- Noise is sampled independently per pixel on each frame.
+    </link>
+    <gazebo reference="${name}">
+      <material value="Gazebo/Grey"/>
+    </gazebo>
+    <gazebo reference="${name}">
+      <sensor type="camera" name="${name}_left">
+        <update_rate>30.0</update_rate>
+        <camera name="head">
+          <pose>0 0 0 0 0 0</pose>
+          <horizontal_fov>1.7</horizontal_fov>
+          <image>
+            <width>1280</width>
+            <height>720</height>
+            <format>B8G8R8</format>
+          </image>
+          <clip>
+            <near>0.02</near>
+            <far>300</far>
+          </clip>
+          <noise>
+            <type>gaussian</type>
+            <!-- Noise is sampled independently per pixel on each frame.
                That pixel's noise value is added to each of its color
                channels, which at that point lie in the range [0,1]. -->
-          <mean>0.0</mean>
-          <stddev>0.007</stddev>
-        </noise>
-      </camera>
-      <plugin name="camera_controller" filename="libgazebo_ros_camera.so">
-        <robotNamespace>${robot_ns}</robotNamespace>
-        <alwaysOn>true</alwaysOn>
-        <updateRate>30.0</updateRate>
-        <cameraName>${name}</cameraName>
-        <imageTopicName>left/image_raw</imageTopicName>
-        <cameraInfoTopicName>left/camera_info</cameraInfoTopicName>
-        <frameName>${frame_name}/left_frame</frameName>
-        <hackBaseline>0.06</hackBaseline>
-        <distortionK1>0.0</distortionK1>
-        <distortionK2>0.0</distortionK2>
-        <distortionK3>0.0</distortionK3>
-        <distortionT1>0.0</distortionT1>
-        <distortionT2>0.0</distortionT2>
-      </plugin>
-    </sensor>
-  </gazebo>
-</xacro:macro>
+            <mean>0.0</mean>
+            <stddev>0.007</stddev>
+          </noise>
+        </camera>
+        <plugin name="camera_controller" filename="libgazebo_ros_camera.so">
+          <robotNamespace>${robot_ns}</robotNamespace>
+          <alwaysOn>false</alwaysOn>
+          <updateRate>30.0</updateRate>
+          <cameraName>${name}</cameraName>
+          <imageTopicName>left/image_raw</imageTopicName>
+          <cameraInfoTopicName>left/camera_info</cameraInfoTopicName>
+          <frameName>${frame_name}/left_frame</frameName>
+          <hackBaseline>0.06</hackBaseline>
+          <distortionK1>0.0</distortionK1>
+          <distortionK2>0.0</distortionK2>
+          <distortionK3>0.0</distortionK3>
+          <distortionT1>0.0</distortionT1>
+          <distortionT2>0.0</distortionT2>
+        </plugin>
+      </sensor>
+    </gazebo>
+  </xacro:macro>
 </robot>

File: tuw_gazebo_models/models/sensors/laser/hokuyo_30LX.xacro (robot description, xacro)
@@ -61,5 +61,5 @@
             <type>gaussian</type>
             <mean>0.0</mean>
-            <stddev>0.003</stddev>
+            <stddev>0.006</stddev>
           </noise>
         </ray>
