Commit message: sally model updates

File: tuw_gazebo_models/models/platforms/sally/body/chassis.xacro (robot description, xacro)
@@ -14,5 +14,5 @@
   <link name="${name}">
     <visual>
-      <origin xyz="-0.045 0 0.085" rpy="0 0 0"/>
+      <origin xyz="-0.0 0 -0.04" rpy="0 0 ${M_PI}"/>
       <geometry>
 	<mesh filename="file://${model_dir}/meshes/chassis.dae"/>

File: tuw_gazebo_models/models/platforms/sally/main.xacro (robot description, xacro)
@@ -36,5 +36,5 @@
   <xacro:property name="model_dir" value="$(find tuw_gazebo_models)/models/sensors/laser"/>
   <xacro:include filename="${model_dir}/Sick-LMS100.xacro"/>
-  <xacro:laser name="laser_front_center" frame_names="laser_front_center" topic_names="laser_front_center/scan" parent="top" xyz="0.08 0.0 0.26" rpy="${pi} 0 0" driver="cpu"/>
+  <xacro:laser name="laser_front_center" frame_names="laser_front_center" topic_names="laser_front_center/scan" parent="top" xyz="0.15 0.0 0.5" rpy="${pi} 0 0" driver="cpu"/>
   <!-- xyz="0.16 0 0.125" -->
   <!-- IMU
