Commit message: model update

File: tuw_gazebo_models/models/platforms/sally/body/body.xacro (robot description, xacro)
@@ -3,9 +3,6 @@
   <xacro:include filename="$(find tuw_gazebo_models)/models/inertia_tensors.xacro"/>
   <xacro:include filename="chassis.xacro"/>
-  <xacro:include filename="mount.xacro"/>
-  <xacro:include filename="battery_block.xacro"/>
   <xacro:include filename="wheel.xacro"/>
   <xacro:include filename="swivel.xacro"/>
-  <xacro:include filename="sonar.xacro"/>
   <xacro:property name="wheel_radius" value="0.097" />
   <xacro:macro name="sally_body" params="name parent">
@@ -14,10 +11,4 @@
     <!-- Chassis -->
     <xacro:chassis name="${name}" parent="${parent}" xyz="0 0 0.068" rpy="0 0 0"/>
-    <!-- Mount -->
-    <xacro:pioneer_mount name="mount" parent="top" xyz="0 0 0.0" rpy="0 0 0"/>
-    <!-- Front Sonar -->
-    <xacro:pioneer_sonar name="sonar" parent="${name}" xyz="0.109 0 0.15" rpy="0 0 0"/>
-    <!-- Akku0 -->
-    <xacro:pioneer_battery_block name="battery0" parent="${name}" x="-0.14" y="0.00"  z="${0.13-0.068}" mass="2.5" />
     <!-- Wheels -->
     <xacro:property name="contact_data">
@@ -28,7 +19,8 @@
 	<!--kd value="10.0"/-->
     </xacro:property>
-    <xacro:pioneer_swivel             parent="${parent}"  xyz="-0.185 0    0.0535" rpy="0 0 0">               <container> <xacro:insert_block name="contact_data"/> </container> </xacro:pioneer_swivel>
-    <xacro:pioneer_wheel side="right" parent="${parent}"  xyz=" 0    -0.165 ${wheel_radius}" rpy="0 0 0" radius="${wheel_radius}"> <container> <xacro:insert_block name="contact_data"/> </container> </xacro:pioneer_wheel>
-    <xacro:pioneer_wheel side="left"  parent="${parent}"  xyz=" 0     0.165 ${wheel_radius}" rpy="0 0 0" radius="${wheel_radius}"> <container> <xacro:insert_block name="contact_data"/> </container> </xacro:pioneer_wheel>
+    <xacro:swivel side="front" parent="${parent}"  xyz=" 0.200 0    0.0535" rpy="0 0 0">               <container> <xacro:insert_block name="contact_data"/> </container> </xacro:swivel>
+    <xacro:swivel side="back"  parent="${parent}"  xyz="-0.200 0    0.0535" rpy="0 0 0">               <container> <xacro:insert_block name="contact_data"/> </container> </xacro:swivel>
+    <xacro:wheel  side="right" parent="${parent}"  xyz=" 0    -0.225 ${wheel_radius}" rpy="0 0 0" radius="${wheel_radius}"> <container> <xacro:insert_block name="contact_data"/> </container> </xacro:wheel>
+    <xacro:wheel  side="left"  parent="${parent}"  xyz=" 0     0.225 ${wheel_radius}" rpy="0 0 0" radius="${wheel_radius}"> <container> <xacro:insert_block name="contact_data"/> </container> </xacro:wheel>
   </xacro:macro>
 </robot>

File: tuw_gazebo_models/models/platforms/sally/body/chassis.xacro (robot description, xacro)
@@ -33,27 +33,18 @@
   <!-- Top -->
   <joint name="${name}_top_joint" type="fixed">
-    <origin xyz="0 0 0.245" rpy="0 0 0"/>
+    <origin xyz="0 0 0.5" rpy="0 0 0"/>
     <parent link="${parent}"/>
     <child link="top"/>
   </joint>
   <link name="top">
-    <visual>
-      <origin xyz="-0.045 0 0" rpy="0 0 0"/>
-      <geometry>
-        <mesh filename="file://${model_dir}/meshes/top.dae"/>
+    <visual name="${name}_visual">
+      <origin xyz="0 0 0" rpy="0 0 0"/>
+      <geometry name="${name}_geometry">
+        <box size="0.6 0.4 0.01"/>
       </geometry>
-      <material name="TopBlack">
+      <material name="${name}_material">
         <color rgba="0.038 0.038 0.038 1.0"/>
       </material>
     </visual>
-    <collision>
-    <origin xyz="${-0.045-0.05} 0 ${-0.235+0.15}" rpy="0 0 0"/>
-    <geometry><cylinder radius="0.17" length="0.17"/> </geometry>
-    <!--origin xyz="0.0 0 0.0" rpy="0 0 0"/>
-      <geometry>
-        <mesh filename="file://${model_dir}/meshes/top.dae"/>
-      </geometry-->
-    </collision>
-    <box_inertial_with_origin x="0.45" y="0.35"  z="0.001" mass="1.0"> <origin xyz="0.00 0 0.00" rpy="0 0 0"/> </box_inertial_with_origin>
   </link>
   <gazebo reference="top">

File: tuw_gazebo_models/models/platforms/sally/body/swivel.xacro (robot description, xacro)
@@ -2,7 +2,7 @@
 <robot xmlns:xacro="http://ros.org/wiki/xacro">
   <xacro:property name="M_PI" value="3.1415926535897931" />
-  <xacro:macro name="pioneer_swivel" params="parent xyz rpy model_dir:=^ **contact_data">
+  <xacro:macro name="swivel" params="side parent xyz rpy model_dir:=^ **contact_data">
   <!-- Swivel -->
-  <joint name="chassis_swivel_joint" type="continuous">
+  <joint name="${side}_swivel_joint" type="continuous">
     <origin xyz="${xyz}" rpy="${rpy}"/>
     <axis xyz="0 0 1"/>
@@ -11,7 +11,7 @@
     <joint_properties damping="0.1" friction="0.0"/>
     <parent link="${parent}"/>
-    <child link="swivel"/>
+    <child link="${side}_swivel"/>
   </joint>
-  <link name="swivel">
+  <link name="${side}_swivel">
     <box_inertial_with_origin x="0.07" y="0.07" z="0.05" mass="0.1"> <origin xyz="0 0 0" rpy="0 0 0"/> </box_inertial_with_origin>
     <!--inertial>
@@ -40,5 +40,5 @@
   </gazebo>
   <!-- Center Wheel -->
-  <joint name="swivel_wheel_joint" type="continuous">
+  <joint name="${side}_swivel_wheel_joint" type="continuous">
     <origin xyz="-0.026 0 -0.016" rpy="0 0 0"/>
     <axis xyz="0 1 0"/>
@@ -46,8 +46,8 @@
     <!--limit effort="100" velocity="100" k_velocity="0"/-->
     <joint_properties damping="0.0" friction="0.0"/>
-    <parent link="swivel"/>
-    <child link="center_wheel"/>
+    <parent link="${side}_swivel"/>
+    <child link="${side}_center_wheel"/>
   </joint>
-  <link name="center_wheel">
+  <link name="${side}_center_wheel">
     <cylinder_inertial_with_origin radius="0.0375" length="0.03" mass="0.1"> <origin xyz="0 0 0" rpy="${pi/2} 0 0"/> </cylinder_inertial_with_origin>
     <!--inertial>
@@ -78,10 +78,10 @@
   </gazebo>
   <!-- Center Hubcap -->
-  <joint name="wheel_hubcap_joint" type="fixed">
+  <joint name="${side}_wheel_hubcap_joint" type="fixed">
     <origin xyz="0 0 0" rpy="0 0 0"/>
-    <parent link="center_wheel"/>
-    <child link="center_hubcap"/>
+    <parent link="${side}_center_wheel"/>
+    <child link="${side}_center_hubcap"/>
   </joint>
-  <link name="center_hubcap">
+  <link name="${side}_center_hubcap">
     <cylinder_inertial_with_origin radius="0.01" length="0.03" mass="0.01"> <origin xyz="0 0 0" rpy="${pi/2} 0 0"/> </cylinder_inertial_with_origin>
     <!--inertial>

File: tuw_gazebo_models/models/platforms/sally/body/wheel.xacro (robot description, xacro)
@@ -3,50 +3,11 @@
   xmlns:xacro="http://ros.org/wiki/xacro">
   <xacro:property name="M_PI" value="3.1415926535897931" />
-  <xacro:macro name="pioneer_wheel" params="side parent xyz rpy radius model_dir:=^ **contact_data">
-    <!-- Hubcap Mount -->
-      <joint name="${side}_hub_mount_joint" type="fixed">
-	<origin xyz="${xyz}" rpy="${rpy}"/>
-	<parent link="${parent}"/>
-	<child link="${side}_hub_mount"/>
-	<axis xyz="0 1 0"/>
-    </joint>
-    <link name="${side}_hub_mount">
-	<cylinder_inertial_with_origin radius="0.01" length="0.01" mass="0.01"> <origin xyz="0 0 0" rpy="0 0 0"/> </cylinder_inertial_with_origin>
-	<visual>
-	    <origin xyz="0 0 0" rpy="0 0 0"/>
-	    <geometry> <box size="0.001 0.001 0.001"/> </geometry>
-	</visual>
-	<collision>
-	    <origin xyz="0 0 0" rpy="0 0 0"/>
-	    <geometry> <box size="0.001 0.001 0.001"/> </geometry>
-	</collision>
-    </link>
-    <!-- Hubcap -->
-    <joint name="${side}_hub_joint" type="continuous">
-	<origin xyz="0 0 0" rpy="0 0 0"/>
-	<parent link="${side}_hub_mount"/>
-	<child link="${side}_hub"/>
-	<axis xyz="0 1 0"/>
-    </joint>
-    <link name="${side}_hub">
-	<cylinder_inertial_with_origin radius="${radius}" length="0.03" mass="0.5"> <origin xyz="0 0 0" rpy="${pi/2} 0 0"/> </cylinder_inertial_with_origin>
-	<visual>
-	    <origin xyz="0 0 0" rpy="0 0 0"/>
-	    <geometry> <mesh filename="file://${model_dir}/meshes/hubcap.dae"/> </geometry>
-	    <material name="HubcapYellow"> <color rgba="1.0 0.811 0.151 1.0"/> </material>
-	</visual>
-	<collision>
-	    <origin xyz="0 0 0" rpy="0 0 0"/>
-	    <geometry> <box size="0.001 0.001 0.001"/> </geometry>
-	</collision>
-    </link>
-    <gazebo reference="${side}_hub">
-	<material value="Gazebo/Yellow"/>
-    </gazebo>
+  <xacro:macro name="wheel" params="side parent xyz rpy radius model_dir:=^ **contact_data">
     <!-- Wheel -->
     <joint name="${side}_wheel_joint" type="fixed">
+	<origin xyz="${xyz}" rpy="${rpy}"/>
 	<axis xyz="0 1 0"/>
 	<origin xyz="0 0 0" rpy="0 0 0"/>
-	<parent link="${side}_hub"/>
+	<parent link="${parent}"/>
 	<child link="${side}_wheel"/>
     </joint>
@@ -54,7 +15,6 @@
 	<cylinder_inertial_with_origin radius="${radius}" length="0.03" mass="0.5"> <origin xyz="0 0 0" rpy="${pi/2} 0 0"/> </cylinder_inertial_with_origin>
 	<visual>
-	    <origin xyz="0 0 0" rpy="0 0 0"/>
-	    <geometry> <mesh filename="file://${model_dir}/meshes/wheel.dae"/> </geometry>
-	    <material name="WheelBlack"> <color rgba="0.117 0.117 0.117 1"/> </material>
+	    <origin xyz="0 0 0.015" rpy="${pi/2} 0 0"/>
+	    <geometry> <cylinder radius="${radius}" length="0.03"/> <!--<mesh filename="${meshes}/${side}_wheel.stl"/>--> </geometry>
 	</visual>
 	<collision>

File: tuw_gazebo_models/models/platforms/sally/main.xacro (robot description, xacro)
@@ -36,5 +36,5 @@
   <xacro:property name="model_dir" value="$(find tuw_gazebo_models)/models/sensors/laser"/>
   <xacro:include filename="${model_dir}/Sick-LMS100.xacro"/>
-  <xacro:laser name="laser_front_center" frame_names="laser_front_center" topic_names="laser_front_center/scan" parent="top" xyz="0.15 0.0 0.5" rpy="${pi} 0 0" driver="cpu"/>
+  <xacro:laser name="laser_front_center" frame_names="laser_front_center" topic_names="laser_front_center/scan" parent="top" xyz="0.15 0.0 -0.20" rpy="${pi} 0 0" driver="cpu"/>
   <!-- xyz="0.16 0 0.125" -->
   <!-- IMU

File: tuw_gazebo_models/models/platforms/sally/plugins.xacro (robot description, xacro)
@@ -26,6 +26,6 @@
           <!-- odom source world or encoder, world uses the simulated ground truth and encoder the wheel odometry -->
           <odometrySource>encoder</odometrySource>
-          <leftJoint>left_hub_joint</leftJoint>
-          <rightJoint>right_hub_joint</rightJoint>
+          <leftJoint>left_wheel_jointt</leftJoint>
+          <rightJoint>right_wheel_joint</rightJoint>
           <wheelSeparation>0.3</wheelSeparation>
           <wheelDiameter>0.18</wheelDiameter>

File: tuw_gazebo_models/models/platforms/sally/plugins_param.xacro (robot description, xacro)
@@ -8,5 +8,5 @@
 	<alwaysOn>true</alwaysOn>
 	<updateRate>100.0</updateRate>
-	<revolute_joints_names>right_hub_joint, left_hub_joint</revolute_joints_names>
+	<revolute_joints_names>right_wheel_joint, left_wheel_joint</revolute_joints_names>
 	<revolute_max_torque>        10.0</revolute_max_torque> <!-- Nm  -->
 	<revolute_max_vel>           50.0</revolute_max_vel>    <!--rad/s-->
