Commit message: sally model working

File: tuw_gazebo_models/models/platforms/sally/body/battery_block.xacro (robot description, xacro)
@@ -2,5 +2,5 @@
 <robot xmlns:xacro="http://ros.org/wiki/xacro">
   <xacro:property name="M_PI" value="3.1415926535897931" />
-  <xacro:macro name="pioneer_battery_block" params="name parent x y z mass">
+  <xacro:macro name="battery_block" params="name parent x y z mass">
   <joint name="${parent}_${name}_joint" type="fixed">
     <origin xyz="${x} ${y} ${z}" rpy="0 0 0"/>

File: tuw_gazebo_models/models/platforms/sally/body/body.xacro (robot description, xacro)
@@ -4,6 +4,7 @@
   <xacro:include filename="chassis.xacro"/>
   <xacro:include filename="wheel.xacro"/>
+  <xacro:include filename="battery_block.xacro"/>
   <xacro:include filename="swivel.xacro"/>
-  <xacro:property name="wheel_radius" value="0.097" />
+  <xacro:property name="wheel_radius" value="0.104" />
   <xacro:macro name="sally_body" params="name parent">
     <!-- base_link -->
@@ -11,4 +12,6 @@
     <!-- Chassis -->
     <xacro:chassis name="${name}" parent="${parent}" xyz="0 0 0.068" rpy="0 0 0"/>
+    <!-- Akku0 -->
+    <xacro:battery_block name="battery0" parent="${name}" x="-0.14" y="0.00"  z="${0.13-0.068}" mass="2.5" />
     <!-- Wheels -->
     <xacro:property name="contact_data">
@@ -19,6 +22,6 @@
 	<!--kd value="10.0"/-->
     </xacro:property>
-    <xacro:swivel side="front" parent="${parent}"  xyz=" 0.200 0    0.0535" rpy="0 0 0">               <container> <xacro:insert_block name="contact_data"/> </container> </xacro:swivel>
-    <xacro:swivel side="back"  parent="${parent}"  xyz="-0.200 0    0.0535" rpy="0 0 0">               <container> <xacro:insert_block name="contact_data"/> </container> </xacro:swivel>
+    <xacro:swivel side="front" parent="${parent}"  xyz=" 0.200 0    0.055" rpy="0 0 0">               <container> <xacro:insert_block name="contact_data"/> </container> </xacro:swivel>
+    <xacro:swivel side="back"  parent="${parent}"  xyz="-0.200 0    0.055" rpy="0 0 0">               <container> <xacro:insert_block name="contact_data"/> </container> </xacro:swivel>
     <xacro:wheel  side="right" parent="${parent}"  xyz=" 0    -0.225 ${wheel_radius}" rpy="0 0 0" radius="${wheel_radius}"> <container> <xacro:insert_block name="contact_data"/> </container> </xacro:wheel>
     <xacro:wheel  side="left"  parent="${parent}"  xyz=" 0     0.225 ${wheel_radius}" rpy="0 0 0" radius="${wheel_radius}"> <container> <xacro:insert_block name="contact_data"/> </container> </xacro:wheel>

File: tuw_gazebo_models/models/platforms/sally/body/chassis.xacro (robot description, xacro)
@@ -14,5 +14,5 @@
   <link name="${name}">
     <visual>
-      <origin xyz="-0.0 0 -0.04" rpy="0 0 ${M_PI}"/>
+      <origin xyz="-0.0 0 -0.04" rpy="0 0 0"/>
       <geometry>
 	<mesh filename="file://${model_dir}/meshes/chassis.dae"/>
@@ -22,6 +22,8 @@
     </visual>
     <collision>
-      <origin xyz="0.01 0 0.09" rpy="0 0 0"/>
-      <geometry><cylinder radius="0.17" length="0.17"/> </geometry>
+      <origin xyz="-0.0 0 -0.04" rpy="0 0 0"/>
+      <geometry>
+	  <mesh filename="file://${model_dir}/meshes/chassis.dae"/>>
+      </geometry>
       <!--origin xyz="-0.045 0 0.148" rpy="0 0 0"/>
       <geometry>
@@ -38,5 +40,5 @@
   </joint>
   <link name="top">
-    <visual name="${name}_visual">
+    <!--visual name="${name}_visual">
       <origin xyz="0 0 0" rpy="0 0 0"/>
       <geometry name="${name}_geometry">
@@ -46,5 +48,5 @@
         <color rgba="0.038 0.038 0.038 1.0"/>
       </material>
-    </visual>
+    </visual-->
   </link>
   <gazebo reference="top">

File: tuw_gazebo_models/models/platforms/sally/body/wheel.xacro (robot description, xacro)
@@ -15,9 +15,9 @@
 	<cylinder_inertial_with_origin radius="${radius}" length="0.03" mass="0.5"> <origin xyz="0 0 0" rpy="${pi/2} 0 0"/> </cylinder_inertial_with_origin>
 	<visual>
-	    <origin xyz="0 0 0.015" rpy="${pi/2} 0 0"/>
+	    <origin xyz="0 0 0.0" rpy="${pi/2} 0 0"/>
 	    <geometry> <cylinder radius="${radius}" length="0.03"/> <!--<mesh filename="${meshes}/${side}_wheel.stl"/>--> </geometry>
 	</visual>
 	<collision>
-	    <origin xyz="0 0 0" rpy="${pi/2} 0 0"/>
+	    <origin xyz="0 0 0.0" rpy="${pi/2} 0 0"/>
 	    <geometry> <cylinder radius="${radius}" length="0.001"/> <!--<mesh filename="${meshes}/${side}_wheel.stl"/>--> </geometry>
 	</collision>

File: tuw_gazebo_models/models/platforms/sally/main.xacro (robot description, xacro)
@@ -36,5 +36,5 @@
   <xacro:property name="model_dir" value="$(find tuw_gazebo_models)/models/sensors/laser"/>
   <xacro:include filename="${model_dir}/Sick-LMS100.xacro"/>
-  <xacro:laser name="laser_front_center" frame_names="laser_front_center" topic_names="laser_front_center/scan" parent="top" xyz="0.15 0.0 -0.20" rpy="${pi} 0 0" driver="cpu"/>
+  <xacro:laser name="laser_front_center" frame_names="laser_front_center" topic_names="laser_front_center/scan" parent="top" xyz="0.25 0.0 -0.20" rpy="${pi} 0 0" driver="cpu"/>
   <!-- xyz="0.16 0 0.125" -->
   <!-- IMU
