Commit message: diffdrive not working

File: tuw_gazebo_models/models/platforms/sally/body/swivel.xacro (robot description, xacro)
@@ -77,37 +77,4 @@
     <xacro:insert_block name="contact_data"/>
   </gazebo>
-  <!-- Center Hubcap -->
-  <joint name="${side}_wheel_hubcap_joint" type="fixed">
-    <origin xyz="0 0 0" rpy="0 0 0"/>
-    <parent link="${side}_center_wheel"/>
-    <child link="${side}_center_hubcap"/>
-  </joint>
-  <link name="${side}_center_hubcap">
-    <cylinder_inertial_with_origin radius="0.01" length="0.03" mass="0.01"> <origin xyz="0 0 0" rpy="${pi/2} 0 0"/> </cylinder_inertial_with_origin>
-    <!--inertial>
-      <mass value="0.01"/>
-      <origin xyz="0 0 0"/>
-      <inertia ixx="0.012411765597" ixy="-0.000711733678" ixz="0.00050272983" iyy="0.015218160428" iyz="-0.000004273467" izz="0.011763977943"/>
-    </inertial-->
-    <visual>
-      <origin xyz="0 0 0" rpy="0 0 0"/>
-      <geometry>
-        <mesh filename="file://${model_dir}/meshes/center_hubcap.stl"/>
-      </geometry>
-      <material name="swivel">
-        <color rgba="0.5 0.5 0.5 1"/>
-      </material>
-    </visual>
-    <collision>
-      <origin xyz="0 0 0" rpy="0 0 0"/>
-      <geometry>
-        <box size="0.001 0.001 0.001"/>
-      </geometry>
-    </collision>
-  </link>
-  <gazebo reference="center_hubcap">
-    <material value="Gazebo/Grey"/>
-    <xacro:insert_block name="contact_data"/>
-  </gazebo>
   </xacro:macro>
 </robot>

File: tuw_gazebo_models/models/platforms/sally/main.xacro (robot description, xacro)
@@ -26,5 +26,5 @@
     <xacro:differential_drive/>
     <!-- Joints plugin -->
-	<xacro:diff_joints_state_publisher ns="${namespace}"/>
+	<!-- xacro:diff_joints_state_publisher ns="${namespace}"/-->
   </xacro:if>
   <!-- Laser

File: tuw_gazebo_models/models/platforms/sally/plugins.xacro (robot description, xacro)
@@ -26,5 +26,5 @@
           <!-- odom source world or encoder, world uses the simulated ground truth and encoder the wheel odometry -->
           <odometrySource>encoder</odometrySource>
-          <leftJoint>left_wheel_jointt</leftJoint>
+          <leftJoint>left_wheel_joint</leftJoint>
           <rightJoint>right_wheel_joint</rightJoint>
           <wheelSeparation>0.3</wheelSeparation>
