Commit message: sally working

File: tuw_gazebo_models/models/platforms/sally/body/wheel.xacro (robot description, xacro)
@@ -5,25 +5,26 @@
   <xacro:macro name="wheel" params="side parent xyz rpy radius model_dir:=^ **contact_data">
     <!-- Wheel -->
-    <joint name="${side}_wheel_joint" type="fixed">
-	<origin xyz="${xyz}" rpy="${rpy}"/>
-	<axis xyz="0 1 0"/>
-	<origin xyz="0 0 0" rpy="0 0 0"/>
-	<parent link="${parent}"/>
-	<child link="${side}_wheel"/>
+    <joint name="${side}_wheel_joint" type="continuous">
+        <origin xyz="${xyz}" rpy="${rpy}"/>
+        <axis xyz="0 1 0"/>
+        <parent link="${parent}"/>
+        <child link="${side}_wheel"/>
     </joint>
     <link name="${side}_wheel">
-	<cylinder_inertial_with_origin radius="${radius}" length="0.03" mass="0.5"> <origin xyz="0 0 0" rpy="${pi/2} 0 0"/> </cylinder_inertial_with_origin>
-	<visual>
-	    <origin xyz="0 0 0.0" rpy="${pi/2} 0 0"/>
-	    <geometry> <cylinder radius="${radius}" length="0.03"/> <!--<mesh filename="${meshes}/${side}_wheel.stl"/>--> </geometry>
-	</visual>
-	<collision>
-	    <origin xyz="0 0 0.0" rpy="${pi/2} 0 0"/>
-	    <geometry> <cylinder radius="${radius}" length="0.001"/> <!--<mesh filename="${meshes}/${side}_wheel.stl"/>--> </geometry>
-	</collision>
+        <cylinder_inertial_with_origin radius="${radius}" length="0.03" mass="0.5"> <origin xyz="0 0 0" rpy="${pi/2} 0 0"/> </cylinder_inertial_with_origin>
+        <visual>
+            <origin xyz="0 0 0.0" rpy="${pi/2} 0 0"/>
+            <geometry> <cylinder radius="${radius}" length="0.03"/> <!--<mesh filename="${meshes}/${side}_wheel.stl"/>--> </geometry>
+        </visual>
+        <collision>
+            <origin xyz="0 0 0.0" rpy="${pi/2} 0 0"/>
+            <geometry>
+                <cylinder radius="${radius}" length="0.001"/> <!--<mesh filename="${meshes}/${side}_wheel.stl"/>-->
+            </geometry>
+        </collision>
     </link>
     <gazebo reference="${side}_wheel">
-	<material value="Gazebo/Black"/>
-	<xacro:insert_block name="contact_data"/>
+        <material value="Gazebo/Black"/>
+        <xacro:insert_block name="contact_data"/>
     </gazebo>
   </xacro:macro>

File: tuw_gazebo_models/models/platforms/sally/main.xacro (robot description, xacro)
@@ -26,5 +26,5 @@
     <xacro:differential_drive/>
     <!-- Joints plugin -->
-	<!-- xacro:diff_joints_state_publisher ns="${namespace}"/-->
+    <xacro:diff_joints_state_publisher ns=""/>
   </xacro:if>
   <!-- Laser

File: tuw_gazebo_models/models/platforms/sally/plugins.xacro (robot description, xacro)
@@ -5,5 +5,5 @@
         <plugin name="joint_state_publisher" filename="libgazebo_ros_joint_state_publisher.so">
           <robotNamespace>${ns}</robotNamespace>
-          <jointName>chassis_swivel_joint, swivel_wheel_joint, left_hub_joint, right_hub_joint</jointName>
+          <jointName>front_swivel_joint, back_swivel_joint, front_swivel_wheel_joint, back_swivel_wheel_joint</jointName>
           <updateRate>10.0</updateRate>
           <alwaysOn>true</alwaysOn>
