Commit message: * copy internal branch to master working tree

File: tuw_gazebo_models/models/platforms/blue/blue.xacro (robot description, xacro)
@@ -11,17 +11,17 @@
     <xacro:property name="model_dir" value="$(arg model_dir)"/>
     <xacro:include filename="${model_dir}/blue_plugins.xacro" />
-    <xacro:BlueGazeboRosBridgePlugin        />
-    <xacro:BlueGazeboRosFlatControllerPlugin/>
+    <xacro:BlueGazeboRosModelBridgePlugin />
     <!-- Laser -->
     <xacro:property name="model_dir" value="$(find tuw_gazebo_models)/models/sensors/laser"/>
     <xacro:include filename="${model_dir}/Sick-LMS100.xacro"/>
-    <xacro:laser name="front_laser" parent="base_link" xyz="0 0.16 0.4" rpy="0 0 ${pi/2}" driver="cpu"/>
-    <!-- IMU -->
+    <xacro:laser name="front_laser" frame_names="front_laser" topic_names="front_laser/scan" parent="base_link" xyz="0.16 0 0.4" rpy="0 0 0" driver="cpu"/>
+    <!-- IMU
     <xacro:property name="model_dir" value="$(find tuw_gazebo_models)/models/sensors/imu"/>
     <xacro:include filename="$(find tuw_gazebo_models)/models/sensors/imu/imu.xacro"/>
-    <xacro:imu_sensor name="imu9dof" parent="base_link" xyz="0.0 0.05 0.262" rpy="0 0 ${pi/2}"/>
+    <xacro:imu_sensor name="imu9dof" parent="base_link" xyz=" 0.050.0 0.262" rpy="0 0 0"/>
+      -->
     <!-- Camera
-    <xacro:include filename="$(find blue_gazebo)/xacro/camera/camera.xacro"/>
-    <xacro:cam name="front_camera" parent="body" xyz="0 0 0.5" rpy="0 0 ${pi/2}"/>
-    -->
+    <xacro:include filename="$(find tuw_gazebo_models)/models/sensors/camera/camera.xacro"/>
+    <xacro:cam name="front_camera" parent="base_link" xyz="-0.5 0 0.7" rpy="${pi/2-0.2} ${pi} ${pi/2}"/>
+-->
 </robot>

File: tuw_gazebo_models/models/platforms/blue/blue_body/body.xacro (robot description, xacro)
@@ -9,8 +9,8 @@
     <xacro:BlueChassis name="${name}" parent="${parent}"/>
     <!-- Piston-Steering-Wheel modules -->
-    <Piston_SteerMnt_Steer_WheelMnt_Wheel fb="F" lr="R" parent="${name}" TransDirX= "1" TransDirY= "1" RotYaw="0"/>
-    <Piston_SteerMnt_Steer_WheelMnt_Wheel fb="F" lr="L" parent="${name}" TransDirX= "1" TransDirY="-1" RotYaw="0"/>
-    <Piston_SteerMnt_Steer_WheelMnt_Wheel fb="B" lr="R" parent="${name}" TransDirX="-1" TransDirY= "1" RotYaw="0"/>
-    <Piston_SteerMnt_Steer_WheelMnt_Wheel fb="B" lr="L" parent="${name}" TransDirX="-1" TransDirY="-1" RotYaw="0"/>
+    <Piston_SteerMnt_Steer_WheelMnt_Wheel fb="F" lr="R" parent="${name}" TransDirX= "1" TransDirY="-1" RotYaw="0"/>
+    <Piston_SteerMnt_Steer_WheelMnt_Wheel fb="F" lr="L" parent="${name}" TransDirX= "1" TransDirY= "1" RotYaw="0"/>
+    <Piston_SteerMnt_Steer_WheelMnt_Wheel fb="B" lr="L" parent="${name}" TransDirX="-1" TransDirY= "1" RotYaw="0"/>
+    <Piston_SteerMnt_Steer_WheelMnt_Wheel fb="B" lr="R" parent="${name}" TransDirX="-1" TransDirY="-1" RotYaw="0"/>
 </xacro:macro>
 </robot>

File: tuw_gazebo_models/models/platforms/blue/blue_body/chassis.xacro (robot description, xacro)
@@ -10,5 +10,5 @@
     </xacro:property>
     <xacro:property name="ThisLink2STL"> <!--this link 2 mesh center tf, file-->
-	<origin xyz="0 0   0" rpy="${pi/2} 0 ${pi}"/>
+	<origin xyz="0 0   0" rpy="${pi/2} 0 ${pi/2}"/>
 	<geometry> <mesh filename="file://${model_dir}/meshes/mobile_base_red.stl"/> </geometry>
 	<material name="light_blue"/>

File: tuw_gazebo_models/models/platforms/blue/blue_body/piston.xacro (robot description, xacro)
@@ -7,5 +7,5 @@
     <xacro:property name="z_ParrentLink2Piston_Link"  value="0.3400" />
     <xacro:property name="ParrentLink2ThisLink"> <!--parrent link to this joint tf-->
-	<origin xyz="${x_ParrentLink2Piston_Link*TransDirX} ${y_ParrentLink2Piston_Link*TransDirY} ${z_ParrentLink2Piston_Link}"  rpy="0 0 ${RotYaw}"/>
+	<origin xyz="${x_ParrentLink2Piston_Link*TransDirX} ${y_ParrentLink2Piston_Link*TransDirY} ${z_ParrentLink2Piston_Link}"  rpy="0 0 ${RotYaw-pi/2}"/>
     </xacro:property>
     <xacro:property name="ThisLink2Inert"> <!--this link 2 inertial center tf, mass data-->

File: tuw_gazebo_models/models/platforms/blue/blue_body/piston_steering_wheel.xacro (robot description, xacro)
@@ -13,5 +13,5 @@
 	<xacro:BlueSteeringMount name="${steering_mount_name}" fb="${fb}" lr="${lr}" parent="${piston_name}"        />
 	<xacro:BlueWheelMount    name="${wheel_mount_name}"    fb="${fb}" lr="${lr}" parent="${steering_mount_name}"/>
-	<xacro:BlueWheel         name="${wheel_name}"          fb="${fb}" lr="${lr}" parent="${wheel_mount_name}"   wheel_radius="0.05" wheel_length="0.001"/><!--0.025-->
+	<xacro:BlueWheel         name="${wheel_name}"          fb="${fb}" lr="${lr}" parent="${wheel_mount_name}"   wheel_radius="0.05" wheel_length="0.0005"/><!--0.025-->
 </xacro:macro>
 </robot>

File: tuw_gazebo_models/models/platforms/blue/blue_body/steering_mount.xacro (robot description, xacro)
@@ -4,16 +4,16 @@
 <xacro:macro name="BlueSteeringMount" params="name parent fb lr mesh_collis:=^|simplified mesh_visual:=^|detailed model_dir:=^">
     <xacro:property name="ParrentLink2ThisLink"> <!--parrent link to this joint tf-->
-	<origin xyz="0 0 0"  rpy="0 0 0"/>
+	<origin xyz="0 0 ${-0.309-0.060}"  rpy="0 0 0"/>
     </xacro:property>
     <xacro:property name="ThisLink2Inert"> <!--this link 2 inertial center tf, mass data-->
-	<cylinder_inertial_with_origin radius="0.04" length="0.1666" mass="0.251"> <origin xyz="0 0 -0.23" rpy="0 0 0"/> </cylinder_inertial_with_origin>
+	<cylinder_inertial_with_origin radius="0.04" length="0.1666" mass="0.251"> <origin xyz="0 0 ${-0.23+0.309+0.060}" rpy="0 0 0"/> </cylinder_inertial_with_origin>
     </xacro:property>
     <xacro:property name="ThisLink2STL"> <!--this link 2 mesh center tf, file-->
-	<origin xyz="0 0 -0.371" rpy="${-pi/2} 0 0"/>
+	<origin xyz="0 0 ${+0.309-0.371+0.060}" rpy="${-pi/2} 0 0"/>
 	<geometry> <mesh filename="file://${model_dir}/meshes/steering_mount_red.stl"/> </geometry>
 	<material name="red"/>
     </xacro:property>
     <xacro:property name="ThisLink2XML"> <!--this link 2 simple mesh center tf, file-->
-	<origin xyz="0 0 -0.23" rpy="0 0 0"/>
+	<origin xyz="0 0 ${-0.23+0.309+0.060}" rpy="0 0 0"/>
 	<geometry> <cylinder length="0.1666" radius="0.04"/> </geometry>
 	<material name="red"/>

File: tuw_gazebo_models/models/platforms/blue/blue_body/wheel.xacro (robot description, xacro)
@@ -4,5 +4,5 @@
 <xacro:macro name="BlueWheel" params="name parent fb lr wheel_radius wheel_length mesh_collis:=^|simplified mesh_visual:=^|detailed model_dir:=^">
     <xacro:property name="ParrentLink2ThisLink"> <!--parrent link to this joint tf-->
-	<origin xyz="0 0 -0.060"  rpy="0 ${pi/2} 0"/>
+	<origin xyz="0 0 0"  rpy="${pi} ${pi/2} 0"/>
     </xacro:property>
     <xacro:property name="ThisLink2Inert"> <!--this link 2 inertial center tf, mass data-->
@@ -10,5 +10,5 @@
     </xacro:property>
     <xacro:property name="ThisLink2STL"> <!--this link 2 mesh center tf, file-->
-	<origin xyz="0 0 0" rpy="0 -${pi/2} 0"/>
+	<origin xyz="0 0 0" rpy="0 ${pi/2} 0"/>
 	<geometry> <mesh filename="file://${model_dir}/meshes/wheel_red.stl"/> </geometry>
 	<material name="white"/>
@@ -42,5 +42,5 @@
 	<mu2 value="5.9"/>
 	<!--fdir1>0 0 1</fdir1-->
-	<minDepth value="0.002"/>
+	<minDepth value="0.0002"/>
 	<kp value="1000000.0"/>
 	<kd value="10.0"/>

File: tuw_gazebo_models/models/platforms/blue/blue_body/wheel_mount.xacro (robot description, xacro)
@@ -4,16 +4,16 @@
 <xacro:macro name="BlueWheelMount" params="name parent fb lr mesh_collis:=^|simplified mesh_visual:=^|detailed model_dir:=^">
     <xacro:property name="ParrentLink2ThisLink"> <!--parrent link to this joint tf-->
-	<origin xyz="0 0 -0.309"  rpy="0 0 0"/>
+	<origin xyz="0 0 0"  rpy="0 0 0"/>
     </xacro:property>
     <xacro:property name="ThisLink2Inert"> <!--this link 2 inertial center tf, mass data-->
-	<cylinder_inertial_with_origin radius="0.05" length="0.025" mass="0.197"> <origin xyz="0 0 -0.060" rpy="0 ${-pi/2} 0"/> </cylinder_inertial_with_origin>
+	<cylinder_inertial_with_origin radius="0.05" length="0.025" mass="0.197"> <origin xyz="0 0 0" rpy="0 ${-pi/2} 0"/> </cylinder_inertial_with_origin>
     </xacro:property>
     <xacro:property name="ThisLink2STL"> <!--this link 2 mesh center tf, file-->
-	<origin xyz="0 0 -0.060" rpy="${-pi/2} 0 0"/>
+	<origin xyz="0 0 0" rpy="${-pi/2} 0 0"/>
 	<geometry> <mesh filename="file://${model_dir}/meshes/wheel_mount_red.stl"/> </geometry>
 	<material name="orange"/>
     </xacro:property>
     <xacro:property name="ThisLink2XML"> <!--this link 2 simple mesh center tf, file-->
-	<origin xyz="0 0 -0.060" rpy="${-pi/2} 0 0"/>
+	<origin xyz="0 0 0" rpy="${-pi/2} 0 0"/>
 	<geometry> <box size="0.0001 0.0001 0.0001" /> </geometry>
 	<material name="orange"/>
@@ -31,5 +31,5 @@
 	<child  link="${name}${fb}${lr}_link"/>
 	<axis xyz=" 0 0 1"/>
-	<limit effort="12" velocity="12" lower= "${-M_PI}" upper="${M_PI}" /> <!--velocity="5" -->
+	<limit effort="50" velocity="50" lower= "${-M_PI}" upper="${M_PI}" /> <!--velocity="5" -->
 	<xacro:insert_block name="ParrentLink2ThisLink" />
     </joint>

File: tuw_gazebo_models/models/platforms/blue/blue_plugins.xacro (robot description, xacro)
@@ -2,16 +2,9 @@
 <robot xmlns:xacro="http://ros.org/wiki/xacro">
 <xacro:include filename="blue_plugins_param.xacro"/>
-<xacro:macro name="BlueGazeboRosBridgePlugin">
+<xacro:macro name="BlueGazeboRosModelBridgePlugin">
     <gazebo>
-        <plugin name="tuw_gazebo_ros_i4ws_bridge_plugin" filename="libtuw_gazebo_ros_i4ws_bridge_plugin.so">
+        <plugin name="tuw_gazebo_ros_bridge_model_plugin" filename="libtuw_gazebo_ros_bridge_model.so">
             <xacro:insert_block name="BlueGazeboPluginsData" />
         </plugin>
-    </gazebo>
-</xacro:macro>
-<xacro:macro name="BlueGazeboRosFlatControllerPlugin">
-    <gazebo>
-	<plugin name="tuw_gazebo_ros_iws_controller_plugin" filename="libtuw_gazebo_ros_iws_controller_plugin.so">
-	    <xacro:insert_block name="BlueGazeboPluginsData" />
-	</plugin>
     </gazebo>
 </xacro:macro>
@@ -20,8 +13,6 @@
 	<plugin name="joint_state_publisher" filename="libgazebo_ros_joint_state_publisher.so">
 	    <robotNamespace></robotNamespace>
-	    <jointName>  pistonFR2steermntFR_joint,   pistonFL2steermntFL_joint,   pistonBR2steermntBR_joint,   pistonBL2steermntBL_joint,
-		       steermntFR2wheelmntFR_joint, steermntFL2wheelmntFL_joint, steermntBR2wheelmntBR_joint, steermntBL2wheelmntBL_joint,
-			  wheelmntFR2wheelFR_joint,    wheelmntFL2wheelFL_joint,    wheelmntBR2wheelBR_joint,    wheelmntBL2wheelBL_joint  </jointName>
-	    <updateRate>10.0</updateRate>
+	    <!--jointName>  pistonFR2steermntFR_joint,   pistonFL2steermntFL_joint,   pistonBR2steermntBR_joint,   pistonBL2steermntBL_joint </jointName-->
+	    <updateRate>50.0</updateRate>
 	    <alwaysOn>true</alwaysOn>
 	</plugin>

File: tuw_gazebo_models/models/platforms/i2ws/i2ws.xacro (robot description, xacro)
@@ -11,10 +11,11 @@
     <xacro:property name="model_dir" value="$(arg model_dir)"/>
     <xacro:include filename="${model_dir}/i2ws_plugins.xacro" />
-    <xacro:BlueGazeboRosBridgePlugin        />
-    <!--xacro:BlueGazeboRosFlatControllerPlugin/-->
+    <xacro:I2wsRosBridgeModelPlugin/>
+    <xacro:i2ws_joints_state_publisher ns=""/>
+    <xacro:i2ws_joints_state_publisher ns="i2ws/ground_truth"/>
     <!-- Laser -->
     <xacro:property name="model_dir" value="$(find tuw_gazebo_models)/models/sensors/laser"/>
     <xacro:include filename="${model_dir}/Sick-LMS100.xacro"/>
-    <xacro:laser name="front_laser" parent="base_link" xyz="0.16 0  0.4" rpy="0 0 0" driver="gpu"/>
+    <xacro:laser name="front_laser" frame_names="front_laser" topic_names="front_laser/scan" parent="base_link" xyz="0.16 0  0.4" rpy="0 0 0" driver="cpu"/>
     <!-- IMU
     <xacro:property name="model_dir" value="$(find tuw_gazebo_models)/models/sensors/imu"/>

File: tuw_gazebo_models/models/platforms/i2ws/i2ws_body/body.xacro (robot description, xacro)
@@ -10,6 +10,6 @@
     <xacro:I2wsChassis name="${name}" parent="${parent}"/>
     <!-- Piston-Steering-Wheel modules -->
-    <Steer_WheelMnt_Wheel fb="F" lr="R" parent="${name}" TransDirX=  "1" TransDirY= "-1" RotYaw="0"/>
-    <Steer_WheelMnt_Wheel fb="B" lr="L" parent="${name}" TransDirX= "-1" TransDirY=  "1" RotYaw="0"/>
+    <Steer_WheelMnt_Wheel fb="F" lr="L" parent="${name}" TransDirX=  "1" TransDirY= "-1" RotYaw="0"/>
+    <Steer_WheelMnt_Wheel fb="B" lr="R" parent="${name}" TransDirX= "-1" TransDirY=  "1" RotYaw="0"/>
     <xacro:property name="swivel_contact_data">
       <mu1 value="0.7"/>
@@ -19,6 +19,6 @@
       <minDepth value="0.002"/>
     </xacro:property>
-    <Swivel fb="F" lr="L" parent="${name}" TransDirX=  "1" TransDirY=  "1" RotYaw="0"> <container> <xacro:insert_block name="swivel_contact_data"/> </container> </Swivel>
-    <Swivel fb="B" lr="R" parent="${name}" TransDirX= "-1" TransDirY= "-1" RotYaw="0"> <container> <xacro:insert_block name="swivel_contact_data"/> </container> </Swivel>
+    <Swivel fb="F" lr="R" parent="${name}" TransDirX=  "1" TransDirY=  "1" RotYaw="0"> <container> <xacro:insert_block name="swivel_contact_data"/> </container> </Swivel>
+    <Swivel fb="B" lr="L" parent="${name}" TransDirX= "-1" TransDirY= "-1" RotYaw="0"> <container> <xacro:insert_block name="swivel_contact_data"/> </container> </Swivel>
 </xacro:macro>
 </robot>

File: tuw_gazebo_models/models/platforms/i2ws/i2ws_body/chassis.xacro (robot description, xacro)
@@ -4,5 +4,5 @@
 <xacro:macro name="I2wsChassis" params="name parent mesh_collis:=^|simplified mesh_visual:=^|detailed model_dir:=^" >
     <xacro:property name="ParrentLink2ThisLink"> <!--parrent link to this joint tf-->
-	<origin xyz="0 0 0.07" rpy="0 0 ${-pi/2}"/>
+	<origin xyz="0 0 0.07" rpy="0 0 0"/>
     </xacro:property>
     <xacro:property name="ThisLink2Inert"> <!--this link 2 inertial center tf, mass data-->

File: tuw_gazebo_models/models/platforms/i2ws/i2ws_body/steering_mount.xacro (robot description, xacro)
@@ -5,18 +5,18 @@
     <xacro:property name="x_ParrentLink2Piston_Link"  value="0.1750" />
     <xacro:property name="y_ParrentLink2Piston_Link"  value="0.1744" />
-    <xacro:property name="z_ParrentLink2Piston_Link"  value="0.3400" />
+    <xacro:property name="z_ParrentLink2Piston_Link"  value="${0.3400-0.309-0.060}" />
     <xacro:property name="ParrentLink2ThisLink"> <!--parrent link to this joint tf-->
-	<origin xyz="${x_ParrentLink2Piston_Link*TransDirX} ${y_ParrentLink2Piston_Link*TransDirY} ${z_ParrentLink2Piston_Link}"  rpy="0 0 ${RotYaw}"/>
+	<origin xyz="${x_ParrentLink2Piston_Link*TransDirX} ${y_ParrentLink2Piston_Link*TransDirY} ${z_ParrentLink2Piston_Link}"  rpy="0 0 ${RotYaw-pi/2}"/>
     </xacro:property>
     <xacro:property name="ThisLink2Inert"> <!--this link 2 inertial center tf, mass data-->
-	<cylinder_inertial_with_origin radius="0.04" length="0.1666" mass="0.251"> <origin xyz="0 0 -0.23" rpy="0 0 0"/> </cylinder_inertial_with_origin>
+	<cylinder_inertial_with_origin radius="0.04" length="0.1666" mass="0.251"> <origin xyz="0 0 ${-0.23+0.309+0.060}" rpy="0 0 0"/> </cylinder_inertial_with_origin>
     </xacro:property>
     <xacro:property name="ThisLink2STL"> <!--this link 2 mesh center tf, file-->
-	<origin xyz="0 0 -0.371" rpy="${-pi/2} 0 0"/>
+	<origin xyz="0 0 ${+0.309-0.371+0.060}" rpy="${-pi/2} 0 0"/>
 	<geometry> <mesh filename="file://${model_dir}/meshes/steering_mount_red.stl"/> </geometry>
 	<material name="red"/>
     </xacro:property>
     <xacro:property name="ThisLink2XML"> <!--this link 2 simple mesh center tf, file-->
-	<origin xyz="0 0 -0.23" rpy="0 0 0"/>
+	<origin xyz="0 0 ${-0.23+0.309+0.060}" rpy="0 0 0"/>
 	<geometry> <cylinder length="0.1666" radius="0.04"/> </geometry>
 	<material name="red"/>

File: tuw_gazebo_models/models/platforms/i2ws/i2ws_body/wheel.xacro (robot description, xacro)
@@ -4,5 +4,5 @@
 <xacro:macro name="I2wsWheel" params="name parent fb lr wheel_radius wheel_length mesh_collis:=^|simplified mesh_visual:=^|detailed model_dir:=^">
     <xacro:property name="ParrentLink2ThisLink"> <!--parrent link to this joint tf-->
-	<origin xyz="0 0 -0.060"  rpy="0 ${pi/2} 0"/>
+	<origin xyz="0 0 0"  rpy="${pi} ${pi/2} 0"/>
     </xacro:property>
     <xacro:property name="ThisLink2Inert"> <!--this link 2 inertial center tf, mass data-->
@@ -10,5 +10,5 @@
     </xacro:property>
     <xacro:property name="ThisLink2STL"> <!--this link 2 mesh center tf, file-->
-	<origin xyz="0 0 0" rpy="0 -${pi/2} 0"/>
+	<origin xyz="0 0 0" rpy="0 ${pi/2} 0"/>
 	<geometry> <mesh filename="file://${model_dir}/meshes/wheel_red.stl"/> </geometry>
 	<material name="white"/>

File: tuw_gazebo_models/models/platforms/i2ws/i2ws_body/wheel_mount.xacro (robot description, xacro)
@@ -4,16 +4,16 @@
 <xacro:macro name="I2wsWheelMount" params="name parent fb lr mesh_collis:=^|simplified mesh_visual:=^|detailed model_dir:=^">
     <xacro:property name="ParrentLink2ThisLink"> <!--parrent link to this joint tf-->
-	<origin xyz="0 0 -0.309"  rpy="0 0 0"/>
+	<origin xyz="0 0 0"  rpy="0 0 0"/>
     </xacro:property>
     <xacro:property name="ThisLink2Inert"> <!--this link 2 inertial center tf, mass data-->
-	<cylinder_inertial_with_origin radius="0.05" length="0.025" mass="0.197"> <origin xyz="0 0 -0.060" rpy="0 ${-pi/2} 0"/> </cylinder_inertial_with_origin>
+	<cylinder_inertial_with_origin radius="0.05" length="0.025" mass="0.197"> <origin xyz="0 0 0" rpy="0 ${-pi/2} 0"/> </cylinder_inertial_with_origin>
     </xacro:property>
     <xacro:property name="ThisLink2STL"> <!--this link 2 mesh center tf, file-->
-	<origin xyz="0 0 -0.060" rpy="${-pi/2} 0 0"/>
+	<origin xyz="0 0 0" rpy="${-pi/2} 0 0"/>
 	<geometry> <mesh filename="file://${model_dir}/meshes/wheel_mount_red.stl"/> </geometry>
 	<material name="orange"/>
     </xacro:property>
     <xacro:property name="ThisLink2XML"> <!--this link 2 simple mesh center tf, file-->
-	<origin xyz="0 0 -0.060" rpy="${-pi/2} 0 0"/>
+	<origin xyz="0 0 0" rpy="${-pi/2} 0 0"/>
 	<geometry> <box size="0.0001 0.0001 0.0001" /> </geometry>
 	<material name="orange"/>

File: tuw_gazebo_models/models/platforms/i2ws/i2ws_plugins.xacro (robot description, xacro)
@@ -2,28 +2,18 @@
 <robot xmlns:xacro="http://ros.org/wiki/xacro">
 <xacro:include filename="i2ws_plugins_param.xacro"/>
-<xacro:macro name="BlueGazeboRosBridgePlugin">
+<xacro:macro name="I2wsRosBridgeModelPlugin">
     <gazebo>
-        <plugin name="tuw_gazebo_ros_i2ws_bridge_plugin" filename="libtuw_gazebo_ros_i2ws_bridge_plugin.so">
-            <xacro:insert_block name="BlueGazeboPluginsData" />
+        <plugin name="tuw_gazebo_ros_bridge_model_plugin" filename="libtuw_gazebo_ros_bridge_model.so">
+            <xacro:insert_block name="I2wsGazeboPluginsData" />
         </plugin>
     </gazebo>
 </xacro:macro>
-<xacro:macro name="BlueGazeboRosFlatControllerPlugin">
-    <gazebo>
-	<plugin name="tuw_gazebo_ros_i2ws_controller_plugin" filename="libtuw_gazebo_ros_i2ws_controller_plugin.so">
-	    <xacro:insert_block name="BlueGazeboPluginsData" />
-	</plugin>
-    </gazebo>
-</xacro:macro>
-<xacro:macro name="blue_joints_state_publisher">
+<xacro:macro name="i2ws_joints_state_publisher" params="ns">
     <gazebo>
 	<plugin name="joint_state_publisher" filename="libgazebo_ros_joint_state_publisher.so">
-	    <robotNamespace></robotNamespace>
-	    <jointName>  pistonFR2steermntFR_joint,   pistonBL2steermntBL_joint,
-		       steermntFR2wheelmntFR_joint, steermntBL2wheelmntBL_joint,
-			  wheelmntFR2wheelFR_joint,    wheelmntBL2wheelBL_joint,
-			  chassis_swivelFL_joint, swivelFL_wheel_joint,
-			  chassis_swivelBR_joint, swivelBR_wheel_joint</jointName>
-	    <updateRate>10.0</updateRate>
+	    <robotNamespace>${ns}</robotNamespace>
+	    <jointName>   chassis_swivelFR_joint, swivelFR_wheel_joint,
+			  chassis_swivelBL_joint, swivelBL_wheel_joint</jointName>
+	    <updateRate>50.0</updateRate>
 	    <alwaysOn>true</alwaysOn>
 	</plugin>
