Commit message: * copy internal branch to master working tree

File: tuw_gazebo_models/models/platforms/i2ws/i2ws_plugins_param.xacro (robot description, xacro)
@@ -1,23 +1,12 @@
 <?xml version="1.0"?>
 <robot xmlns:xacro="http://ros.org/wiki/xacro">
-<xacro:property name="BlueGazeboPluginsData">
+<xacro:property name="I2wsGazeboPluginsData">
 	<rosDebugLevel>Debug</rosDebugLevel>
 	<robotNamespace></robotNamespace>
-	<publishJointStates>true</publishJointStates>
-	<publishTfs>true</publishTfs>
-	<publishSimWorldOdom>true</publishSimWorldOdom>
+	<publish_joints_states>true</publish_joints_states>
+	<publish_tfs>false</publish_tfs>
 	<alwaysOn>true</alwaysOn>
 	<updateRate>100.0</updateRate>
-	<robotBaseFrame>base_link</robotBaseFrame>
-	<tr_piston_joint>pistonFR2steermntFR_joint</tr_piston_joint>
-	<bl_piston_joint>pistonBL2steermntBL_joint</bl_piston_joint>
-	<piston_hi_stop>       0.0</piston_hi_stop>
-	<piston_lo_stop>     -0.17</piston_lo_stop>
-	<piston_max_torque>    0.0</piston_max_torque>
-	<piston_max_vel>       0.0</piston_max_vel>
-	<piston_damping>       0.0</piston_damping>
-	<piston_friction>      0.0</piston_friction>
-	<tr_steering_joint>steermntFR2wheelmntFR_joint</tr_steering_joint>
-	<bl_steering_joint>steermntBL2wheelmntBL_joint</bl_steering_joint>
+	<steering_joints_names>steermntFL2wheelmntFL_joint, steermntBR2wheelmntBR_joint</steering_joints_names>
 	<steering_hi_stop>     2.70526034</steering_hi_stop>    <!-- rad -->
 	<steering_lo_stop>    -2.70526034</steering_lo_stop>    <!-- rad -->
@@ -26,17 +15,19 @@
 	<steering_damping>            0.1</steering_damping>    <!--Nms/rad-->
 	<steering_friction>           0.0</steering_friction>   <!--Nm   -->
-	<tr_wheel_joint>wheelmntFR2wheelFR_joint</tr_wheel_joint>
-	<bl_wheel_joint>wheelmntBL2wheelBL_joint</bl_wheel_joint>
-	<wheel_max_torque>           10.0</wheel_max_torque> <!-- Nm  -->
-	<wheel_max_vel>              10.0</wheel_max_vel>    <!--rad/s-->
-	<wheel_damping>               0.1</wheel_damping>    <!--Nms/rad-->
-	<wheel_friction>              0.0</wheel_friction>   <!--Nm   -->
-	<jointsStatesTopic>joint_states</jointsStatesTopic>
-	<jointsMeasurementsTopic>joint_measures</jointsMeasurementsTopic>
-	<baseCommandTopic>base_cmds</baseCommandTopic>
-	<jointsCommandTopic>joint_cmds</jointsCommandTopic>
-	<odometryTopic>odom</odometryTopic>
-	<odometryFrame>odom</odometryFrame>
-	<useForceControl>false</useForceControl>
+	<revolute_joints_names>wheelmntFL2wheelFL_joint, wheelmntBR2wheelBR_joint</revolute_joints_names>
+	<revolute_max_torque>        10.0</revolute_max_torque> <!-- Nm  -->
+	<revolute_max_vel>           50.0</revolute_max_vel>    <!--rad/s-->
+	<revolute_damping>            0.1</revolute_damping>    <!--Nms/rad-->
+	<revolute_friction>           0.0</revolute_friction>   <!--Nm   -->
+	<steering_measures_type>measured_position</steering_measures_type>
+	<revolute_measures_type>measured_velocity</revolute_measures_type>
+	<publish_odom_ground_truth>true</publish_odom_ground_truth>
+	<model_base_frame>ground_truth/base_link</model_base_frame>
+	<joints_states_topic>ground_truth/joint_states</joints_states_topic>
+	<odom_topic>ground_truth/odom</odom_topic>
+	<odom_frame>/map</odom_frame>
+	<joints_measures_topic>joint_measures</joints_measures_topic>
+	<base_cmd_topic>base_cmds</base_cmd_topic>
+	<joints_cmd_topic>joint_cmds</joints_cmd_topic>
 </xacro:property>
 </robot>

File: tuw_gazebo_models/models/platforms/pioneer3dx/pioneer3dx.xacro (robot description, xacro)
@@ -11,17 +11,23 @@
   <xacro:property name="model_dir" value="$(arg model_dir)"/>
   <xacro:include filename="${model_dir}/pioneer3dx_plugins.xacro" />
-  <xacro:pioneer3dx_diff_drive             /> <!-- Motor  plugin -->
-  <xacro:pioneer3dx_joints_state_publisher /> <!-- Joints plugin -->
+  <!--xacro:pioneer3dx_diff_drive             /--> <!-- Motor  plugin -->
+  <!--xacro:pioneer3dx_joints_state_publisher /--> <!-- Joints plugin -->
+  <xacro:P3dxRosBridgeModelPlugin/>
+  <xacro:p3dx_joints_state_publisher ns=""/>
+  <xacro:p3dx_joints_state_publisher ns="p3dx/ground_truth"/>
   <!-- Laser -->
   <xacro:property name="model_dir" value="$(find tuw_gazebo_models)/models/sensors/laser"/>
   <xacro:include filename="${model_dir}/hokuyo.xacro"/>
-  <xacro:laser name="front_laser" parent="chassis" xyz="0.16 0 0.125" rpy="0 0 0" driver="cpu"/>
-  <!-- IMU -->
+  <xacro:laser name="laser_front" frame_names="laser_front" topic_names="laser_front/scan" parent="top" xyz="0.17 0 0.04" rpy="0 0 0" driver="cpu"/>
+  <!-- xyz="0.16 0 0.125" -->
+  <!-- IMU
   <xacro:property name="model_dir" value="$(find tuw_gazebo_models)/models/sensors/imu"/>
   <xacro:include filename="$(find tuw_gazebo_models)/models/sensors/imu/imu.xacro"/>
   <xacro:imu_sensor name="imu9dof" parent="chassis" xyz="0.05 0.0 0.262" rpy="0 0 0"/>
-  <!-- Camera -->
+  -->
+  <!-- Camera
   <xacro:property name="model_dir" value="$(find tuw_gazebo_models)/models/sensors/camera"/>
   <xacro:include filename="${model_dir}/camera.xacro"/>
   <xacro:cam name="front_camera" parent="chassis" xyz="0 0 0.5" rpy="${-pi/2}  0 ${-pi/2}" />
+  -->
 </robot>

File: tuw_gazebo_models/models/platforms/pioneer3dx/pioneer3dx_body/body.xacro (robot description, xacro)
@@ -18,9 +18,9 @@
     <!-- Wheels -->
     <xacro:property name="contact_data">
-      <mu1 value="0.7"/>
-      <mu2 value="0.7"/>
-      <kp value="100000000.0"/>
-      <kd value="1000.0"/>
-      <minDepth value="0.002"/>
+        <mu1 value="5.9"/>
+	<mu2 value="5.9"/>
+	<minDepth value="0.002"/>
+	<kp value="1000000.0"/>
+	<kd value="10.0"/>
     </xacro:property>
     <xacro:pioneer_swivel             parent="${name}"  xyz="-0.185 0    0.055" rpy="0 0 0">               <container> <xacro:insert_block name="contact_data"/> </container> </xacro:pioneer_swivel>

File: tuw_gazebo_models/models/platforms/pioneer3dx/pioneer3dx_body/chassis.xacro (robot description, xacro)
@@ -32,5 +32,5 @@
   <!-- Top -->
   <joint name="${name}_top_joint" type="fixed">
-    <origin xyz="-0.045 0 0.234" rpy="0 0 0"/>
+    <origin xyz="-0.045 0 0.235" rpy="0 0 0"/>
     <parent link="${name}"/>
     <child link="top"/>

Commit message: better simulation model

File: tuw_gazebo_models/models/platforms/blue/blue.xacro (robot description, xacro)
@@ -16,4 +16,9 @@
     <xacro:include filename="${model_dir}/Sick-LMS100.xacro"/>
     <xacro:laser name="front_laser" frame_names="front_laser" topic_names="front_laser/scan" parent="base_link" xyz="0.16 0 0.4" rpy="0 0 0" driver="cpu"/>
+    <!--gazebo>
+	<plugin name="gazebo_ros_control" filename="libgazebo_ros_control.so">
+	    <robotNamespace>/blue</robotNamespace>
+	</plugin>
+    </gazebo-->
     <!-- IMU
     <xacro:property name="model_dir" value="$(find tuw_gazebo_models)/models/sensors/imu"/>

File: tuw_gazebo_models/models/platforms/blue/blue_body/wheel.xacro (robot description, xacro)
@@ -30,4 +30,5 @@
 	<axis   xyz="0 0 1"/>
 	<xacro:insert_block name="ParrentLink2ThisLink" />
+	<!--dynamics damping="0.7"/-->
     </joint>
     <link name="${name}${fb}${lr}_link">
@@ -39,6 +40,6 @@
 	<material>Gazebo/White</material>
 	<selfCollide>false</selfCollide>
-	<mu1 value="5.9"/>
-	<mu2 value="5.9"/>
+	<mu1 value="0.7"/>
+	<mu2 value="0.7"/>
 	<!--fdir1>0 0 1</fdir1-->
 	<minDepth value="0.0002"/>
@@ -46,4 +47,14 @@
 	<kd value="10.0"/>
     </gazebo>
+    <!--transmission name="trans_${name}${fb}${lr}">
+	<type>transmission_interface/SimpleTransmission</type>
+	<joint name="${parent}${fb}${lr}2${name}${fb}${lr}_joint">
+	    <hardwareInterface>EffortJointInterface</hardwareInterface>
+	</joint>
+	<actuator name="motor_${parent}${fb}${lr}2${name}${fb}${lr}">
+	    <hardwareInterface>EffortJointInterface</hardwareInterface>
+	    <mechanicalReduction>1</mechanicalReduction>
+	</actuator>
+    </transmission-->
 </xacro:macro>
 </robot>

File: tuw_gazebo_models/models/platforms/blue/blue_body/wheel_mount.xacro (robot description, xacro)
@@ -33,4 +33,5 @@
 	<limit effort="50" velocity="50" lower= "${-M_PI}" upper="${M_PI}" /> <!--velocity="5" -->
 	<xacro:insert_block name="ParrentLink2ThisLink" />
+	<!--dynamics damping="0.7"/-->
     </joint>
     <link name="${name}${fb}${lr}_link">
@@ -43,4 +44,14 @@
 	<selfCollide>false</selfCollide>
     </gazebo>
+    <!--transmission name="trans_${name}${fb}${lr}">
+	<type>transmission_interface/SimpleTransmission</type>
+	<joint name="${parent}${fb}${lr}2${name}${fb}${lr}_joint">
+	    <hardwareInterface>EffortJointInterface</hardwareInterface>
+	</joint>
+	<actuator name="motor_${parent}${fb}${lr}2${name}${fb}${lr}">
+	    <hardwareInterface>EffortJointInterface</hardwareInterface>
+	    <mechanicalReduction>1</mechanicalReduction>
+	</actuator>
+    </transmission-->
 </xacro:macro>
 </robot>

File: tuw_gazebo_models/models/platforms/blue/blue_plugins_param.xacro (robot description, xacro)
@@ -13,10 +13,10 @@
 	<steering_max_torque>        10.0</steering_max_torque> <!-- Nm  -->
 	<steering_max_vel>            5.0</steering_max_vel>    <!--rad/s-->
-	<steering_damping>            0.1</steering_damping>    <!--Nms/rad-->
+	<steering_damping>            0.7</steering_damping>    <!--Nms/rad-->
 	<steering_friction>           0.0</steering_friction>   <!--Nm   -->
 	<revolute_joints_names>wheelmntFL2wheelFL_joint, wheelmntBL2wheelBL_joint, wheelmntBR2wheelBR_joint, wheelmntFR2wheelFR_joint</revolute_joints_names>
 	<revolute_max_torque>        10.0</revolute_max_torque> <!-- Nm  -->
 	<revolute_max_vel>           50.0</revolute_max_vel>    <!--rad/s-->
-	<revolute_damping>            0.1</revolute_damping>    <!--Nms/rad-->
+	<revolute_damping>            0.7</revolute_damping>    <!--Nms/rad-->
 	<revolute_friction>           0.0</revolute_friction>   <!--Nm   -->
 	<steering_measures_type>measured_position</steering_measures_type>

Commit message: wall texture added and visulize fag on laser

File: tuw_gazebo_models/models/platforms/blue/blue.xacro (robot description, xacro)
@@ -15,5 +15,5 @@
     <xacro:property name="model_dir" value="$(find tuw_gazebo_models)/models/sensors/laser"/>
     <xacro:include filename="${model_dir}/Sick-LMS100.xacro"/>
-    <xacro:laser name="front_laser" frame_names="front_laser" topic_names="front_laser/scan" parent="base_link" xyz="0.16 0 0.4" rpy="0 0 0" driver="cpu"/>
+    <xacro:laser name="front_laser" frame_names="front_laser" topic_names="front_laser/scan" parent="base_link" xyz="0.16 0 0.4" rpy="0 0 0" driver="cpu"  visualize="true"/>
     <!--gazebo>
 	<plugin name="gazebo_ros_control" filename="libgazebo_ros_control.so">

File: tuw_gazebo_models/models/platforms/pioneer3dx/main.xacro (robot description, xacro)
@@ -31,9 +31,9 @@
   <xacro:property name="model_dir" value="$(find tuw_gazebo_models)/models/sensors/laser"/>
   <xacro:include filename="${model_dir}/hokuyo.xacro"/>
-  <xacro:laser name="laser_front_right" frame_names="laser_front_right" topic_names="laser_front_right/scan/raw" parent="top" xyz="0.06 -0.14 0.08" rpy="0 0 ${-pi/4}" driver="cpu"/>
+  <xacro:laser name="laser_front_right" frame_names="laser_front_right" topic_names="laser_front_right/scan/raw" parent="top" xyz="0.06 -0.14 0.08" rpy="0 0 ${-pi/4}" driver="cpu" visualize="true"/>
   <!-- Laser -->
   <xacro:property name="model_dir" value="$(find tuw_gazebo_models)/models/sensors/laser"/>
   <xacro:include filename="${model_dir}/Sick-LMS100.xacro"/>
-  <xacro:laser name="laser_front_center" frame_names="laser_front_center" topic_names="laser_front_center/scan/raw" parent="top" xyz="0.08 0.0 0.26" rpy="${pi} 0 0" driver="cpu"/>
+  <xacro:laser name="laser_front_center" frame_names="laser_front_center" topic_names="laser_front_center/scan/raw" parent="top" xyz="0.08 0.0 0.26" rpy="${pi} 0 0" driver="cpu" visualize="false"/>
   <!-- xyz="0.16 0 0.125" -->
   <!-- IMU

File: tuw_gazebo_models/models/platforms/sally/main.xacro (robot description, xacro)
@@ -36,5 +36,5 @@
   <xacro:property name="model_dir" value="$(find tuw_gazebo_models)/models/sensors/laser"/>
   <xacro:include filename="${model_dir}/Sick-LMS100.xacro"/>
-  <xacro:laser name="laser_front_center" frame_names="laser_front_center" topic_names="laser_front_center/scan" parent="top" xyz="0.25 0.0 -0.20" rpy="${pi} 0 0" driver="cpu"/>
+  <xacro:laser name="laser_front_center" frame_names="laser_front_center" topic_names="laser_front_center/scan" parent="top" xyz="0.25 0.0 -0.20" rpy="${pi} 0 0" driver="cpu" visualize="true"/>
   <!-- xyz="0.16 0 0.125" -->
   <!-- IMU

File: tuw_gazebo_models/models/sensors/laser/RPLidar.xacro (robot description, xacro)
@@ -2,5 +2,5 @@
 <robot xmlns:xacro="http://ros.org/wiki/xacro">
 <!-- Front Laser -->
-<xacro:macro name="laser" params="name frame_names topic_names xyz rpy driver:=cpu model_dir:=^" >
+<xacro:macro name="laser" params="name frame_names topic_names xyz rpy driver:=cpu visualize:=true model_dir:=^" >
     <xacro:if     value="${driver == 'gpu'}"> <xacro:property name="sensor_type" value="gpu_ray"/> <xacro:property name="driver_type" value="libtuw_gazebo_ros_gpu_laser.so"/> </xacro:if>
     <xacro:unless value="${driver == 'gpu'}"> <xacro:property name="sensor_type" value="ray"    /> <xacro:property name="driver_type" value="libtuw_gazebo_ros_laser.so"    /> </xacro:unless>
@@ -34,5 +34,5 @@
 	    <pose>0 0 0 0 0 0</pose>
 	    <update_rate>5.5</update_rate>
-	    <visualize>true</visualize>
+	    <visualize>${visualize}</visualize>
 	    <always_on>1</always_on>
 	    <ray>

File: tuw_gazebo_models/models/sensors/laser/Sick-LMS100.xacro (robot description, xacro)
@@ -2,5 +2,5 @@
 <robot xmlns:xacro="http://ros.org/wiki/xacro">
 <!-- Front Laser -->
-<xacro:macro name="laser" params="name frame_names topic_names parent xyz rpy driver:=cpu model_dir:=^">
+<xacro:macro name="laser" params="name frame_names topic_names parent xyz rpy driver:=cpu visualize:=true model_dir:=^">
     <xacro:if     value="${driver == 'gpu'}"> <xacro:property name="sensor_type" value="gpu_ray"/> <xacro:property name="driver_type" value="libtuw_gazebo_ros_gpu_laser.so"/> </xacro:if>
     <xacro:unless value="${driver == 'gpu'}"> <xacro:property name="sensor_type" value="ray"    /> <xacro:property name="driver_type" value="libtuw_gazebo_ros_laser.so"    /> </xacro:unless>
@@ -41,5 +41,5 @@
 	    <update_rate>25</update_rate>
 	    <always_on>1</always_on>
-	    <visualize>false</visualize>
+	    <visualize>${visualize}</visualize>
 	    <ray>
 		<scan>

File: tuw_gazebo_models/models/sensors/laser/hokuyo.xacro (robot description, xacro)
@@ -2,5 +2,5 @@
 <robot xmlns:xacro="http://ros.org/wiki/xacro">
 <!-- Front Laser -->
-<xacro:macro name="laser" params="name frame_names topic_names parent xyz rpy driver:=cpu model_dir:=^" >
+<xacro:macro name="laser" params="name frame_names topic_names parent xyz rpy driver:=cpu visualize:=true model_dir:=^" >
     <xacro:if     value="${driver == 'gpu'}"> <xacro:property name="sensor_type" value="gpu_ray"/> <xacro:property name="driver_type" value="libtuw_gazebo_ros_gpu_laser.so"/> </xacro:if>
     <xacro:unless value="${driver == 'gpu'}"> <xacro:property name="sensor_type" value="ray"    /> <xacro:property name="driver_type" value="libtuw_gazebo_ros_laser.so"    /> </xacro:unless>
@@ -34,5 +34,5 @@
 	    <pose>0 0 0 0 0 0</pose>
 	    <update_rate>10</update_rate>
-	    <visualize>true</visualize>
+	    <visualize>${visualize}</visualize>
 	    <always_on>1</always_on>
 	    <ray>

File: tuw_gazebo_models/models/sensors/laser/hokuyo_30LX.xacro (robot description, xacro)
@@ -2,5 +2,5 @@
 <robot xmlns:xacro="http://ros.org/wiki/xacro">
   <!-- Front Laser -->
-  <xacro:macro name="laser" params="name frame_names topic_names parent xyz rpy max_angle:=2.3562 driver:=cpu model_dir:=^">
+  <xacro:macro name="laser" params="name frame_names topic_names parent xyz rpy max_angle:=2.3562 driver:=cpu visualize:=true model_dir:=^">
     <xacro:if value="${driver == 'gpu'}">
       <xacro:property name="sensor_type" value="gpu_ray"/>
@@ -40,5 +40,5 @@
         <pose>0 0 0 0 0 0</pose>
         <update_rate>40</update_rate>
-        <visualize>true</visualize>
+        <visualize>${visualize}</visualize>
         <always_on>1</always_on>
         <ray>
