Commit message: sally model fixed

File: tuw_gazebo_models/models/platforms/pioneer3dx/body/chassis.xacro (robot description, xacro)
@@ -13,5 +13,5 @@
       <origin xyz="-0.045 0 0.085" rpy="0 0 0"/>
       <geometry>
-	<mesh filename="file://${model_dir}/meshes/chassis.dae"/>
+        <mesh filename="file://${model_dir}/meshes/chassis.dae"/>
       </geometry>
       <material name="ChassisRed">
@@ -21,11 +21,15 @@
     <collision>
       <origin xyz="0.01 0 0.09" rpy="0 0 0"/>
-      <geometry><cylinder radius="0.17" length="0.17"/> </geometry>
+      <geometry>
+          <cylinder radius="0.17" length="0.17"/>
+      </geometry>
       <!--origin xyz="-0.045 0 0.148" rpy="0 0 0"/>
       <geometry>
-	<mesh filename="file://${model_dir}/meshes/chassis.dae"/>
+        <mesh filename="file://${model_dir}/meshes/chassis.dae"/>
       </geometry-->
     </collision>
-    <box_inertial_with_origin x="0.35" y="0.25"  z="0.17" mass="9.0"> <origin xyz="-0.04 0 0.15" rpy="0 0 0"/> </box_inertial_with_origin>
+    <box_inertial_with_origin x="0.35" y="0.25"  z="0.17" mass="9.0">
+        <origin xyz="-0.04 0 0.15" rpy="0 0 0"/>
+    </box_inertial_with_origin>
   </link>
   <gazebo reference="${name}">

File: tuw_gazebo_models/models/platforms/sally/body/body.xacro (robot description, xacro)
@@ -11,5 +11,5 @@
     <link name="${parent}"/>
     <!-- Chassis -->
-    <xacro:chassis name="${name}" parent="${parent}" xyz="0 0 0.068" rpy="0 0 0"/>
+    <xacro:sally_chassis name="${name}" parent="${parent}" xyz="0 0 0.068" rpy="0 0 0"/>
     <!-- Akku0 -->
     <xacro:battery_block name="battery0" parent="${name}" x="-0.14" y="0.00"  z="${0.13-0.068}" mass="2.5" />
@@ -22,8 +22,24 @@
 	<!--kd value="10.0"/-->
     </xacro:property>
-    <xacro:swivel side="front" parent="${parent}"  xyz=" 0.200 0    0.055" rpy="0 0 0">               <container> <xacro:insert_block name="contact_data"/> </container> </xacro:swivel>
-    <xacro:swivel side="back"  parent="${parent}"  xyz="-0.200 0    0.055" rpy="0 0 0">               <container> <xacro:insert_block name="contact_data"/> </container> </xacro:swivel>
-    <xacro:wheel  side="right" parent="${parent}"  xyz=" 0    -0.225 ${wheel_radius}" rpy="0 0 0" radius="${wheel_radius}"> <container> <xacro:insert_block name="contact_data"/> </container> </xacro:wheel>
-    <xacro:wheel  side="left"  parent="${parent}"  xyz=" 0     0.225 ${wheel_radius}" rpy="0 0 0" radius="${wheel_radius}"> <container> <xacro:insert_block name="contact_data"/> </container> </xacro:wheel>
+    <xacro:swivel side="front" parent="${parent}"  xyz=" 0.200 0    0.055" rpy="0 0 0">
+        <container>
+            <xacro:insert_block name="contact_data"/>
+        </container>
+    </xacro:swivel>
+    <xacro:swivel side="back"  parent="${parent}"  xyz="-0.200 0    0.055" rpy="0 0 0">
+        <container>
+            <xacro:insert_block name="contact_data"/>
+        </container>
+    </xacro:swivel>
+    <xacro:wheel  side="right" parent="${parent}"  xyz=" 0    -0.225 ${wheel_radius}" rpy="0 0 0" radius="${wheel_radius}">
+        <container>
+            <xacro:insert_block name="contact_data"/>
+        </container>
+    </xacro:wheel>
+    <xacro:wheel  side="left"  parent="${parent}"  xyz=" 0     0.225 ${wheel_radius}" rpy="0 0 0" radius="${wheel_radius}">
+        <container>
+            <xacro:insert_block name="contact_data"/>
+        </container>
+    </xacro:wheel>
   </xacro:macro>
 </robot>

File: tuw_gazebo_models/models/platforms/sally/body/chassis.xacro (robot description, xacro)
@@ -2,8 +2,5 @@
 <robot xmlns:xacro="http://ros.org/wiki/xacro">
   <xacro:property name="M_PI" value="3.1415926535897931" />
-  <xacro:macro name="chassis" params="name parent xyz rpy model_dir:=^">
-    <material name="SallyWhite">
-	<color rgba="${200/255} ${200/255} ${200/255} 1.0"/>
-    </material>
+  <xacro:macro name="sally_chassis" params="name parent xyz rpy model_dir:=^">
   <!-- Chassis -->
   <joint name="${parent}_${name}_joint" type="fixed">
@@ -16,7 +13,8 @@
       <origin xyz="-0.0 0 -0.04" rpy="0 0 0"/>
       <geometry>
-	<mesh filename="file://${model_dir}/meshes/chassis.dae"/>
+        <mesh filename="file://${model_dir}/meshes/chassis.dae"/>
       </geometry>
       <material name="SallyWhite">
+        <color rgba="${200/255} ${200/255} ${200/255} 1.0"/>
       </material>
     </visual>
@@ -24,12 +22,14 @@
       <origin xyz="-0.0 0 -0.04" rpy="0 0 0"/>
       <geometry>
-	  <mesh filename="file://${model_dir}/meshes/chassis.dae"/>>
+        <mesh filename="file://${model_dir}/meshes/chassis.dae"/>>
       </geometry>
       <!--origin xyz="-0.045 0 0.148" rpy="0 0 0"/>
       <geometry>
-	<mesh filename="file://${model_dir}/meshes/chassis.dae"/>
+        <mesh filename="file://${model_dir}/meshes/chassis.dae"/>
       </geometry-->
     </collision>
-    <box_inertial_with_origin x="0.35" y="0.25"  z="0.17" mass="9.0"> <origin xyz="-0.04 0 0.15" rpy="0 0 0"/> </box_inertial_with_origin>
+    <box_inertial_with_origin x="0.35" y="0.25"  z="0.17" mass="9.0">
+        <origin xyz="-0.04 0 0.15" rpy="0 0 0"/>
+    </box_inertial_with_origin>
   </link>
   <!-- Top -->

File: tuw_gazebo_models/models/platforms/sally/main.xacro (robot description, xacro)
@@ -2,5 +2,5 @@
 <robot xmlns:xacro="http://ros.org/wiki/xacro" name="sally" >
   <xacro:arg name="model_dir"   default="$(find tuw_gazebo_models)/models/platforms/sally"/>
-  <xacro:arg name="namespace"   default="sally"/>
+  <xacro:arg name="namespace"   default="r1"/>
   <xacro:arg name="motor_plugin" default="diff_twist"/> <!-- diffdrive or iws. If something else is set, no plugin will be loaded-->
   <!-- Import Rviz colors -->
