Commit message: updates on launch and models

File: tuw_gazebo_models/models/platforms/pioneer3dx/body/body.xacro (robot description, xacro)
@@ -4,10 +4,10 @@
   <xacro:include filename="chassis.xacro"/>
   <xacro:include filename="mount.xacro"/>
+  <xacro:include filename="wheel.xacro"/>
   <xacro:include filename="battery_block.xacro"/>
-  <xacro:include filename="wheel.xacro"/>
   <xacro:include filename="swivel.xacro"/>
   <xacro:include filename="sonar.xacro"/>
   <xacro:property name="wheel_radius" value="0.097" />
-  <xacro:macro name="pioneer3dx_body" params="name parent">
+  <xacro:macro name="vehicle_body" params="name parent">
     <!-- base_link -->
     <link name="${parent}"/>
@@ -23,10 +23,12 @@
     <xacro:property name="contact_data">
         <mu1 value="0.7"/>
-	<mu2 value="0.7"/>
-	<minDepth value="0.002"/>
-	<!--kp value="1000000.0"/-->
-	<!--kd value="10.0"/-->
+        <mu2 value="0.7"/>
+        <minDepth value="0.002"/>
+        <!--kp value="1000000.0"/-->
+        <!--kd value="10.0"/-->
     </xacro:property>
+    <!-- Swivels -->
     <xacro:pioneer_swivel             parent="${parent}"  xyz="-0.185 0    0.0535" rpy="0 0 0">               <container> <xacro:insert_block name="contact_data"/> </container> </xacro:pioneer_swivel>
+    <!-- Wheels -->
     <xacro:pioneer_wheel side="right" parent="${parent}"  xyz=" 0    -0.165 ${wheel_radius}" rpy="0 0 0" radius="${wheel_radius}"> <container> <xacro:insert_block name="contact_data"/> </container> </xacro:pioneer_wheel>
     <xacro:pioneer_wheel side="left"  parent="${parent}"  xyz=" 0     0.165 ${wheel_radius}" rpy="0 0 0" radius="${wheel_radius}"> <container> <xacro:insert_block name="contact_data"/> </container> </xacro:pioneer_wheel>

File: tuw_gazebo_models/models/platforms/pioneer3dx/main.xacro (robot description, xacro)
@@ -3,6 +3,6 @@
   <xacro:arg name="model_dir"      default=""/>
   <xacro:arg name="platform_dir"   default=""/>
-  <xacro:arg name="namespace"      default="r1"/>
-  <xacro:arg name="motor_plugin" default="diff_twist"/> <!-- diffdrive or iws. If something else is set, no plugin will be loaded-->
+  <xacro:arg name="namespace"      default="r0"/>
+  <xacro:arg name="motor_plugin"   default="diff_twist"/> <!-- diffdrive or diff_iws. If something else is set, no plugin will be loaded-->
   <!-- Import Rviz colors -->
   <xacro:include filename="$(arg model_dir)/materials.xacro" />
@@ -10,5 +10,5 @@
   <xacro:property name="model_dir" value="$(arg model_dir)/$(arg platform_dir)/body"/>
   <xacro:include filename="${model_dir}/body.xacro"/>
-  <xacro:pioneer3dx_body name="chassis" parent="base_link"/>
+  <xacro:vehicle_body name="chassis" parent="base_link"/>
   <!-- Import platform plugins -->
   <xacro:property name="model_dir"   value="$(arg model_dir)/$(arg platform_dir)"/>
@@ -27,14 +27,14 @@
     <xacro:differential_drive/>
     <!-- Joints plugin -->
-	<xacro:diff_joints_state_publisher ns="${namespace}"/>
+    <xacro:diff_joints_state_publisher ns="${namespace}"/>
   </xacro:if>
   <!-- Laser -->
   <xacro:property name="model_dir" value="$(arg model_dir)/sensors/laser"/>
   <xacro:include filename="${model_dir}/hokuyo.xacro"/>
-  <xacro:laser name="laser0" frame_names="laser0" topic_names="laser_front_center/scan/raw" parent="top" xyz="0.15 0.0 0.06" rpy="0 0 0" driver="cpu" visualize="true"/>
+  <xacro:laser name="laser0" frame_names="laser0" topic_names="laser0/scan/raw" parent="top" xyz="0.15 0.0 0.06" rpy="0 0 0" driver="cpu" visualize="true"/>
   <!-- Laser -->
   <xacro:property name="model_dir" value="$(arg model_dir)/sensors/laser"/>
   <xacro:include filename="${model_dir}/Sick-LMS100.xacro"/>
-  <xacro:laser name="laser1" frame_names="laser1" topic_names="laser_front_top/scan/raw" parent="top" xyz="0.08 0.0 0.26" rpy="${pi} 0 0" driver="cpu" visualize="false"/>
+  <xacro:laser name="laser1" frame_names="laser1" topic_names="laser1/scan/raw" parent="top" xyz="0.08 0.0 0.26" rpy="${pi} 0 0" driver="cpu" visualize="false"/>
   <!-- xyz="0.16 0 0.125" -->
   <!-- IMU
