Commit message: inertia problem workaround

File: tuw_gazebo_models/models/platforms/pioneer3dx/body/swivel.xacro (robot description, xacro)
@@ -14,10 +14,9 @@
   </joint>
   <link name="swivel">
-    <box_inertial_with_origin x="0.07" y="0.07" z="0.05" mass="0.1"> <origin xyz="0 0 0" rpy="0 0 0"/> </box_inertial_with_origin>
-    <!--inertial>
+    <inertial>
       <mass value="0.1"/>
       <origin xyz="0 0 0"/>
       <inertia ixx="0.01" ixy="0" ixz="0" iyy="0.01" iyz="0" izz="0.01"/>
-    </inertial-->
+    </inertial>
     <visual>
       <origin xyz="0 0 0" rpy="0 0 0"/>
@@ -50,10 +49,9 @@
   </joint>
   <link name="center_wheel">
-    <cylinder_inertial_with_origin radius="0.0375" length="0.03" mass="0.1"> <origin xyz="0 0 0" rpy="${pi/2} 0 0"/> </cylinder_inertial_with_origin>
-    <!--inertial>
+    <inertial>
       <mass value="0.1"/>
       <origin xyz="0 0 0"/>
       <inertia ixx="0.012411765597" ixy="-0.000711733678" ixz="0.00050272983" iyy="0.015218160428" iyz="-0.000004273467" izz="0.011763977943"/>
-    </inertial-->
+    </inertial>
     <visual>
       <origin xyz="0 0 0" rpy="0 0 0"/>
@@ -84,10 +82,9 @@
   </joint>
   <link name="center_hubcap">
-    <cylinder_inertial_with_origin radius="0.01" length="0.03" mass="0.01"> <origin xyz="0 0 0" rpy="${pi/2} 0 0"/> </cylinder_inertial_with_origin>
-    <!--inertial>
+    <inertial>
       <mass value="0.01"/>
       <origin xyz="0 0 0"/>
       <inertia ixx="0.012411765597" ixy="-0.000711733678" ixz="0.00050272983" iyy="0.015218160428" iyz="-0.000004273467" izz="0.011763977943"/>
-    </inertial-->
+    </inertial>
     <visual>
       <origin xyz="0 0 0" rpy="0 0 0"/>

File: tuw_gazebo_models/models/platforms/pioneer3dx/body/wheel.xacro (robot description, xacro)
@@ -12,5 +12,9 @@
     </joint>
     <link name="${side}_hub_mount">
-	<cylinder_inertial_with_origin radius="0.01" length="0.01" mass="0.01"> <origin xyz="0 0 0" rpy="0 0 0"/> </cylinder_inertial_with_origin>
+    <inertial>
+      <mass value="0.01"/>
+      <origin xyz="0 0 0"/>
+      <inertia ixx="0.012411765597" ixy="0" ixz="0" iyy="0.015218160428" iyz="0" izz="0.011763977943"/>
+    </inertial>
 	<visual>
 	    <origin xyz="0 0 0" rpy="0 0 0"/>
@@ -30,5 +34,9 @@
     </joint>
     <link name="${side}_hub">
-	<cylinder_inertial_with_origin radius="${radius}" length="0.03" mass="0.5"> <origin xyz="0 0 0" rpy="${pi/2} 0 0"/> </cylinder_inertial_with_origin>
+    <inertial>
+      <mass value="0.01"/>
+      <origin xyz="0 0 0"/>
+      <inertia ixx="0.012411765597" ixy="0" ixz="0" iyy="0.015218160428" iyz="0" izz="0.011763977943"/>
+    </inertial>
 	<visual>
 	    <origin xyz="0 0 0" rpy="0 0 0"/>
@@ -52,5 +60,9 @@
     </joint>
     <link name="${side}_wheel">
-	<cylinder_inertial_with_origin radius="${radius}" length="0.03" mass="0.5"> <origin xyz="0 0 0" rpy="${pi/2} 0 0"/> </cylinder_inertial_with_origin>
+    <inertial>
+      <mass value="0.5"/>
+      <origin xyz="0 0 0"/>
+      <inertia ixx="0.012411765597" ixy="0" ixz="0" iyy="0.015218160428" iyz="0" izz="0.011763977943"/>
+    </inertial>
 	<visual>
 	    <origin xyz="0 0 0" rpy="0 0 0"/>

File: tuw_gazebo_models/models/platforms/pioneer3dx/main.xacro (robot description, xacro)
@@ -52,6 +52,4 @@
     </VLP-16>
   </xacro:if>
-    <xacro:include filename="$(find tuw_gazebo_models)/models/sensors/imu/imu_sensor.xacro"/>
-    <xacro:imu_sensor name="imu" parent="top" topic="imu" xyz="0.0 0.0 0.1" rpy="0 0 0" />
   <!-- Laser
   <xacro:property name="model_dir" value="$(arg model_dir)/sensors/laser"/>
