Commit message: model transportbuddy update

File: tuw_gazebo_models/models/platforms/TransportBuddy/body/body.xacro (robot description, xacro)
@@ -13,5 +13,5 @@
     <!-- Camera -->
     <xacro:sensor_zr300 parent="${parent}">
-      <origin xyz="-0.240 0 1.145" rpy="0 0 0"/>
+      <origin xyz="-0.240 0 1.160" rpy="0 0 0"/>
     </xacro:sensor_zr300>
     <!-- Chassis -->

Commit message: sally model update

File: tuw_gazebo_models/models/platforms/TransportBuddy/body/body.xacro (robot description, xacro)
@@ -13,5 +13,5 @@
     <!-- Camera -->
     <xacro:sensor_zr300 parent="${parent}">
-      <origin xyz="-0.240 0 1.160" rpy="0 0 0"/>
+      <origin xyz="-0.220 0 1.300" rpy="0 0.20 0"/>
     </xacro:sensor_zr300>
     <!-- Chassis -->

File: tuw_gazebo_models/models/platforms/sally/main.xacro (robot description, xacro)
@@ -1,5 +1,6 @@
 <?xml version="1.0"?>
 <robot xmlns:xacro="http://ros.org/wiki/xacro" name="sally" >
-  <xacro:arg name="model_dir"   default="$(find tuw_gazebo_models)/models/platforms/sally"/>
+  <xacro:arg name="model_dir"   default="$(find tuw_gazebo_models)/models"/>
+  <xacro:arg name="platform_dir"   default="/platforms/sally"/>
   <xacro:arg name="namespace"   default="r1"/>
   <xacro:arg name="motor_plugin" default="diff_twist"/> <!-- diffdrive or iws. If something else is set, no plugin will be loaded-->
@@ -7,5 +8,5 @@
   <xacro:include filename="$(find tuw_gazebo_models)/models/materials.xacro" />
   <!-- Import platform -->
-  <xacro:property name="model_dir" value="$(arg model_dir)/body"/>
+  <xacro:property name="model_dir" value="$(arg model_dir)$(arg platform_dir)/body"/>
   <xacro:include filename="${model_dir}/body.xacro"/>
   <xacro:sally_body name="chassis" parent="base_link"/>
@@ -14,5 +15,5 @@
   <xacro:property name="namespace"   value="$(arg namespace)"/>
   <xacro:property name="motor_plugin" value="$(arg motor_plugin)"/>
-  <xacro:include filename="${model_dir}/plugins.xacro" />
+  <xacro:include filename="${model_dir}$(arg platform_dir)/plugins.xacro" />
   <xacro:if value="${motor_plugin == 'diff_iws'}">
     <!-- Motor  plugin -->
@@ -29,25 +30,25 @@
   </xacro:if>
   <!-- Laser
-  <xacro:property name="model_dir" value="$(find tuw_gazebo_models)/models/sensors/laser"/>
+  <xacro:property name="model_dir" value="$(arg model_dir)/sensors/laser"/>
   <xacro:include filename="${model_dir}/hokuyo.xacro"/>
   <xacro:laser name="laser_front_right" frame_names="laser_front_right" topic_names="laser_front_right/scan" parent="top" xyz="0.06 -0.14 0.08" rpy="0 0 ${-pi/4}" driver="cpu"/>
    -->
   <!-- Laser -->
-  <xacro:property name="model_dir" value="$(find tuw_gazebo_models)/models/sensors/laser"/>
+  <xacro:property name="model_dir" value="$(arg model_dir)/sensors/laser"/>
   <xacro:include filename="${model_dir}/Sick-LMS100.xacro"/>
   <xacro:laser name="laser_front_center" frame_names="laser_front_center" topic_names="laser_front_center/scan" parent="top" xyz="0.25 0.0 -0.20" rpy="${pi} 0 0" driver="cpu" visualize="true"/>
   <!-- xyz="0.16 0 0.125" -->
   <!-- IMU
-  <xacro:property name="model_dir" value="$(find tuw_gazebo_models)/models/sensors/imu"/>
-  <xacro:include filename="$(find tuw_gazebo_models)/models/sensors/imu/imu.xacro"/>
+  <xacro:property name="model_dir" value="$(arg model_dir)/sensors/imu"/>
+  <xacro:include filename="$(arg model_dir)/models/sensors/imu/imu.xacro"/>
   <xacro:imu_sensor name="imu9dof" parent="chassis" xyz="0.05 0.0 0.262" rpy="0 0 0"/>
   -->
   <!-- Camera
-  <xacro:property name="model_dir" value="$(find tuw_gazebo_models)/models/sensors/camera"/>
+  <xacro:property name="model_dir" value="$(arg model_dir)/sensors/camera"/>
   <xacro:include filename="${model_dir}/camera.xacro"/>
   <xacro:cam name="front_camera" parent="top" xyz="0 0 1" rpy="${-pi/2}  0 ${-pi/2}" />
    -->
   <!-- Depth Camera
-  <xacro:property name="model_dir" value="$(find tuw_gazebo_models)/models/sensors/camera"/>
+  <xacro:property name="model_dir" value="$(arg model_dir)/sensors/camera"/>
   <xacro:include filename="${model_dir}/depth_camera.xacro"/>
   <xacro:cam name="front_depth_camera" parent="top" xyz="0 0 1" rpy="0  0 0" />

Commit message: TransportBuddy model

File: tuw_gazebo_models/models/platforms/TransportBuddy/body/body.xacro (robot description, xacro)
@@ -8,5 +8,5 @@
   <xacro:include filename="zr300.xacro" />
   <xacro:property name="wheel_radius" value="0.104" />
-  <xacro:macro name="sally_body" params="name parent">
+  <xacro:macro name="vehicle_body" params="name parent">
     <!-- base_link -->
     <link name="${parent}"/>

File: tuw_gazebo_models/models/platforms/TransportBuddy/main.xacro (robot description, xacro)
@@ -1,15 +1,16 @@
 <?xml version="1.0"?>
 <robot xmlns:xacro="http://ros.org/wiki/xacro" name="TransportBuddy" >
-  <xacro:arg name="model_dir"   default="$(find tuw_gazebo_models)/models/platforms/TransportBuddy"/>
-  <xacro:arg name="namespace"   default="TransportBuddy"/>
-  <xacro:arg name="motor_plugin" default="diff_twist"/> <!-- diffdrive or iws. If something else is set, no plugin will be loaded-->
+  <xacro:arg name="model_dir"      default=""/>
+  <xacro:arg name="platform_dir"   default=""/>
+  <xacro:arg name="namespace"      default="r0"/>
+  <xacro:arg name="motor_plugin"   default="diff_twist"/> <!-- diffdrive or diff_iws. If something else is set, no plugin will be loaded-->
   <!-- Import Rviz colors -->
-  <xacro:include filename="$(find tuw_gazebo_models)/models/materials.xacro" />
+  <xacro:include filename="$(arg model_dir)/materials.xacro" />
   <!-- Import platform -->
-  <xacro:property name="model_dir" value="$(arg model_dir)/body"/>
+  <xacro:property name="model_dir" value="$(arg model_dir)/$(arg platform_dir)/body"/>
   <xacro:include filename="${model_dir}/body.xacro"/>
-  <xacro:sally_body name="chassis" parent="base_link"/>
+  <xacro:vehicle_body name="chassis" parent="base_link"/>
   <!-- Import platform plugins -->
-  <xacro:property name="model_dir"   value="$(arg model_dir)"/>
+  <xacro:property name="model_dir"   value="$(arg model_dir)/$(arg platform_dir)"/>
   <xacro:property name="namespace"   value="$(arg namespace)"/>
   <xacro:property name="motor_plugin" value="$(arg motor_plugin)"/>
@@ -18,5 +19,5 @@
     <!-- Motor  plugin -->
     <xacro:iws_drive/>
-    <!-- Joints plugin-->
+    <!-- Joints plugin -->
     <xacro:iws_joints_state_publisher ns=""/>
     <xacro:iws_joints_state_publisher ns="${namespace}/ground_truth"/>
@@ -26,30 +27,26 @@
     <xacro:differential_drive/>
     <!-- Joints plugin -->
-    <xacro:diff_joints_state_publisher ns=""/>
+    <xacro:diff_joints_state_publisher ns="${namespace}"/>
   </xacro:if>
   <!-- camera plugin -->
   <xacro:camera_zr300_rgb />
   <!-- Laser
-  <xacro:property name="model_dir" value="$(find tuw_gazebo_models)/models/sensors/laser"/>
-  <xacro:include filename="${model_dir}/hokuyo.xacro"/>
-  <xacro:laser name="laser_front_right" frame_names="laser_front_right" topic_names="laser_front_right/scan" parent="top" xyz="0.06 -0.14 0.08" rpy="0 0 ${-pi/4}" driver="cpu"/>
-   -->
-  <!-- Laser -->
-  <xacro:property name="model_dir" value="$(find tuw_gazebo_models)/models/sensors/laser"/>
+  <xacro:property name="model_dir" value="$(arg model_dir)/sensors/laser"/>
   <xacro:include filename="${model_dir}/Sick-LMS100.xacro"/>
-  <xacro:laser name="laser_front_center" frame_names="laser_front_center" topic_names="laser_front_center/scan" parent="top" xyz="0.25 0.0 -0.20" rpy="${pi} 0 0" driver="cpu" visualize="true"/>
+  <xacro:laser name="laser1" frame_names="laser1" topic_names="laser1/scan/raw" parent="top" xyz="0.08 0.0 0.26" rpy="${pi} 0 0" driver="cpu" visualize="false"/>
+  -->
   <!-- xyz="0.16 0 0.125" -->
   <!-- IMU
-  <xacro:property name="model_dir" value="$(find tuw_gazebo_models)/models/sensors/imu"/>
-  <xacro:include filename="$(find tuw_gazebo_models)/models/sensors/imu/imu.xacro"/>
+  <xacro:property name="model_dir" value="$(arg model_dir)/sensors/imu"/>
+  <xacro:include filename="$(arg model_dir)/sensors/imu/imu.xacro"/>
   <xacro:imu_sensor name="imu9dof" parent="chassis" xyz="0.05 0.0 0.262" rpy="0 0 0"/>
   -->
   <!-- Camera
-  <xacro:property name="model_dir" value="$(find tuw_gazebo_models)/models/sensors/camera"/>
+  <xacro:property name="model_dir" value="$(arg model_dir)/sensors/camera"/>
   <xacro:include filename="${model_dir}/camera.xacro"/>
   <xacro:cam name="front_camera" parent="top" xyz="0 0 1" rpy="${-pi/2}  0 ${-pi/2}" />
    -->
   <!-- Depth Camera
-  <xacro:property name="model_dir" value="$(find tuw_gazebo_models)/models/sensors/camera"/>
+  <xacro:property name="model_dir" value="$(arg model_dir)/sensors/camera"/>
   <xacro:include filename="${model_dir}/depth_camera.xacro"/>
   <xacro:cam name="front_depth_camera" parent="top" xyz="0 0 1" rpy="0  0 0" />
