Commit message: laser plugin removed

File: tuw_gazebo_models/models/platforms/transportbuddy/main.xacro (robot description, xacro)
@@ -31,9 +31,8 @@
   <!-- camera plugin -->
   <xacro:camera_zr300_rgb />
-  <!-- Laser
+  <!-- Laser   -->
   <xacro:property name="model_dir" value="$(arg model_dir)/sensors/laser"/>
-  <xacro:include filename="${model_dir}/Sick-LMS100.xacro"/>
-  <xacro:laser name="laser1" frame_names="laser1" topic_names="laser1/scan/raw" parent="top" xyz="0.08 0.0 0.26" rpy="${pi} 0 0" driver="cpu" visualize="false"/>
-  -->
+  <xacro:include filename="${model_dir}/Sick-S300.xacro"/>
+  <xacro:laser name="laser0" frame_names="laser0" topic_names="laser0/scan/raw" parent="top" xyz="0.25 0.0 -0.20" rpy="${pi} 0 0" driver="cpu" visualize="true"/>
   <!-- xyz="0.16 0 0.125" -->
   <!-- IMU

File: tuw_gazebo_models/models/sensors/laser/Sick-LMS100.xacro (robot description, xacro)
@@ -3,6 +3,12 @@
 <!-- Front Laser -->
 <xacro:macro name="laser" params="name frame_names topic_names parent xyz rpy driver:=cpu visualize:=true model_dir:=^">
-    <xacro:if     value="${driver == 'gpu'}"> <xacro:property name="sensor_type" value="gpu_ray"/> <xacro:property name="driver_type" value="libtuw_gazebo_ros_gpu_laser.so"/> </xacro:if>
-    <xacro:unless value="${driver == 'gpu'}"> <xacro:property name="sensor_type" value="ray"    /> <xacro:property name="driver_type" value="libtuw_gazebo_ros_laser.so"    /> </xacro:unless>
+    <xacro:if value="${driver == 'gpu'}">
+      <xacro:property name="sensor_type" value="gpu_ray"/>
+      <xacro:property name="driver_type" value="libgazebo_ros_gpu_laser.so"/>
+    </xacro:if>
+    <xacro:if value="${driver == 'cpu'}">
+      <xacro:property name="sensor_type" value="ray"/>
+      <xacro:property name="driver_type" value="libgazebo_ros_laser.so"/>
+    </xacro:if>
     <joint name="${parent}_${name}_chassis_joint" type="fixed">
 	<axis xyz="0 0 1" />

File: tuw_gazebo_models/models/sensors/laser/hokuyo.xacro (robot description, xacro)
@@ -3,6 +3,12 @@
 <!-- Front Laser -->
 <xacro:macro name="laser" params="name frame_names topic_names parent xyz rpy driver:=cpu visualize:=true model_dir:=^" >
-    <xacro:if     value="${driver == 'gpu'}"> <xacro:property name="sensor_type" value="gpu_ray"/> <xacro:property name="driver_type" value="libtuw_gazebo_ros_gpu_laser.so"/> </xacro:if>
-    <xacro:unless value="${driver == 'gpu'}"> <xacro:property name="sensor_type" value="ray"    /> <xacro:property name="driver_type" value="libtuw_gazebo_ros_laser.so"    /> </xacro:unless>
+    <xacro:if value="${driver == 'gpu'}">
+      <xacro:property name="sensor_type" value="gpu_ray"/>
+      <xacro:property name="driver_type" value="libgazebo_ros_gpu_laser.so"/>
+    </xacro:if>
+    <xacro:if value="${driver == 'cpu'}">
+      <xacro:property name="sensor_type" value="ray"/>
+      <xacro:property name="driver_type" value="libgazebo_ros_laser.so"/>
+    </xacro:if>
     <joint name="${parent}_${name}_joint" type="fixed">
 	<axis xyz="0 0 1" />

File: tuw_gazebo_models/models/sensors/laser/hokuyo_30LX.xacro (robot description, xacro)
@@ -5,10 +5,10 @@
     <xacro:if value="${driver == 'gpu'}">
       <xacro:property name="sensor_type" value="gpu_ray"/>
-      <xacro:property name="driver_type" value="libtuw_gazebo_ros_gpu_laser.so"/>
+      <xacro:property name="driver_type" value="libgazebo_ros_gpu_laser.so"/>
     </xacro:if>
-    <xacro:unless value="${driver == 'gpu'}">
+    <xacro:if value="${driver == 'cpu'}">
       <xacro:property name="sensor_type" value="ray"/>
-      <xacro:property name="driver_type" value="libtuw_gazebo_ros_laser.so"/>
-    </xacro:unless>
+      <xacro:property name="driver_type" value="libgazebo_ros_laser.so"/>
+    </xacro:if>
     <joint name="${parent}_${name}_joint" type="fixed">
       <axis xyz="0 0 1"/>
