Commit message: model renamed

File: tuw_gazebo_models/models/platforms/transportbuddy/body/chassis.xacro (robot description, xacro)
@@ -16,5 +16,5 @@
       <origin xyz="-0.0 0 -0.07" rpy="0 0 ${M_PI}"/>
       <geometry>
-	<mesh filename="file://${model_dir}/meshes/TransportBuddy.dae"/>
+	<mesh filename="file://${model_dir}/meshes/chassis.dae"/>
       </geometry>
       <material name="SallyWhite">

Commit message: model update on tb

File: tuw_gazebo_models/models/platforms/transportbuddy/body/chassis.xacro (robot description, xacro)
@@ -16,5 +16,5 @@
       <origin xyz="-0.0 0 -0.07" rpy="0 0 ${M_PI}"/>
       <geometry>
-	<mesh filename="file://${model_dir}/meshes/chassis.dae"/>
+	<mesh filename="file://${model_dir}/meshes/tb01.dae"/>
       </geometry>
       <material name="SallyWhite">
