Commit message: namespace added

File: tuw_gazebo_description/models/pioneer3dx/body/body.xacro (robot description, xacro)
@@ -31,6 +31,6 @@
     <xacro:pioneer_swivel             parent="${parent}"  xyz="-0.185 0    0.0535" rpy="0 0 0">               <container> <xacro:insert_block name="contact_data"/> </container> </xacro:pioneer_swivel>
     <!-- Wheels -->
-    <xacro:pioneer_wheel side="right" parent="${parent}"  xyz=" 0    -0.165 ${wheel_radius}" rpy="0 0 0" radius="${wheel_radius}"> <container> <xacro:insert_block name="contact_data"/> </container> </xacro:pioneer_wheel>
-    <xacro:pioneer_wheel side="left"  parent="${parent}"  xyz=" 0     0.165 ${wheel_radius}" rpy="0 0 0" radius="${wheel_radius}"> <container> <xacro:insert_block name="contact_data"/> </container> </xacro:pioneer_wheel>
+    <xacro:pioneer_wheel name="right" parent="${parent}"  xyz=" 0    -0.165 ${wheel_radius}" rpy="0 0 0" radius="${wheel_radius}"> <container> <xacro:insert_block name="contact_data"/> </container> </xacro:pioneer_wheel>
+    <xacro:pioneer_wheel name="left"  parent="${parent}"  xyz=" 0     0.165 ${wheel_radius}" rpy="0 0 0" radius="${wheel_radius}"> <container> <xacro:insert_block name="contact_data"/> </container> </xacro:pioneer_wheel>
   </xacro:macro>
 </robot>

File: tuw_gazebo_description/models/pioneer3dx/body/wheel.xacro (robot description, xacro)
@@ -3,79 +3,57 @@
   xmlns:xacro="http://ros.org/wiki/xacro">
   <xacro:property name="M_PI" value="3.1415926535897931" />
-  <xacro:macro name="pioneer_wheel" params="side parent xyz rpy radius model_dir:=^ **contact_data">
-    <!-- Hubcap Mount -->
-      <joint name="${side}_hub_mount_joint" type="fixed">
-	<origin xyz="${xyz}" rpy="${rpy}"/>
-	<parent link="${parent}"/>
-	<child link="${side}_hub_mount"/>
-	<axis xyz="0 1 0"/>
+  <xacro:macro name="pioneer_wheel" params="name parent xyz rpy radius model_dir:=^ **contact_data">
+    <!-- Wheel -->
+    <joint name="${name}_wheel_joint" type="continuous">
+		<origin xyz="${xyz}" rpy="${rpy}"/>
+		<axis xyz="0 1 0"/>
+		<parent link="${parent}"/>
+		<child link="${name}_wheel"/>
     </joint>
-    <link name="${side}_hub_mount">
-    <inertial>
-      <mass value="0.01"/>
-      <origin xyz="0 0 0"/>
-      <inertia ixx="0.012411765597" ixy="0" ixz="0" iyy="0.015218160428" iyz="0" izz="0.011763977943"/>
-    </inertial>
-	<visual>
-	    <origin xyz="0 0 0" rpy="0 0 0"/>
-	    <geometry> <box size="0.001 0.001 0.001"/> </geometry>
-	</visual>
-	<collision>
-	    <origin xyz="0 0 0" rpy="0 0 0"/>
-	    <geometry> <box size="0.001 0.001 0.001"/> </geometry>
-	</collision>
+    <link name="${name}_wheel">
+		<inertial>
+			<mass value="0.5"/>
+			<origin xyz="0 0 0"/>
+			<inertia ixx="0.012411765597" ixy="0" ixz="0" iyy="0.015218160428" iyz="0" izz="0.011763977943"/>
+		</inertial>
+		<visual>
+			<origin xyz="0 0 0" rpy="0 0 0"/>
+			<geometry> <mesh filename="file://${model_dir}/meshes/wheel.dae"/> </geometry>
+			<material name="WheelBlack"> <color rgba="0.117 0.117 0.117 1"/> </material>
+		</visual>
+		<collision>
+			<origin xyz="0 0 0" rpy="${pi/2} 0 0"/>
+			<geometry> <cylinder radius="${radius}" length="0.001"/> <!--<mesh filename="${meshes}/${name}_wheel.stl"/>--> </geometry>
+		</collision>
     </link>
+		<gazebo reference="${name}_wheel">
+		<material value="Gazebo/Black"/>
+	<xacro:insert_block name="contact_data"/>
+    </gazebo>
     <!-- Hubcap -->
-    <joint name="${side}_hub_joint" type="continuous">
-	<origin xyz="0 0 0" rpy="0 0 0"/>
-	<parent link="${side}_hub_mount"/>
-	<child link="${side}_hub"/>
-	<axis xyz="0 1 0"/>
+    <joint name="${name}_hub_joint" type="fixed">
+		<origin xyz="0 0 0" rpy="0 0 0"/>
+		<axis xyz="0 1 0"/>
+		<parent link="${name}_wheel"/>
+		<child link="${name}_hub"/>
     </joint>
-    <link name="${side}_hub">
-    <inertial>
-      <mass value="0.01"/>
-      <origin xyz="0 0 0"/>
-      <inertia ixx="0.012411765597" ixy="0" ixz="0" iyy="0.015218160428" iyz="0" izz="0.011763977943"/>
-    </inertial>
-	<visual>
-	    <origin xyz="0 0 0" rpy="0 0 0"/>
-	    <geometry> <mesh filename="file://${model_dir}/meshes/hubcap.dae"/> </geometry>
-	    <material name="HubcapYellow"> <color rgba="1.0 0.811 0.151 1.0"/> </material>
-	</visual>
-	<collision>
-	    <origin xyz="0 0 0" rpy="0 0 0"/>
-	    <geometry> <box size="0.001 0.001 0.001"/> </geometry>
-	</collision>
+    <link name="${name}_hub">
+		<inertial>
+			<mass value="0.01"/>
+			<origin xyz="0 0 0"/>
+			<inertia ixx="0.012411765597" ixy="0" ixz="0" iyy="0.015218160428" iyz="0" izz="0.011763977943"/>
+		</inertial>
+		<visual>
+			<origin xyz="0 0 0" rpy="0 0 0"/>
+			<geometry> <mesh filename="file://${model_dir}/meshes/hubcap.dae"/> </geometry>
+			<material name="HubcapYellow"> <color rgba="1.0 0.811 0.151 1.0"/> </material>
+		</visual>
+		<collision>
+			<origin xyz="0 0 0" rpy="0 0 0"/>
+			<geometry> <box size="0.001 0.001 0.001"/> </geometry>
+		</collision>
     </link>
-    <gazebo reference="${side}_hub">
-	<material value="Gazebo/Yellow"/>
-    </gazebo>
-    <!-- Wheel -->
-    <joint name="${side}_wheel_joint" type="fixed">
-	<axis xyz="0 1 0"/>
-	<origin xyz="0 0 0" rpy="0 0 0"/>
-	<parent link="${side}_hub"/>
-	<child link="${side}_wheel"/>
-    </joint>
-    <link name="${side}_wheel">
-    <inertial>
-      <mass value="0.5"/>
-      <origin xyz="0 0 0"/>
-      <inertia ixx="0.012411765597" ixy="0" ixz="0" iyy="0.015218160428" iyz="0" izz="0.011763977943"/>
-    </inertial>
-	<visual>
-	    <origin xyz="0 0 0" rpy="0 0 0"/>
-	    <geometry> <mesh filename="file://${model_dir}/meshes/wheel.dae"/> </geometry>
-	    <material name="WheelBlack"> <color rgba="0.117 0.117 0.117 1"/> </material>
-	</visual>
-	<collision>
-	    <origin xyz="0 0 0" rpy="${pi/2} 0 0"/>
-	    <geometry> <cylinder radius="${radius}" length="0.001"/> <!--<mesh filename="${meshes}/${side}_wheel.stl"/>--> </geometry>
-	</collision>
-    </link>
-    <gazebo reference="${side}_wheel">
-	<material value="Gazebo/Black"/>
-	<xacro:insert_block name="contact_data"/>
+		<gazebo reference="${name}_hub">
+		<material value="Gazebo/Yellow"/>
     </gazebo>
   </xacro:macro>

File: tuw_gazebo_description/models/pioneer3dx/main.xacro (robot description, xacro)
@@ -11,4 +11,4 @@
   <xacro:vehicle_body name="chassis" parent="base_link"/>
   <xacro:include filename="$(arg model_dir)/$(arg platform_dir)/plugins.xacro"/>
-  <xacro:differential_drive ns="r0" />
+  <xacro:differential_drive namespace="$(arg namespace)" />
 </robot>

File: tuw_gazebo_description/models/pioneer3dx/plugins.xacro (robot description, xacro)
@@ -1,14 +1,14 @@
 <?xml version="1.0"?>
 <robot xmlns:xacro="http://ros.org/wiki/xacro">
-  <xacro:macro name="differential_drive" params="ns">
+  <xacro:macro name="differential_drive" params="namespace">
     <gazebo>
         <plugin name='diff_drive' filename='libgazebo_ros_diff_drive.so'>
           <ros>
-            <namespace>/${ns}</namespace>
+            <namespace>/${namespace}</namespace>
             <remapping>cmd_vel:=cmd_vel</remapping>
             <remapping>odom:=odom</remapping>
           </ros>
-          <left_joint>left_hub_joint</left_joint>
-          <right_joint>right_hub_joint</right_joint>
+          <left_joint>left_wheel_joint</left_joint>
+          <right_joint>right_wheel_joint</right_joint>
           <wheel_separation>0.3</wheel_separation>
           <wheel_diameter>0.18</wheel_diameter>

Commit message: xacro cleanup in progress

File: tuw_gazebo_description/models/pioneer3dx/body/body.xacro (robot description, xacro)
@@ -9,4 +9,5 @@
   <xacro:include filename="sonar.xacro"/>
   <xacro:property name="wheel_radius" value="0.097" />
+  <!-- name="body" parent="base_link" -->
   <xacro:macro name="vehicle_body" params="name parent">
     <!-- base_link -->

File: tuw_gazebo_description/models/pioneer3dx/body/mount.xacro (robot description, xacro)
@@ -36,10 +36,10 @@
   </gazebo>
   <!--  mount bottom left -->
-  <joint name="${parent}_${name}_bottom_left_joint" type="fixed">
+  <joint name="${parent}_${name}_bottom_joint" type="fixed">
     <origin xyz="0 0 0" rpy="${rpy}"/>
     <parent link="${parent}"/>
-    <child link="${name}_bottom_left"/>
+    <child link="${name}_bottom"/>
   </joint>
-  <link name="${name}_bottom_left">
+  <link name="${name}_bottom">
     <!-- right base bar -->
     <visual>
@@ -171,5 +171,5 @@
     </collision>
   </link>
-  <gazebo reference="${name}_bottom_left">
+  <gazebo reference="${name}_bottom">
     <material value="Gazebo/Grey"/>
   </gazebo>

File: tuw_gazebo_description/models/pioneer3dx/main.xacro (robot description, xacro)
@@ -9,5 +9,5 @@
   <xacro:property name="model_dir" value="$(arg model_dir)/$(arg platform_dir)/body"/>
   <xacro:include filename="${model_dir}/body.xacro"/>
-  <xacro:vehicle_body name="chassis" parent="base_link"/>
+  <xacro:vehicle_body name="body" parent="base_link"/>
   <xacro:include filename="$(arg model_dir)/$(arg platform_dir)/plugins.xacro"/>
   <xacro:differential_drive namespace="$(arg namespace)" />

File: tuw_gazebo_description/models/pioneer3dx/plugins.xacro (robot description, xacro)
@@ -18,6 +18,6 @@
           <publish_odom_tf>true</publish_odom_tf>
           <publish_wheel_tf>true</publish_wheel_tf>
-          <odometry_frame>odom_frame_test</odometry_frame>
-          <robot_base_frame>chassis</robot_base_frame>
+          <odometry_frame>odom</odometry_frame>
+          <robot_base_frame>base_link</robot_base_frame>
       </plugin>
     </gazebo>

Commit message: swivel xacro cleanup

File: tuw_gazebo_description/models/pioneer3dx/body/body.xacro (robot description, xacro)
@@ -30,5 +30,5 @@
     </xacro:property>
     <!-- Swivels -->
-    <xacro:pioneer_swivel             parent="${parent}"  xyz="-0.185 0    0.0535" rpy="0 0 0">               <container> <xacro:insert_block name="contact_data"/> </container> </xacro:pioneer_swivel>
+    <xacro:pioneer_swivel  name="swivel"    parent="${parent}"  xyz="-0.185 0    0.0535" rpy="0 0 0">               <container> <xacro:insert_block name="contact_data"/> </container> </xacro:pioneer_swivel>
     <!-- Wheels -->
     <xacro:pioneer_wheel name="right" parent="${parent}"  xyz=" 0    -0.165 ${wheel_radius}" rpy="0 0 0" radius="${wheel_radius}"> <container> <xacro:insert_block name="contact_data"/> </container> </xacro:pioneer_wheel>

File: tuw_gazebo_description/models/pioneer3dx/body/swivel.xacro (robot description, xacro)
@@ -2,7 +2,7 @@
 <robot xmlns:xacro="http://ros.org/wiki/xacro">
   <xacro:property name="M_PI" value="3.1415926535897931" />
-  <xacro:macro name="pioneer_swivel" params="parent xyz rpy model_dir:=^ **contact_data">
+  <xacro:macro name="pioneer_swivel" params="name parent xyz rpy model_dir:=^ **contact_data">
   <!-- Swivel -->
-  <joint name="chassis_swivel_joint" type="continuous">
+  <joint name="${name}_joint" type="continuous">
     <origin xyz="${xyz}" rpy="${rpy}"/>
     <axis xyz="0 0 1"/>
@@ -11,7 +11,7 @@
     <joint_properties damping="0.1" friction="0.0"/>
     <parent link="${parent}"/>
-    <child link="swivel"/>
+    <child link="${name}"/>
   </joint>
-  <link name="swivel">
+  <link name="${name}">
     <inertial>
       <mass value="0.1"/>
@@ -35,9 +35,9 @@
     </collision>
   </link>
-  <gazebo reference="swivel">
+  <gazebo reference="${name}">
     <material value="Gazebo/Grey"/>
   </gazebo>
   <!-- Center Wheel -->
-  <joint name="swivel_wheel_joint" type="continuous">
+  <joint name="${name}_wheel_joint" type="continuous">
     <origin xyz="-0.026 0 -0.016" rpy="0 0 0"/>
     <axis xyz="0 1 0"/>
@@ -46,7 +46,7 @@
     <joint_properties damping="0.0" friction="0.0"/>
     <parent link="swivel"/>
-    <child link="center_wheel"/>
+    <child link="${name}_wheel"/>
   </joint>
-  <link name="center_wheel">
+  <link name="${name}_wheel">
     <inertial>
       <mass value="0.1"/>
@@ -71,15 +71,15 @@
     </collision>
   </link>
-  <gazebo reference="center_wheel">
+  <gazebo reference="${name}_wheel">
     <material value="Gazebo/Black"/>
     <xacro:insert_block name="contact_data"/>
   </gazebo>
   <!-- Center Hubcap -->
-  <joint name="wheel_hubcap_joint" type="fixed">
+  <joint name="${name}_hubcap_joint" type="fixed">
     <origin xyz="0 0 0" rpy="0 0 0"/>
-    <parent link="center_wheel"/>
-    <child link="center_hubcap"/>
+    <parent link="${name}_wheel"/>
+    <child link="${name}_hubcap"/>
   </joint>
-  <link name="center_hubcap">
+  <link name="${name}_hubcap">
     <inertial>
       <mass value="0.01"/>
@@ -103,5 +103,5 @@
     </collision>
   </link>
-  <gazebo reference="center_hubcap">
+  <gazebo reference="${name}_hubcap">
     <material value="Gazebo/Grey"/>
     <xacro:insert_block name="contact_data"/>
