Commit message: swivel tf not yet working

File: tuw_gazebo_description/models/pioneer3dx/body/swivel.xacro (robot description, xacro)
@@ -45,5 +45,5 @@
     <!--limit effort="100" velocity="100" k_velocity="0"/-->
     <joint_properties damping="0.0" friction="0.0"/>
-    <parent link="swivel"/>
+    <parent link="${name}"/>
     <child link="${name}_wheel"/>
   </joint>

File: tuw_gazebo_description/models/pioneer3dx/main.xacro (robot description, xacro)
@@ -4,4 +4,5 @@
   <xacro:arg name="platform_dir"   default="pioneer3dx"/>
   <xacro:arg name="namespace"      default="r0"/>
+  <xacro:arg name="robot_name"     default="r0"/>
   <!-- Import Rviz colors -->
   <xacro:include filename="$(arg model_dir)/materials.xacro" />
@@ -11,4 +12,5 @@
   <xacro:vehicle_body name="body" parent="base_link"/>
   <xacro:include filename="$(arg model_dir)/$(arg platform_dir)/plugins.xacro"/>
-  <xacro:differential_drive namespace="$(arg namespace)" />
+  <xacro:differential_drive    name="$(arg robot_name)" namespace="$(arg namespace)" />
+  <xacro:joint_state_publisher name="$(arg robot_name)" namespace="$(arg namespace)" />
 </robot>

File: tuw_gazebo_description/models/pioneer3dx/plugins.xacro (robot description, xacro)
@@ -1,7 +1,7 @@
 <?xml version="1.0"?>
 <robot xmlns:xacro="http://ros.org/wiki/xacro">
-  <xacro:macro name="differential_drive" params="namespace">
+  <xacro:macro name="differential_drive" params="name namespace">
     <gazebo>
-        <plugin name='diff_drive' filename='libgazebo_ros_diff_drive.so'>
+        <plugin name='${name}_diff_drive' filename='libgazebo_ros_diff_drive.so'>
           <ros>
             <namespace>/${namespace}</namespace>
@@ -17,5 +17,5 @@
           <publish_odom>true</publish_odom>
           <publish_odom_tf>true</publish_odom_tf>
-          <publish_wheel_tf>true</publish_wheel_tf>
+          <publish_wheel_tf>false</publish_wheel_tf>
           <odometry_frame>odom</odometry_frame>
           <robot_base_frame>base_link</robot_base_frame>
@@ -23,3 +23,18 @@
     </gazebo>
   </xacro:macro>
+  <xacro:macro name="joint_state_publisher" params="name namespace">
+    <gazebo>
+    <plugin name="${name}_gazebo_ros_joint_state_publisher"
+        filename="libgazebo_ros_joint_state_publisher.so">
+      <ros>
+        <namespace>/${namespace}</namespace>
+        <remapping>joint_states:=joint_states</remapping>
+      </ros>
+      <update_rate>10</update_rate>
+      <joint_name>left_wheel_joint</joint_name>
+      <joint_name>right_wheel_joint</joint_name>
+      <joint_name>swivel_joint</joint_name>
+    </plugin>
+    </gazebo>
+  </xacro:macro>
 </robot>
