Commit message: laser added without plugin, models dir updated

File: tuw_gazebo_description/models/pioneer3dx/body/chassis.xacro (robot description, xacro)
@@ -2,5 +2,5 @@
 <robot xmlns:xacro="http://ros.org/wiki/xacro">
   <xacro:property name="M_PI" value="3.1415926535897931" />
-  <xacro:macro name="pioneer_chassis" params="name parent xyz rpy model_dir:=^">
+  <xacro:macro name="pioneer_chassis" params="name parent xyz rpy models_dir:=^">
   <!-- Chassis -->
   <joint name="${parent}_${name}_joint" type="fixed">
@@ -13,5 +13,5 @@
       <origin xyz="-0.045 0 0.085" rpy="0 0 0"/>
       <geometry>
-        <mesh filename="file://${model_dir}/meshes/chassis.dae"/>
+        <mesh filename="file://${models_dir}/pioneer3dx/body/meshes/chassis.dae"/>
       </geometry>
       <material name="ChassisRed">
@@ -26,5 +26,5 @@
       <!--origin xyz="-0.045 0 0.148" rpy="0 0 0"/>
       <geometry>
-        <mesh filename="file://${model_dir}/meshes/chassis.dae"/>
+        <mesh filename="file://${model_dir}/meshes/body/chassis.dae"/>
       </geometry-->
     </collision>
@@ -46,5 +46,5 @@
       <origin xyz="-0.045 0 0" rpy="0 0 0"/>
       <geometry>
-        <mesh filename="file://${model_dir}/meshes/top.dae"/>
+        <mesh filename="file://${models_dir}/pioneer3dx/body/meshes/top.dae"/>
       </geometry>
       <material name="TopBlack">
@@ -57,5 +57,5 @@
     <!--origin xyz="0.0 0 0.0" rpy="0 0 0"/>
       <geometry>
-        <mesh filename="file://${model_dir}/meshes/top.dae"/>
+        <mesh filename="file://${models_dir}/pioneer3dx/body/meshes/top.dae"/>
       </geometry-->
     </collision>

File: tuw_gazebo_description/models/pioneer3dx/body/mount.xacro (robot description, xacro)
@@ -2,5 +2,5 @@
 <robot xmlns:xacro="http://ros.org/wiki/xacro">
   <xacro:property name="M_PI" value="3.1415926535897931" />
-  <xacro:macro name="pioneer_mount" params="name parent xyz rpy model_dir:=^">
+  <xacro:macro name="pioneer_mount" params="name parent xyz rpy">
   <xacro:property name="mount_base_width" value="0.14" />
   <xacro:property name="mount_bar_width" value="0.02" />

File: tuw_gazebo_description/models/pioneer3dx/body/sonar.xacro (robot description, xacro)
@@ -2,5 +2,5 @@
 <robot xmlns:xacro="http://ros.org/wiki/xacro">
   <xacro:property name="M_PI" value="3.1415926535897931" />
-  <xacro:macro name="pioneer_sonar" params="name parent xyz rpy model_dir:=^">
+  <xacro:macro name="pioneer_sonar" params="name parent xyz rpy models_dir:=^">
   <!-- Front Sonar -->
   <joint name="${parent}_${name}_joint" type="fixed">
@@ -14,5 +14,5 @@
       <origin xyz="0 0 0" rpy="0 0 0"/>
       <geometry>
-        <mesh filename="file://${model_dir}/meshes/back_sonar.dae"/>
+        <mesh filename="file://${models_dir}/pioneer3dx/meshes/back_sonar.dae"/>
       </geometry>
       <material name="SonarYellow">

File: tuw_gazebo_description/models/pioneer3dx/body/swivel.xacro (robot description, xacro)
@@ -2,5 +2,5 @@
 <robot xmlns:xacro="http://ros.org/wiki/xacro">
   <xacro:property name="M_PI" value="3.1415926535897931" />
-  <xacro:macro name="pioneer_swivel" params="name parent xyz rpy model_dir:=^ **contact_data">
+  <xacro:macro name="pioneer_swivel" params="name parent xyz rpy models_dir:=^ **contact_data">
   <!-- Swivel -->
   <joint name="${name}_joint" type="continuous">
@@ -22,5 +22,5 @@
       <origin xyz="0 0 0" rpy="0 0 0"/>
       <geometry>
-        <mesh filename="file://${model_dir}/meshes/swivel.stl"/>
+        <mesh filename="file://${models_dir}/pioneer3dx/body/meshes/swivel.stl"/>
       </geometry>
       <material name="swivel">
@@ -57,5 +57,5 @@
       <origin xyz="0 0 0" rpy="0 0 0"/>
       <geometry>
-        <mesh filename="file://${model_dir}/meshes/center_wheel.stl"/>
+        <mesh filename="file://${models_dir}/pioneer3dx/body/meshes/center_wheel.stl"/>
       </geometry>
       <material name="WheelBlack">
@@ -90,5 +90,5 @@
       <origin xyz="0 0 0" rpy="0 0 0"/>
       <geometry>
-        <mesh filename="file://${model_dir}/meshes/center_hubcap.stl"/>
+        <mesh filename="file://${models_dir}/pioneer3dx/body/meshes/center_hubcap.stl"/>
       </geometry>
       <material name="swivel">

File: tuw_gazebo_description/models/pioneer3dx/body/wheel.xacro (robot description, xacro)
@@ -3,5 +3,5 @@
   xmlns:xacro="http://ros.org/wiki/xacro">
   <xacro:property name="M_PI" value="3.1415926535897931" />
-  <xacro:macro name="pioneer_wheel" params="name parent xyz rpy radius model_dir:=^ **contact_data">
+  <xacro:macro name="pioneer_wheel" params="name parent xyz rpy radius models_dir:=^ **contact_data">
     <!-- Wheel -->
     <joint name="${name}_wheel_joint" type="continuous">
@@ -19,5 +19,5 @@
 		<visual>
 			<origin xyz="0 0 0" rpy="0 0 0"/>
-			<geometry> <mesh filename="file://${model_dir}/meshes/wheel.dae"/> </geometry>
+			<geometry> <mesh filename="file://${models_dir}/pioneer3dx/meshes/wheel.dae"/> </geometry>
 			<material name="WheelBlack"> <color rgba="0.117 0.117 0.117 1"/> </material>
 		</visual>
@@ -46,5 +46,5 @@
 		<visual>
 			<origin xyz="0 0 0" rpy="0 0 0"/>
-			<geometry> <mesh filename="file://${model_dir}/meshes/hubcap.dae"/> </geometry>
+			<geometry> <mesh filename="file://${models_dir}/pioneer3dx/meshes/hubcap.dae"/> </geometry>
 			<material name="HubcapYellow"> <color rgba="1.0 0.811 0.151 1.0"/> </material>
 		</visual>

File: tuw_gazebo_description/models/pioneer3dx/main.xacro (robot description, xacro)
@@ -1,16 +1,22 @@
 <?xml version="1.0"?>
 <robot xmlns:xacro="http://ros.org/wiki/xacro" name="pioneer3dx" >
-  <xacro:arg name="model_dir"      default="/home/max/projects/ros2/gazebo/ws01/src/tuw2_gazebo/tuw_gazebo_description/models"/>
-  <xacro:arg name="platform_dir"   default="pioneer3dx"/>
-  <xacro:arg name="namespace"      default="r0"/>
-  <xacro:arg name="robot_name"     default="r0"/>
+  <xacro:arg name="models_dir"      default="/home/max/projects/ros2/gazebo/ws01/src/tuw2_gazebo/tuw_gazebo_description/models"/>
+  <xacro:arg name="robot_model"     default="pioneer3dx"/>
+  <xacro:arg name="laser_model"     default="hokuyo"/>
+  <xacro:arg name="namespace"       default="r0"/>
+  <xacro:arg name="robot_name"      default="r0"/>
+  <xacro:arg name="laser0_topic"    default="scan_raw"/>
+  <xacro:property name="models_dir" value="$(arg models_dir)"/>
+  <xacro:property name="robot_model" value="$(arg robot_model)"/>
+  <xacro:property name="laser_model" value="$(arg laser_model)"/>
   <!-- Import Rviz colors -->
-  <xacro:include filename="$(arg model_dir)/materials.xacro" />
+  <xacro:include filename="$(arg models_dir)/materials.xacro" />
   <!-- Import platform -->
-  <xacro:property name="model_dir" value="$(arg model_dir)/$(arg platform_dir)/body"/>
-  <xacro:include filename="${model_dir}/body.xacro"/>
+  <xacro:include filename="${models_dir}/${robot_model}/body/body.xacro"/>
   <xacro:vehicle_body name="body" parent="base_link"/>
-  <xacro:include filename="$(arg model_dir)/$(arg platform_dir)/plugins.xacro"/>
+  <xacro:include filename="${models_dir}/${robot_model}/plugins.xacro"/>
   <xacro:differential_drive    name="$(arg robot_name)" namespace="$(arg namespace)" />
   <xacro:joint_state_publisher name="$(arg robot_name)" namespace="$(arg namespace)" />
+  <xacro:include filename="${models_dir}/${laser_model}/main.xacro"/>
+  <xacro:laser name="laser0" frame_names="$(arg namespace)/laser0" topic_names="$(arg laser0_topic)" parent="top" xyz="0.15 0.0 0.06" rpy="0 0 0" driver="gpu" visualize="true"/>
 </robot>
