Commit message: laser added without plugin, models dir updated

File: tuw_gazebo_description/models/pioneer3dx/body/sonar.xacro (robot description, xacro)
@@ -14,5 +14,5 @@
       <origin xyz="0 0 0" rpy="0 0 0"/>
       <geometry>
-        <mesh filename="file://${models_dir}/pioneer3dx/meshes/back_sonar.dae"/>
+        <mesh filename="file://${models_dir}/pioneer3dx/body/meshes/back_sonar.dae"/>
       </geometry>
       <material name="SonarYellow">

File: tuw_gazebo_description/models/pioneer3dx/body/wheel.xacro (robot description, xacro)
@@ -19,5 +19,5 @@
 		<visual>
 			<origin xyz="0 0 0" rpy="0 0 0"/>
-			<geometry> <mesh filename="file://${models_dir}/pioneer3dx/meshes/wheel.dae"/> </geometry>
+			<geometry> <mesh filename="file://${models_dir}/pioneer3dx/body/meshes/wheel.dae"/> </geometry>
 			<material name="WheelBlack"> <color rgba="0.117 0.117 0.117 1"/> </material>
 		</visual>
@@ -46,5 +46,5 @@
 		<visual>
 			<origin xyz="0 0 0" rpy="0 0 0"/>
-			<geometry> <mesh filename="file://${models_dir}/pioneer3dx/meshes/hubcap.dae"/> </geometry>
+			<geometry> <mesh filename="file://${models_dir}/pioneer3dx/body/meshes/hubcap.dae"/> </geometry>
 			<material name="HubcapYellow"> <color rgba="1.0 0.811 0.151 1.0"/> </material>
 		</visual>
