Commit message: tuw_wanderer

File: tuw_gazebo_models/models/hokuyo/main.xacro (robot description, xacro)
@@ -2,30 +2,65 @@
 <robot xmlns:xacro="http://ros.org/wiki/xacro" name="hokuyo" >
     <!-- hokuyo Laser -->
-    <xacro:macro name="laser" params="name frame_names topic_names parent xyz rpy driver:=cpu visualize:=true models_dir:=^" >
+    <xacro:macro name="laser" params="name namespace topic_name parent xyz rpy driver:=cpu visualize:=true models_dir:=^" >
         <joint name="${parent}_${name}_joint" type="fixed">
-        <axis xyz="0 0 1" />
-        <origin xyz="${xyz}" rpy="${rpy}"/>
-        <parent link="${parent}"/>
-        <child link="${name}"/>
+            <axis xyz="0 0 1" />
+            <origin xyz="${xyz}" rpy="${rpy}"/>
+            <parent link="${parent}"/>
+            <child link="${name}"/>
         </joint>
         <link name="${name}">
-        <collision>
-            <origin xyz="0 0 -0.025" rpy="0 0 0"/>
-            <geometry>
-            <box size="0.05 0.05 0.05"/>
-            </geometry>
-        </collision>
-        <visual>
-            <origin xyz="0 0 -0.025" rpy="0 0 0"/>
-            <geometry>
-            <mesh filename="file://${models_dir}/hokuyo/meshes/hokuyo.dae"/>
-            </geometry>
-        </visual>
-        <inertial>
-            <mass value="1e-2" />
-            <origin xyz="0 0 -0.025" rpy="0 0 0"/>
-            <inertia ixx="1e-6" ixy="0" ixz="0" iyy="1e-6" iyz="0" izz="1e-6" />
-        </inertial>
+            <collision>
+                <origin xyz="0 0 -0.025" rpy="0 0 0"/>
+                <geometry>
+                <box size="0.05 0.05 0.05"/>
+                </geometry>
+            </collision>
+            <visual>
+                <origin xyz="0 0 -0.025" rpy="0 0 0"/>
+                <geometry>
+                <mesh filename="file://${models_dir}/hokuyo/meshes/hokuyo.dae"/>
+                </geometry>
+            </visual>
+            <inertial>
+                <mass value="1e-2" />
+                <origin xyz="0 0 -0.025" rpy="0 0 0"/>
+                <inertia ixx="1e-6" ixy="0" ixz="0" iyy="1e-6" iyz="0" izz="1e-6" />
+            </inertial>
         </link>
+            <!-- ray sensor -->
+            <gazebo reference="${name}">
+                <sensor name="${name}_sensor" type="ray">
+                    <pose>0 0 0 0 0 0</pose>
+                    <update_rate>10</update_rate>
+                    <visualize>${visualize}</visualize>
+                    <always_on>true</always_on>
+                    <ray>
+                        <scan>
+                            <horizontal>
+                                <samples>683</samples>
+                                <resolution>1.0</resolution>
+                                <min_angle>-2.35619449019</min_angle>
+                                <max_angle>2.35619449019</max_angle>
+                            </horizontal>
+                        </scan>
+                        <range>
+                            <min>0.05</min>
+                            <max>10</max>
+                        </range>
+                        <noise>
+                            <type>gaussian</type>
+                            <mean>0.0</mean>
+                            <stddev>0.01</stddev>
+                        </noise>
+                    </ray>
+                    <plugin name="laserscan" filename="libgazebo_ros_ray_sensor.so">
+                        <ros>
+                            <namespace>/rrbot/laser</namespace>
+                            <remapping>~/out:=scan</remapping>
+                        </ros>
+                        <output_type>sensor_msgs/LaserScan</output_type>
+                    </plugin>
+                </sensor>
+            </gazebo>
     </xacro:macro>
 </robot>

File: tuw_gazebo_models/models/pioneer3dx/main.xacro (robot description, xacro)
@@ -19,4 +19,4 @@
   <xacro:joint_state_publisher name="$(arg robot_name)" namespace="$(arg namespace)" />
   <xacro:include filename="${models_dir}/${laser_model}/main.xacro"/>
-  <xacro:laser name="laser0" frame_names="$(arg namespace)/laser0" topic_names="$(arg laser0_topic)" parent="top" xyz="0.15 0.0 0.06" rpy="0 0 0" driver="gpu" visualize="true"/>
+  <xacro:laser name="laser0" namespace="$(arg namespace)" topic_name="$(arg laser0_topic)" parent="top" xyz="0.15 0.0 0.06" rpy="0 0 0" driver="gpu" visualize="true"/>
 </robot>

Commit message: laser working

File: tuw_gazebo_models/models/hokuyo/main.xacro (robot description, xacro)
@@ -2,5 +2,11 @@
 <robot xmlns:xacro="http://ros.org/wiki/xacro" name="hokuyo" >
     <!-- hokuyo Laser -->
-    <xacro:macro name="laser" params="name namespace topic_name parent xyz rpy driver:=cpu visualize:=true models_dir:=^" >
+    <xacro:macro name="laser" params="name parent namespace topic_name frame_name xyz rpy driver:=cpu visualize:=true models_dir:=^" >
+        <xacro:if value="${driver == 'gpu'}">
+            <xacro:property name="sensor_type" value="gpu_ray"/>
+        </xacro:if>
+        <xacro:if value="${driver == 'cpu'}">
+            <xacro:property name="sensor_type" value="ray"/>
+        </xacro:if>
         <joint name="${parent}_${name}_joint" type="fixed">
             <axis xyz="0 0 1" />
@@ -30,7 +36,7 @@
             <!-- ray sensor -->
             <gazebo reference="${name}">
-                <sensor name="${name}_sensor" type="ray">
+                <sensor name="${name}_sensor" type="${sensor_type}">
                     <pose>0 0 0 0 0 0</pose>
-                    <update_rate>10</update_rate>
+                    <update_rate>30</update_rate>
                     <visualize>${visualize}</visualize>
                     <always_on>true</always_on>
@@ -54,5 +60,5 @@
                         </noise>
                     </ray>
-                    <plugin name="laserscan" filename="libgazebo_ros_ray_sensor.so">
+                    <plugin name="${name}_laserscan" filename="libgazebo_ros_ray_sensor.so">
                         <ros>
                             <namespace>${namespace}</namespace>
@@ -60,5 +66,5 @@
                         </ros>
                         <output_type>sensor_msgs/LaserScan</output_type>
-                        <frame_name>${name}</frame_name>
+                        <frame_name>${frame_name}</frame_name>
                     </plugin>
                 </sensor>

File: tuw_gazebo_models/models/pioneer3dx/main.xacro (robot description, xacro)
@@ -19,4 +19,4 @@
   <xacro:joint_state_publisher name="$(arg robot_name)" namespace="$(arg namespace)" />
   <xacro:include filename="${models_dir}/${laser_model}/main.xacro"/>
-  <xacro:laser name="laser0" namespace="$(arg namespace)" topic_name="$(arg laser0_topic)" parent="top" xyz="0.15 0.0 0.06" rpy="0 0 0" driver="gpu" visualize="true"/>
+  <xacro:laser name="laser0" parent="top" namespace="$(arg namespace)" topic_name="$(arg laser0_topic)" frame_name="laser0" xyz="0.15 0.0 0.06" rpy="0 0 0" driver="gpu" visualize="true"/>
 </robot>
