Commit message: swivel

File: tuw_gazebo_models/models/pioneer3dx/body/body.xacro (robot description, xacro)
@@ -30,5 +30,5 @@
     </xacro:property>
     <!-- Swivels -->
-    <xacro:pioneer_swivel  name="swivel"    parent="${parent}"  xyz="-0.185 0    0.0535" rpy="0 0 0">               <container> <xacro:insert_block name="contact_data"/> </container> </xacro:pioneer_swivel>
+    <xacro:pioneer_swivel  name="swivel"    parent="${parent}"  xyz="-0.185 0    0.0535" rpy="0 0 0"/>
     <!-- Wheels -->
     <xacro:pioneer_wheel name="right" parent="${parent}"  xyz=" 0    -0.165 ${wheel_radius}" rpy="0 0 0" radius="${wheel_radius}"> <container> <xacro:insert_block name="contact_data"/> </container> </xacro:pioneer_wheel>

File: tuw_gazebo_models/models/pioneer3dx/body/swivel.xacro (robot description, xacro)
@@ -2,5 +2,5 @@
 <robot xmlns:xacro="http://ros.org/wiki/xacro">
   <xacro:property name="M_PI" value="3.1415926535897931" />
-  <xacro:macro name="pioneer_swivel" params="name parent xyz rpy models_dir:=^ **contact_data">
+  <xacro:macro name="pioneer_swivel" params="name parent xyz rpy models_dir:=^ ">
   <!-- Swivel -->
   <joint name="${name}_joint" type="continuous">
@@ -14,9 +14,5 @@
   </joint>
   <link name="${name}">
-    <inertial>
-      <mass value="0.1"/>
-      <origin xyz="0 0 0"/>
-      <inertia ixx="0.01" ixy="0" ixz="0" iyy="0.01" iyz="0" izz="0.01"/>
-    </inertial>
+    <xacro:box_inertial x="0.01" y="0.01"  z="0.01" mass="0.01" />
     <visual>
       <origin xyz="0 0 0" rpy="0 0 0"/>
@@ -41,17 +37,11 @@
   <joint name="${name}_wheel_joint" type="continuous">
     <origin xyz="-0.026 0 -0.016" rpy="0 0 0"/>
-    <axis xyz="0 1 0"/>
+    <axis xyz="0 1 0" />
     <anchor xyz="0 0 0"/>
-    <!--limit effort="100" velocity="100" k_velocity="0"/-->
-    <joint_properties damping="0.0" friction="0.0"/>
     <parent link="${name}"/>
     <child link="${name}_wheel"/>
   </joint>
   <link name="${name}_wheel">
-    <inertial>
-      <mass value="0.1"/>
-      <origin xyz="0 0 0"/>
-      <inertia ixx="0.012411765597" ixy="-0.000711733678" ixz="0.00050272983" iyy="0.015218160428" iyz="-0.000004273467" izz="0.011763977943"/>
-    </inertial>
+		<xacro:cylinder_inertial_with_origin radius="${0.0375}" length="0.02" mass="0.5" xyz="0 0 0" rpy="${pi/2} 0 0"/>
     <visual>
       <origin xyz="0 0 0" rpy="0 0 0"/>
@@ -66,6 +56,5 @@
       <origin xyz="0 0 0" rpy="${-3.1415927/2.0} 0 0"/>
       <geometry>
-        <!--<mesh filename="meshes/center_wheel.stl"/>-->
-        <cylinder radius="0.0375" length="0.001"/> <!--radius="0.0375"-->
+        <cylinder radius="0.0375" length="0.001"/>
       </geometry>
     </collision>
@@ -73,5 +62,4 @@
   <gazebo reference="${name}_wheel">
     <material value="Gazebo/Black"/>
-    <xacro:insert_block name="contact_data"/>
   </gazebo>
   <!-- Center Hubcap -->
@@ -82,9 +70,5 @@
   </joint>
   <link name="${name}_hubcap">
-    <inertial>
-      <mass value="0.01"/>
-      <origin xyz="0 0 0"/>
-      <inertia ixx="0.012411765597" ixy="-0.000711733678" ixz="0.00050272983" iyy="0.015218160428" iyz="-0.000004273467" izz="0.011763977943"/>
-    </inertial>
+    <xacro:box_inertial x="0.01" y="0.01"  z="0.01" mass="0.01" />
     <visual>
       <origin xyz="0 0 0" rpy="0 0 0"/>
@@ -105,5 +89,4 @@
   <gazebo reference="${name}_hubcap">
     <material value="Gazebo/Grey"/>
-    <xacro:insert_block name="contact_data"/>
   </gazebo>
   </xacro:macro>

Commit message: wheels

File: tuw_gazebo_models/models/pioneer3dx/body/body.xacro (robot description, xacro)
@@ -32,6 +32,6 @@
     <xacro:pioneer_swivel  name="swivel"    parent="${parent}"  xyz="-0.185 0    0.0535" rpy="0 0 0"/>
     <!-- Wheels -->
-    <xacro:pioneer_wheel name="right" parent="${parent}"  xyz=" 0    -0.165 ${wheel_radius}" rpy="0 0 0" radius="${wheel_radius}"> <container> <xacro:insert_block name="contact_data"/> </container> </xacro:pioneer_wheel>
-    <xacro:pioneer_wheel name="left"  parent="${parent}"  xyz=" 0     0.165 ${wheel_radius}" rpy="0 0 0" radius="${wheel_radius}"> <container> <xacro:insert_block name="contact_data"/> </container> </xacro:pioneer_wheel>
+    <xacro:pioneer_wheel name="right" parent="${parent}"  xyz=" 0    -0.165 ${wheel_radius}" rpy="0 0 0" radius="${wheel_radius}"/>
+    <xacro:pioneer_wheel name="left"  parent="${parent}"  xyz=" 0     0.165 ${wheel_radius}" rpy="0 0 0" radius="${wheel_radius}"/>
   </xacro:macro>
 </robot>

File: tuw_gazebo_models/models/pioneer3dx/body/wheel.xacro (robot description, xacro)
@@ -2,32 +2,30 @@
 <robot
   xmlns:xacro="http://ros.org/wiki/xacro">
-  <xacro:property name="M_PI" value="3.1415926535897931" />
-  <xacro:macro name="pioneer_wheel" params="name parent xyz rpy radius models_dir:=^ **contact_data">
+  <xacro:macro name="pioneer_wheel" params="name parent xyz rpy radius models_dir:=^">
     <!-- Wheel -->
     <joint name="${name}_wheel_joint" type="continuous">
 		<origin xyz="${xyz}" rpy="${rpy}"/>
-		<axis xyz="0 1 0"/>
 		<parent link="${parent}"/>
 		<child link="${name}_wheel"/>
+		<axis xyz="0 1 0"/>
     </joint>
     <link name="${name}_wheel">
-		<inertial>
-			<mass value="0.5"/>
-			<origin xyz="0 0 0"/>
-			<inertia ixx="0.012411765597" ixy="0" ixz="0" iyy="0.015218160428" iyz="0" izz="0.011763977943"/>
-		</inertial>
+		<xacro:cylinder_inertial_with_origin radius="${radius}" length="0.02" mass="0.5" xyz="0 0 0" rpy="${pi/2} 0 0"/>
 		<visual>
 			<origin xyz="0 0 0" rpy="0 0 0"/>
-			<geometry> <mesh filename="file://${models_dir}/pioneer3dx/body/meshes/wheel.dae"/> </geometry>
+			<geometry>
+				<mesh filename="file://${models_dir}/pioneer3dx/body/meshes/wheel.dae"/>
+			</geometry>
 			<material name="WheelBlack"> <color rgba="0.117 0.117 0.117 1"/> </material>
 		</visual>
 		<collision>
 			<origin xyz="0 0 0" rpy="${pi/2} 0 0"/>
-			<geometry> <cylinder radius="${radius}" length="0.001"/> <!--<mesh filename="${meshes}/${name}_wheel.stl"/>--> </geometry>
+			<geometry>
+				<cylinder radius="${radius}" length="0.001"/>
+			</geometry>
 		</collision>
     </link>
 		<gazebo reference="${name}_wheel">
 		<material value="Gazebo/Black"/>
-	<xacro:insert_block name="contact_data"/>
     </gazebo>
     <!-- Hubcap -->
@@ -39,17 +37,16 @@
     </joint>
     <link name="${name}_hub">
-		<inertial>
-			<mass value="0.01"/>
-			<origin xyz="0 0 0"/>
-			<inertia ixx="0.012411765597" ixy="0" ixz="0" iyy="0.015218160428" iyz="0" izz="0.011763977943"/>
-		</inertial>
 		<visual>
 			<origin xyz="0 0 0" rpy="0 0 0"/>
-			<geometry> <mesh filename="file://${models_dir}/pioneer3dx/body/meshes/hubcap.dae"/> </geometry>
+			<geometry>
+				<mesh filename="file://${models_dir}/pioneer3dx/body/meshes/hubcap.dae"/>
+			</geometry>
 			<material name="HubcapYellow"> <color rgba="1.0 0.811 0.151 1.0"/> </material>
 		</visual>
 		<collision>
 			<origin xyz="0 0 0" rpy="0 0 0"/>
-			<geometry> <box size="0.001 0.001 0.001"/> </geometry>
+			<geometry>
+				<box size="0.001 0.001 0.001"/>
+			</geometry>
 		</collision>
     </link>
