Commit message: arguments on xacro files are now working

File: tuw_gazebo_models/models/pioneer3dx/main.xacro (robot description, xacro)
@@ -8,16 +8,18 @@
   <xacro:arg name="laser0_topic"     default="scan_raw"/>
   <xacro:arg name="laser0_visualize" default="true"/>
-  <xacro:property name="models_dir" value="$(arg models_dir)"/>
-  <xacro:property name="robot_model" value="$(arg robot_model)"/>
-  <xacro:property name="laser_model" value="$(arg laser_model)"/>
+  <xacro:arg name="laser0_driver"    default="gpu"/>
+  <xacro:property name="models_dir"    value="$(arg models_dir)"/>
+  <xacro:property name="namespace"    value="$(arg namespace)"/>
+  <xacro:property name="robot_model"   value="$(arg robot_model)"/>
+  <xacro:property name="laser_model"   value="$(arg laser_model)"/>
   <!-- Import Rviz colors -->
-  <xacro:include filename="$(arg models_dir)/materials.xacro" />
+  <xacro:include filename="${models_dir}/materials.xacro" />
   <!-- Import platform -->
   <xacro:include filename="${models_dir}/${robot_model}/body/body.xacro"/>
   <xacro:vehicle_body name="body" parent="base_link"/>
   <xacro:include filename="${models_dir}/${robot_model}/plugins.xacro"/>
-  <xacro:differential_drive    name="$(arg robot_name)" namespace="$(arg namespace)" />
-  <xacro:joint_state_publisher name="$(arg robot_name)" namespace="$(arg namespace)" />
+  <xacro:differential_drive    name="$(arg robot_name)" namespace="${namespace}" />
+  <xacro:joint_state_publisher name="$(arg robot_name)" namespace="${namespace}" />
   <xacro:include filename="${models_dir}/${laser_model}/main.xacro"/>
-  <xacro:laser name="laser0" parent="top" namespace="$(arg namespace)" topic_name="$(arg laser0_topic)" frame_name="laser0" xyz="0.15 0.0 0.06" rpy="0 0 0" driver="gpu" visualize="true"/>
+  <xacro:laser name="laser0" parent="top" namespace="${namespace}" topic_name="$(arg laser0_topic)" frame_name="laser0" xyz="0.15 0.0 0.06" rpy="0 0 0" driver="$(arg laser0_driver)" visualize="$(arg laser0_visualize)"/>
 </robot>

Commit message: multi robot simulation in Gazebo

File: tuw_gazebo_models/models/pioneer3dx/main.xacro (robot description, xacro)
@@ -9,8 +9,10 @@
   <xacro:arg name="laser0_visualize" default="true"/>
   <xacro:arg name="laser0_driver"    default="cpu"/>
+  <xacro:arg name="version"  	     default="v1"/>
   <xacro:property name="models_dir"    value="$(arg models_dir)"/>
   <xacro:property name="namespace"    value="$(arg namespace)"/>
   <xacro:property name="robot_model"   value="$(arg robot_model)"/>
   <xacro:property name="laser_model"   value="$(arg laser_model)"/>
+  <xacro:property name="version"    value="$(arg version)"/>
   <!-- Import Rviz colors -->
   <xacro:include filename="${models_dir}/materials.xacro" />
@@ -19,9 +21,9 @@
   <xacro:vehicle_body name="body" parent="base_link"/>
   <!-- differential drive  and joint stage plugin -->
-  <xacro:include filename="${models_dir}/${robot_model}/plugins.xacro"/>
+  <xacro:include filename="${models_dir}/${robot_model}/plugins_${version}.xacro"/>
   <xacro:differential_drive    name="$(arg robot_name)" namespace="${namespace}" />
   <xacro:joint_state_publisher name="$(arg robot_name)" namespace="${namespace}" />
   <!-- Laser -->
-  <xacro:include filename="${models_dir}/${laser_model}/main.xacro"/>
+  <xacro:include filename="${models_dir}/${laser_model}/main_${version}.xacro"/>
   <xacro:laser name="laser0" parent="top" namespace="${namespace}" topic_name="$(arg laser0_topic)" frame_name="laser0" xyz="0.15 0.0 0.06" rpy="0 0 0" driver="$(arg laser0_driver)" visualize="$(arg laser0_visualize)"/>
 </robot>

File: tuw_gazebo_models/models/pioneer3dx/plugins_v1.xacro (robot description, xacro)
@@ -20,6 +20,6 @@
           <odometry_source>0</odometry_source>
           <publish_odom_ground_truth>true</publish_odom_ground_truth>
-          <odometry_frame>odom</odometry_frame>
-          <robot_base_frame>base_link</robot_base_frame>
+          <odometry_frame>${namespace}/odom</odometry_frame>
+          <robot_base_frame>${namespace}/base_link</robot_base_frame>
       </plugin>
     </gazebo>
